File: CAD/MIDIperformer-Rev1/midiperformer/midiperformer.kicad_sch (KiCad schematic)
At the start: 41 parts, among them J1 MIDI IN B, J2 MIDI IN A, J3 MIDI OUT A, J4 MIDI OUT B, J5 Barrel_Jack, SW1 SW_Push_SPDT, SW2 RotaryEncoder_Switch, SW3 SW_Push_SPDT, SW4 SW_Push_SPDT, SW5 SW_Push_SPDT, SW6 SW_Push_SPDT, SW7 SW_Push_SPDT, SW8 SW_Push_SPDT, U1 6N138, U2 6N138, U3 L7805, U4 Teensy-LC, U5 WS2812, U6 MCP23017_SP

Commit message: progress on midiperformer; this one is being printed progress on clarinoid3 schematic; very WIP
Parts:
- C1, C2: footprint Capacitor_THT:C_Disc_D3.8mm_W2.6mm_P2.50mm -> Capacitor_SMD:C_0603_1608Metric
- D1, D2: footprint Diode_THT:D_DO-35_SOD27_P7.62mm_Horizontal -> Diode_SMD:D_SOD-123
- R1, R10, R11, R12, R2, R3, R4, R5, R6, R7, R8, R9: footprint Resistor_THT:R_Axial_DIN0207_L6.3mm_D2.5mm_P10.16mm_Horizontal -> Resistor_SMD:R_0603_1608Metric
- U1, U2: footprint Package_DIP:DIP-8_W7.62mm -> Package_DIP:SMDIP-8_W7.62mm
