File: CAD/clarinoid-devboard/clarinoid-devboard/clarinoid-devboard.kicad_pcb (KiCad board)
At the start: 2 copper layers, 166.6 x 99.8 mm, 120 parts, among them IC1 PCA9554APW,118, IC2 Injoinic IP5306 battery charge, IC3 AT42QT2120-XU, IC4 CY8CMBR3108-LQXIT, J1 TRS jack, J10 MIDI IN, J11 MIDI OUT, J12 SSD1306, J13 conn_buttons_PCA9554, J14 touch_conn_mpr121, J15 conn_buttons_MCP, J16 touch_conn_qtouch, J17 touch_conn_qtouch, J18 conn_buttons_B, J2 USB_C_Receptacle_USB2.0, J3 Molex microSD 503398-1892, J4 CapTouchSlider_8, J5 CapTouchSlider_8, J6 CapTouchSlider_8, J7 CapTouchSlider_8, J8 CapTouchSlider_8, J9 CapTouchSlider_8, SW1 SW_Push, SW10 SW_Push, SW11 RotaryEncoder_Switch, SW2 SW_Push, SW3 SW_Push, SW4 SW_Push, SW5 SW_Push, SW6 SW_Push, SW7 SW_Push, SW8 SW_Push, SW9 SW_Push, U1 PCM5102, U2 TLV75533PDBV, U3 Teensy_4.0_MicroMod, U4 MPR121QR2, U5 octave_keys_7, U6 MCP23017_SP, U7 TLV75533PDBV, U8 6N138, U9 WS2812

Commit message: incremental progress of clarinoid test device renaming midi performer to prepare for rev2
Parts:
- removed BT1: Battery_Cell, clarinoid2:KEYSTONE_1043
- removed C1, C2: 0.1uF, Capacitor_SMD:C_0402_1005Metric
- removed J16, J17: touch_conn_qtouch, clarinoid2:solder point DIP 1x7
- removed J4: CapTouchSlider_8, CapTouchSliders:CaptouchSlider_Masked_x8_2pt_12x6x6x0.5mm
- removed J6: CapTouchSlider_8, CapTouchSliders:CaptouchSlider_Masked_x8_2pt_12x6x6x1.5mm
- removed J7: CapTouchSlider_8, CapTouchSliders:CaptouchSlider_Masked_x8_2pt_12x6x6x2.0mm
- removed SW10, SW8, SW9: SW_Push, clarinoid2:MB2511S2G45
- removed SW7: SW_Push, SamacSys_Parts:B3F-4055
- removed U2: TLV75533PDBV, Package_TO_SOT_SMD:SOT-23-5
- added C26: 10uF, Capacitor_SMD:C_0603_1608Metric, F.Cu at (137.6, 78.6)
- added C28: 0.22uF, Capacitor_SMD:C_0603_1608Metric, F.Cu at (138.8, 79.7)
- added C29: 0.1uF, Capacitor_SMD:C_0603_1608Metric, F.Cu at (139.9, 80.9)
- added C30: 0.1uF, Capacitor_SMD:C_0402_1005Metric, F.Cu at (226.3, 108.5)
- added H1: M.2 riser SMTSO2530CTJ, clarinoid2:Wurth_9774025151_M2.5_spacer_for_micromod, F.Cu at (130.4, 84.1)
- added NT1: NetTie_2, NetTie:NetTie-2_SMD_Pad0.5mm, F.Cu at (112.6, 106.6)
- added R40: 10k, Resistor_SMD:R_0402_1005Metric, F.Cu at (203.0, 86.8)
- added R41: 10k, Resistor_SMD:R_0402_1005Metric, F.Cu at (203.0, 89.7)
- added R43: 10k, Resistor_SMD:R_0402_1005Metric, F.Cu at (230.4, 112.3)
- added R44: 10k, Resistor_SMD:R_0402_1005Metric, F.Cu at (230.4, 110.3)
- added U10: Pressure1_0x28_I2C0, SamacSys_Parts:ABPMAND001PG2A3, F.Cu at (209.6, 87.9)
- added U11: TLV75733PDBV, Package_TO_SOT_SMD:SOT-23-5, F.Cu at (142.0, 82.9)
- added U12: ssd1306_graphic, clarinoid2:SSD1306_128x64_approximate, F.Cu at (119.6, 120.1)
- C11: value 0.1uF -> 10uF
- C14: value 10uF -> 0.1uF
- J12: footprint clarinoid2:solder point DIP 1x7 -> Connector_PinSocket_2.54mm:PinSocket_1x07_P2.54mm_Vertical
- J13: footprint clarinoid2:solder point DIP 1x6 -> Connector_PinSocket_2.54mm:PinSocket_1x08_P2.54mm_Vertical
- J14: value touch_conn_mpr121 -> touch_conn_capsense; footprint clarinoid2:solder point DIP 1x7 -> Connector_PinSocket_2.54mm:PinSocket_1x08_P2.54mm_Vertical
- J15: footprint clarinoid2:solder point DIP 1x7 -> Connector_PinSocket_2.54mm:PinSocket_1x08_P2.54mm_Vertical
- J18: value conn_buttons_B -> conn_buttons_btn; footprint clarinoid2:solder point DIP 1x6 -> Connector_PinSocket_2.54mm:PinSocket_1x04_P2.54mm_Vertical
- J2: value USB_C_Receptacle_USB2.0 -> XKB_U262-16XN-4BVC11 USB-C recept; footprint Connector_USB:USB_C_Receptacle_XKB_U262-16XN-4BVC11 -> clarinoid2:USB_C_Receptacle_XKB_U262-16XN-4BVC11
- J5: value CapTouchSlider_8 -> header_i2c; footprint CapTouchSliders:CaptouchSlider_Masked_x8_2pt_12x6x6x1.0mm -> Connector_PinSocket_2.54mm:PinSocket_1x04_P2.54mm_Vertical
- J8: value CapTouchSlider_8 -> touch_conn_mpr121; footprint CapTouchSliders:CaptouchSlider_Bare_x8_1pt_10x5x5x0.5mm -> Connector_PinSocket_2.54mm:PinSocket_1x08_P2.54mm_Vertical
- J9: value CapTouchSlider_8 -> touch_conn_qtouch; footprint CapTouchSliders:CaptouchSlider_Bare_x8_2pt_16x8x6x2mm -> Connector_PinSocket_2.54mm:PinSocket_1x08_P2.54mm_Vertical
- L1: value 1UH -> 1uH; footprint Inductor_SMD:L_Bourns_SRP7028A_7.3x6.6mm -> clarinoid2:Inductor_MCS0630-1R0MN2
- R1, R2, R3: value 22 -> 22R
- R19: value 220 -> 220R
- R20, R21: value 47 -> 47R
- R22, R5, R6: value 470 -> 470R
- R34, R35, R36, R37, R38, R39: value 500 -> 470R
- SW6: footprint SamacSys_Parts:B3F-4055 -> SamacSys_Parts:TL3305AF160QG
- U1: value PCM5102 -> PCM5102A
- U3: value Teensy_4.0_MicroMod -> APCI0136-P001A Teensy_4.0_MicroMod; footprint Teensy_MicroMod_KiCad:Teensy_4.0_MicroMod -> clarinoid2:Teensy_4.0_MicroMod_nospacer
- U5: value octave_keys_7 -> Keystone 1043; footprint clarinoid2:CLARINOID_M6_6OCTAVES -> SamacSys_Parts:1043
- U9: footprint clarinoid2:solder point DIP 1x3 -> Connector_PinSocket_2.54mm:PinSocket_1x03_P2.54mm_Vertical
- moved J8 339.9 mm to (189.3, 101.7)
- moved J9 314.8 mm to (213.2, 101.7)
- moved R31 307.6 mm to (206.8, 120.5), turned to -90 degrees
- moved IC4 307.5 mm to (227.5, 111.2), turned to -90 degrees
- moved R32 306.5 mm to (205.8, 120.5), turned to -90 degrees
- moved J18 306.3 mm to (208.3, 130.8)
- moved R33 304.3 mm to (203.8, 120.5), turned to -90 degrees
- moved R4 303.7 mm to (197.1, 112.2)
- moved R14 302.5 mm to (198.7, 111.8), turned to -90 degrees
- moved IC3 301.8 mm to (205.5, 115.4), turned to -90 degrees
- moved R25 299.8 mm to (208.4, 109.4), turned to -90 degrees
- moved R13 299.7 mm to (199.4, 109.8), turned to 90 degrees
- moved R26 298.7 mm to (207.4, 109.4), turned to -90 degrees
- moved U4 297.8 mm to (195.6, 109.4), turned to 180 degrees
- moved R27 297.5 mm to (206.4, 109.4), turned to -90 degrees
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Connections:
- C10 pad 2: A3v3 -> GND
- C11 pad 1: A3v3 -> GND
- C11 pad 2: GND -> D3v3
- C13 pad 2: A3v3 -> GND
- C14 pad 1: A3v3 -> GND
- C14 pad 2: GND -> D3v3
- C5 pad 1: D3v3 -> +3V3
- C6 pad 1: D3v3 -> +3V3
- IC1 pad 10: Net-(J13-Pad6) -> Net-(IC1-Pad10)
- IC4 pad 1: unconnected-(IC4-Pad1) -> Net-(IC4-Pad1)
- IC4 pad 11: unconnected-(IC4-Pad11) -> Net-(IC4-Pad11)
- IC4 pad 12: unconnected-(IC4-Pad12) -> Net-(IC4-Pad12)
- IC4 pad 13: unconnected-(IC4-Pad13) -> Net-(IC4-Pad13)
- IC4 pad 14: unconnected-(IC4-Pad14) -> I2C_SDA
- IC4 pad 15: unconnected-(IC4-Pad15) -> I2C_SCL
- IC4 pad 17: unconnected-(IC4-Pad17) -> GND
- IC4 pad 2: unconnected-(IC4-Pad2) -> Net-(IC4-Pad2)
- IC4 pad 4: unconnected-(IC4-Pad4) -> Net-(C30-Pad1)
- IC4 pad 5: unconnected-(IC4-Pad5) -> +3V3
- IC4 pad 6: unconnected-(IC4-Pad6) -> +3V3
- IC4 pad 8: unconnected-(IC4-Pad8) -> Net-(IC4-Pad8)
- IC4 pad 9: unconnected-(IC4-Pad9) -> Net-(IC4-Pad9)
- J13 pad 1: Net-(IC1-Pad4) -> +3V3
- J13 pad 2: Net-(IC1-Pad5) -> GND
- J13 pad 3: Net-(IC1-Pad6) -> Net-(IC1-Pad4)
- J13 pad 4: Net-(IC1-Pad7) -> Net-(IC1-Pad5)
- J13 pad 5: Net-(IC1-Pad9) -> Net-(IC1-Pad6)
- J13 pad 6: Net-(J13-Pad6) -> Net-(IC1-Pad7)
- J14 pad 1: Net-(U4-Pad8) -> GND
- J14 pad 2: Net-(U4-Pad9) -> Net-(IC4-Pad1)
- J14 pad 3: Net-(U4-Pad10) -> Net-(IC4-Pad2)
- J14 pad 4: Net-(U4-Pad11) -> Net-(IC4-Pad12)
- J14 pad 5: Net-(U4-Pad12) -> Net-(IC4-Pad13)
- J14 pad 6: Net-(U4-Pad13) -> Net-(IC4-Pad8)
- J14 pad 7: Net-(U4-Pad14) -> Net-(IC4-Pad9)
- J15 pad 1: Net-(U6-Pad1) -> +3V3
- J15 pad 2: Net-(U6-Pad2) -> GND
- J15 pad 3: Net-(U6-Pad3) -> Net-(J15-Pad3)
- J15 pad 4: Net-(U6-Pad4) -> Net-(J15-Pad4)
- J15 pad 5: Net-(U6-Pad5) -> Net-(J15-Pad5)
- J15 pad 6: Net-(U6-Pad6) -> Net-(J15-Pad6)
- J15 pad 7: (no net) -> Net-(J15-Pad7)
- J2 pad A8: unconnected-(J2-PadA8) -> (no net)
- J2 pad B6: USB data in + -> (no net)
- J2 pad B7: USB data in - -> (no net)
- J2 pad B8: unconnected-(J2-PadB8) -> (no net)
- J5 pad 1: unconnected-(J5-Pad1) -> GND
- J5 pad 2: unconnected-(J5-Pad2) -> +3V3
- J5 pad 3: unconnected-(J5-Pad3) -> I2C_SDA
- J5 pad 4: unconnected-(J5-Pad4) -> I2C_SCL
- J8 pad 1: unconnected-(J8-Pad1) -> GND
- J8 pad 2: unconnected-(J8-Pad2) -> Net-(J8-Pad2)
- J8 pad 3: unconnected-(J8-Pad3) -> Net-(J8-Pad3)
- J8 pad 4: unconnected-(J8-Pad4) -> Net-(J8-Pad4)
- J8 pad 5: unconnected-(J8-Pad5) -> Net-(J8-Pad5)
- J8 pad 6: unconnected-(J8-Pad6) -> Net-(J8-Pad6)
- J8 pad 7: GND -> Net-(J8-Pad7)
- J8 pad 8: GND -> Net-(J8-Pad8)
- J9 pad 1: unconnected-(J9-Pad1) -> GND
- J9 pad 2: unconnected-(J9-Pad2) -> Net-(J9-Pad2)
- J9 pad 3: unconnected-(J9-Pad3) -> Net-(J9-Pad3)
- J9 pad 4: unconnected-(J9-Pad4) -> Net-(J9-Pad4)
- J9 pad 5: unconnected-(J9-Pad5) -> Net-(J9-Pad5)
- J9 pad 6: unconnected-(J9-Pad6) -> Net-(J9-Pad6)
- J9 pad 7: GND -> Net-(J9-Pad7)
- J9 pad 8: GND -> Net-(J9-Pad8)
- R24 pad 1: Net-(J16-Pad3) -> Net-(J9-Pad4)
- R25 pad 1: Net-(J16-Pad7) -> Net-(J9-Pad8)
- R26 pad 1: Net-(J16-Pad6) -> Net-(J9-Pad7)
- R27 pad 1: Net-(J16-Pad5) -> Net-(J9-Pad6)
- R28 pad 1: Net-(J16-Pad4) -> Net-(J9-Pad5)
- R29 pad 1: Net-(J16-Pad2) -> Net-(J9-Pad3)
- R30 pad 1: Net-(J16-Pad1) -> Net-(J9-Pad2)
- SW6 pad 1: GND -> Net-(SW6-Pad1)
- SW6 pad 2: Net-(J18-Pad5) -> GND
- U3 pad 11: unconnected-(U3-Pad11) -> Net-(SW6-Pad1)
- U3 pad 46: OLED_RES -> OLED_DC
- U3 pad 48: OLED_DC -> OLED_RES
- U3 pad 59: SDIO_MOSI -> SPI0_MOSI
- U4 pad 10: Net-(U4-Pad10) -> Net-(J8-Pad4)
- U4 pad 11: Net-(U4-Pad11) -> Net-(J8-Pad5)
- U4 pad 12: Net-(U4-Pad12) -> Net-(J8-Pad6)
- U4 pad 13: Net-(U4-Pad13) -> Net-(J8-Pad7)
- U4 pad 14: Net-(U4-Pad14) -> Net-(J8-Pad8)
- U4 pad 8: Net-(U4-Pad8) -> Net-(J8-Pad2)
- U4 pad 9: Net-(U4-Pad9) -> Net-(J8-Pad3)
- U5 pad 1: unconnected-(U5-Pad1) -> Batt+
- U5 pad 2: unconnected-(U5-Pad2) -> GND
- U6 pad 1: Net-(U6-Pad1) -> Net-(J15-Pad3)
- U6 pad 2: Net-(U6-Pad2) -> Net-(J15-Pad4)
- U6 pad 3: Net-(U6-Pad3) -> Net-(J15-Pad5)
- U6 pad 4: Net-(U6-Pad4) -> Net-(J15-Pad6)
- U6 pad 5: Net-(U6-Pad5) -> Net-(J15-Pad7)
- U6 pad 6: Net-(U6-Pad6) -> Net-(J15-Pad8)
- U7 pad 1: +3V3 -> D3v3
- U7 pad 3: +3V3 -> D3v3
Routing:
- net +3V3: track 9.92 -> 391.6 mm, vias 0 -> 13
- net GND: track 0.00 -> 241.5 mm, vias 0 -> 15
- net I2C_SDA: track 4.93 -> 200.4 mm, vias 0 -> 3
- net I2C_SCL: track 5.30 -> 194.5 mm, vias 0 -> 2
- net Net-(J18-Pad1): track 0.00 -> 131.8 mm
- net Net-(J18-Pad3): track 0.00 -> 126.6 mm
- net Net-(J15-Pad3): track 0.00 -> 124.1 mm, vias 0 -> 3
- net Net-(J15-Pad4): track 0.00 -> 120.5 mm, vias 0 -> 3
- net Net-(J18-Pad2): track 0.00 -> 119.2 mm
- net Net-(J15-Pad5): track 0.00 -> 113.3 mm, vias 0 -> 3
- net Net-(J18-Pad4): track 0.00 -> 110.6 mm
- net Net-(J15-Pad6): track 0.00 -> 109.1 mm, vias 0 -> 3
- net Net-(J15-Pad7): track 0.00 -> 105.6 mm, vias 0 -> 3
- net Supply+5v: track 8.87 -> 113.3 mm, vias 0 -> 6
- net Net-(J15-Pad8): track 0.00 -> 102.2 mm, vias 0 -> 3
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- added copper zone on B.Cu, net GND
Other:
- board size 166.6 x 99.8 mm -> 154 x 99 mm
- board text added: "100% 75% 50% 25%"
- board text added: "Capsense 0x37"
- board text added: "I2C -scl -sda -3v3 -gnd"
- board text added: "MCP23017 0x20"
- board text added: "MPR121 0x5A"
- board text added: "Onboard Buttons"
- board text added: "PCA9554APW,118"
- board text added: "WS2812b +3v Data GND"
- board text removed: "Capsense"
- board text removed: "MCP23017"
- board text removed: "MPR121"
- board text removed: "QTouch"
- board text removed: "adafruit mpr121 footprint"
- board text removed: "chrg"
- board text removed: "hiletgo footprint"
- board text removed: "mh-cd42 footprint"
- board text removed: "teensy 4.0 footprint"
