File: CAD/clarinoid-devboard/clarinoid-devboard-01/clarinoid-devboard.kicad_sch (KiCad schematic)
At the start: 120 parts, among them IC1 PCA9554APW,118, IC2 Injoinic IP5306 battery charge, IC3 AT42QT2120-XU, IC4 CY8CMBR3108-LQXIT, J1 TRS jack, J10 MIDI IN, J11 MIDI OUT, J12 SSD1306, J13 conn_buttons_PCA9554, J14 touch_conn_capsense, J15 conn_buttons_MCP, J18 conn_buttons_btn, J2 XKB_U262-16XN-4BVC11 USB-C re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, J3 Molex microSD 503398-1892, J5 header_i2c, J8 touch_conn_mpr121, J9 touch_conn_qtouch, SW1 SW_Push, SW11 RotaryEncoder_Switch, SW2 SW_Push, SW3 SW_Push, SW4 SW_Push, SW5 SW_Push, SW6 SW_Push, U1 PCM5102A, U10 Pressure1_0x28_I2C0, U11 TLV75733PDBV, U12 ssd1306_graphic, U3 APCI0136-P001A Teensy_4.0_Mic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, U4 MPR121QR2, U5 Keystone 1043, U6 MCP23017_SP, U7 TLV75533PDBV, U8 6N138, U9 WS2812

Commit message: incremental progress of clarinoid test device renaming midi performer to prepare for rev2
Parts:
- removed IC3: AT42QT2120-XU, SamacSys_Parts:SOP65P638X120-20N, symbol clarinoid2:Atmel QTouch AT42QT2120-XU - COMM mode
- removed J15: conn_buttons_MCP, Connector_PinSocket_2.54mm:PinSocket_1x08_P2.54mm_Vertical, symbol Connector_Generic:Conn_01x08
- removed J18: conn_buttons_btn, Connector_PinSocket_2.54mm:PinSocket_1x04_P2.54mm_Vertical, symbol Connector_Generic:Conn_01x04
- removed J9: touch_conn_qtouch, Connector_PinSocket_2.54mm:PinSocket_1x08_P2.54mm_Vertical, symbol Connector_Generic:Conn_01x08
- removed R27, R28, R29, R30: 4.7k, Resistor_SMD:R_0402_1005Metric, symbol Device:R
- removed R31, R32, R33: 10k, Resistor_SMD:R_0402_1005Metric, symbol Device:R
- removed U6: MCP23017_SP, Package_DIP:DIP-28_W7.62mm, symbol Interface_Expansion:MCP23017_SP
- added C1, C2: 0.1uF, Capacitor_SMD:C_0402_1005Metric, symbol Device:C
- added IC3: PCA9554APW,118, SamacSys_Parts:SOP65P640X110-16N, symbol SamacSys_Parts:PCA9554APW,118
- added J15: CapTouchSlider1, CapTouchSliders:CaptouchSlider_Masked_x8_2pt_12x6x6x0.5mm, symbol clarinoid2:CapTouchSlider_8
- added J16: CapTouchSlider2, CapTouchSliders:CaptouchSlider_Masked_x8_2pt_12x6x6x1.0mm, symbol clarinoid2:CapTouchSlider_8
- added J19: SB_slider4_header, Connector_PinSocket_2.54mm:PinSocket_1x06_P2.54mm_Vertical, symbol Connector_Generic:Conn_01x06
- added J20: CapTouchSlider3, CapTouchSliders:CaptouchSlider_Masked_x8_2pt_12x6x6x1.5mm, symbol clarinoid2:CapTouchSlider_8
- added J21: CapTouchSlider4, CapTouchSliders:CaptouchSlider_Masked_x8_2pt_12x6x6x2.0mm, symbol clarinoid2:CapTouchSlider_8
- added J4: capsense_subboard_header, Connector_PinSocket_2.54mm:PinSocket_1x04_P2.54mm_Vertical, symbol Connector_Generic:Conn_01x04
- added J6: SB_octaves_header, Connector_PinSocket_2.54mm:PinSocket_1x06_P2.54mm_Vertical, symbol Connector_Generic:Conn_01x06
- added J7: SB_slider1_header, Connector_PinSocket_2.54mm:PinSocket_1x06_P2.54mm_Vertical, symbol Connector_Generic:Conn_01x06
- added J9: SB_slider2_header, Connector_PinSocket_2.54mm:PinSocket_1x06_P2.54mm_Vertical, symbol Connector_Generic:Conn_01x06
- added U2: octave_keys_6, clarinoid2:CLARINOID_M6_6OCTAVES_offset, symbol clarinoid2:octave_keys_6
- added U6: MPR121, 0x5C, Package_DFN_QFN:UQFN-20_3x3mm_P0.4mm, symbol Sensor_Touch:MPR121QR2
- C10, C11, C15, C16, C3, C5: LCSC part number (none) -> C15525
- C12, C7, C8, C9: LCSC part number (none) -> C12530
- C13, C14, C23, C24, C25, C30, C4, C6: LCSC part number (none) -> C1525
- C17, C18, C19, C20, C21, C22: footprint Capacitor_SMD:C_0402_1005Metric -> Capacitor_SMD:C_0603_1608Metric; LCSC part number (none) -> C59461
- C26: footprint Capacitor_SMD:C_0603_1608Metric -> Capacitor_SMD:C_0402_1005Metric; symbol Device:C_Polarized_US -> Device:C; LCSC part number (none) -> C15525
- C27: footprint Capacitor_SMD:C_0603_1608Metric -> Capacitor_SMD:C_0402_1005Metric; symbol Device:C_Polarized_Small_US -> Device:C; LCSC part number (none) -> C1525
- C28: symbol pspice:C -> Device:C; LCSC part number (none) -> C21120
- C29: symbol pspice:C -> Device:C; LCSC part number (none) -> C14663
- D1, D2, D3, D4: LCSC part number (none) -> C84256
- D10, D11, D5, D7, D8, D9: LCSC part number (none) -> C72038
- D6: LCSC part number (none) -> C2128
- H1: LCSC part number (none) -> C2915631
- IC1: LCSC part number (none) -> C86803
- IC2: LCSC part number (none) -> C181692
- IC4: LCSC part number (none) -> C462528
- J1, J10, J11: LCSC part number (none) -> ??
- J12, J13, J14, J5, J8, NT1, U10, U12, U9: LCSC part number (none) -> -
- J2: LCSC part number (none) -> C319148
- J3: LCSC part number (none) -> C428492
- L1: LCSC part number (none) -> C385251
- R1, R2, R3: LCSC part number (none) -> C25092
- R10: value 10K -> 10k; LCSC part number (none) -> C25744
- R11: LCSC part number (none) -> C880273
- R12: LCSC part number (none) -> C25798
- R13, R14, R15, R17, R18, R23, R4, R40, R41, R43, R44: LCSC part number (none) -> C25744
- R16: value 10k -> 75k; LCSC part number (none) -> C25798
- R19: LCSC part number (none) -> C17557
- R20, R21: LCSC part number (none) -> C17714
- R22: LCSC part number (none) -> C17710
- R24, R25, R26: value 4.7k -> 10k; LCSC part number (none) -> C25744
- R34, R35, R36, R37, R38, R39, R5, R6: LCSC part number (none) -> C25117
- R7, R8: LCSC part number (none) -> C25905
- R9: footprint Resistor_SMD:R_0402_1005Metric -> Resistor_SMD:R_0603_1608Metric; LCSC part number (none) -> C22977
- SW1, SW2, SW3, SW4, SW5: LCSC part number (none) -> C84931
- SW6: LCSC part number (none) -> ???
- U1: LCSC part number (none) -> C107671
- U11: LCSC part number (none) -> C485517
- U3: LCSC part number (none) -> C841670
- U4: value MPR121QR2 -> MPR121, 0x5A; LCSC part number (none) -> C91322
- U5: footprint SamacSys_Parts:1043 -> Battery:BatteryHolder_Keystone_1042_1x18650; LCSC part number (none) -> -
- U7: LCSC part number (none) -> C404027
- U8: LCSC part number (none) -> C571211
Connections:
- net +3V3: now also R24.2, R25.2, R26.2, C2.1, IC3.1 (A0), IC3.16 (VDD), U6.20 (VDD); no longer IC4.5 (VDDIO), IC4.6 (VDD), R16.2, R43.2, R44.2
- net GND: now also R16.2, C1.2, C2.2, IC3.2 (A1), IC3.3 (A2), IC3.8 (VSS), J15.7 (GND7), J15.8 (GND8), J16.7 (GND7), J16.8 (GND8), J20.7 (GND7), J20.8 (GND8), J21.7 (GND7), J21.8 (GND8), U6.6 (VSS); no longer C30.2, IC4.17 (EP), IC4.7 (VSS), J14.1 (Pin_1)
- net I2C_SCL: now also R24.1, R25.1, IC3.14 (SCL), U6.2 (SCL); no longer IC4.15 (I2C_SCL), R16.1, R44.1
- net I2C_SDA: now also R23.1, R26.1, IC3.15 (SDA), U6.3 (SDA), U6.4 (ADDR); no longer IC4.14 (I2C_SDA), R15.1, R43.1
- net at SW4.2: now also IC1.6 (IO2)
- net at SW5.2: now also IC1.7 (IO3)
- net at SW3.2: now also IC1.5 (IO1)
- net at J8.4 (Pin_4): now also U6.10 (ELE2); no longer U4.10 (ELE2)
- net at J8.5 (Pin_5): now also U6.11 (ELE3); no longer U4.11 (ELE3)
- net at J8.6 (Pin_6): now also U6.12 (LED0/ELE4); no longer U4.12 (LED0/ELE4)
- net at J8.7 (Pin_7): now also U6.13 (LED1/ELE5); no longer U4.13 (LED1/ELE5)
- net at J8.8 (Pin_8): now also U6.14 (LED2/ELE6); no longer U4.14 (LED2/ELE6)
- net at J8.2 (Pin_2): now also U6.8 (ELE0); no longer U4.8 (ELE0)
- net at J8.3 (Pin_3): now also U6.9 (ELE1); no longer U4.9 (ELE1)
- net at SW2.2: now also IC1.4 (IO0)
- net at J13.3 (Pin_3): now also IC3.4 (IO0); no longer IC1.4 (IO0)
- net at J13.4 (Pin_4): now also IC3.5 (IO1); no longer IC1.5 (IO1)
- net at J13.5 (Pin_5): now also IC3.6 (IO2); no longer IC1.6 (IO2)
- net at J13.6 (Pin_6): now also IC3.7 (IO3); no longer IC1.7 (IO3)
- net at J13.7 (Pin_7): now also IC3.9 (IO4); no longer IC1.9 (IO4)
- net at J13.8 (Pin_8): now also IC3.10 (IO5); no longer IC1.10 (IO5)
- new net: J16.1 (ELE1), J9.1 (Pin_1)
- new net: J16.2 (ELE2), J9.2 (Pin_2)
- new net: J16.3 (ELE3), J9.3 (Pin_3)
- new net: J16.4 (ELE4), J9.4 (Pin_4)
- new net: J16.5 (ELE5), J9.5 (Pin_5)
- new net: J16.6 (ELE6), J9.6 (Pin_6)
- new net: R16.1, U6.7 (REXT)
- new net: R15.1, U6.1 (~{IRQ})
- new net: C1.1, U6.5 (VREG)
- new net: J19.1 (Pin_1), J21.1 (ELE1)
- new net: J19.2 (Pin_2), J21.2 (ELE2)
- new net: J19.3 (Pin_3), J21.3 (ELE3)
- new net: J19.4 (Pin_4), J21.4 (ELE4)
- new net: J19.5 (Pin_5), J21.5 (ELE5)
- new net: J19.6 (Pin_6), J21.6 (ELE6)
- new net: J15.1 (ELE1), J7.1 (Pin_1)
- new net: J15.2 (ELE2), J7.2 (Pin_2)
- new net: J15.3 (ELE3), J7.3 (Pin_3)
- new net: J15.4 (ELE4), J7.4 (Pin_4)
- new net: J15.5 (ELE5), J7.5 (Pin_5)
- new net: J15.6 (ELE6), J7.6 (Pin_6)
- new net: J20.3 (ELE3), U4.10 (ELE2)
- new net: J20.4 (ELE4), U4.11 (ELE3)
- new net: J20.5 (ELE5), U4.12 (LED0/ELE4)
- new net: J20.6 (ELE6), U4.13 (LED1/ELE5)
- new net: J20.1 (ELE1), U4.8 (ELE0)
- new net: J20.2 (ELE2), U4.9 (ELE1)
- new net: J6.1 (Pin_1), U2.1
- new net: J6.2 (Pin_2), U2.2
- new net: J6.3 (Pin_3), U2.3
- new net: J6.4 (Pin_4), U2.4
- new net: J6.5 (Pin_5), U2.5
- new net: J6.6 (Pin_6), U2.6
- new net capsenseSB_3v3: IC4.5 (VDDIO), IC4.6 (VDD), J4.3 (Pin_3), R43.2, R44.2
- new net capsenseSB_GND: C30.2, IC4.17 (EP), IC4.7 (VSS), J14.1 (Pin_1), J4.4 (Pin_4)
- new net capsenseSB_SCL: IC4.15 (I2C_SCL), J4.1 (Pin_1), R44.1
- new net capsenseSB_SDA: IC4.14 (I2C_SDA), J4.2 (Pin_2), R43.1
- no-connect marks 64 -> 57
Other:
- note added: "MPR121, 0x5A i2c built-in slider"
- note added: "MPR121, 0x5C i2c"
- note added: "PCA9554APW,118 0x38 built-in"
- note added: "PCA9554APW,118 0x39 ext"
- note removed: "MCP23017, 0x20 i2c"
- note removed: "MPR121, 0x5A i2c"
- note removed: "PCA9554APW,118 IO EXP 0x40 or 0x70 i2c"
- note removed: "QTouch, i2c 0x1C"
- moved on the sheet: C24, C25, C30, IC1, IC4, J14, R12, R13, R14, R17, R18, R4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
