File: CAD/clarinoid-devboard/clarinoid-devboard-01/clarinoid-devboard.kicad_pcb (KiCad board)
At the start: 2 copper layers, 162 x 230 mm, 134 parts, among them IC1 PCA9554APW,118, IC2 Injoinic IP5306 battery charge, IC3 PCA9554APW,118, IC4 CY8CMBR3108-LQXIT, J1 TRS jack, J10 MIDI IN, J11 MIDI OUT, J12 SSD1306, J13 conn_buttons_PCA9554, J14 touch_conn_capsense, J15 CapTouchSlider1, J16 CapTouchSlider2, J19 SB_slider4_header, J2 XKB_U262-16XN-4BVC11 USB-C re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, J20 CapTouchSlider3, J21 CapTouchSlider4, J3 Molex microSD 503398-1892, J4 capsense_subboard_header, J5 header_i2c, J6 SB_octaves_header, J7 SB_slider1_header, J8 touch_conn_mpr121, J9 SB_slider2_header, SW1 SW_Push, SW11 RotaryEncoder_Switch, SW2 SW_Push, SW3 SW_Push, SW4 SW_Push, SW5 SW_Push, SW6 SW_Push, U1 PCM5102A, U10 Pressure1_0x28_I2C0, U11 TLV75733PDBV, U12 ssd1306_graphic, U2 octave_keys_6, U3 APCI0136-P001A Teensy_4.0_Mic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, U4 MPR121, 0x5A, U5 Keystone 1043, U6 MPR121, 0x5C, U7 TLV75533PDBV, U8 6N138, U9 WS2812

Commit message: a bunch of PCB work. devboard-04 now in production.
Parts:
- removed J13: conn_buttons_PCA9554, Connector_PinSocket_2.54mm:PinSocket_1x08_P2.54mm_Vertical
- removed J15: CapTouchSlider1, CapTouchSliders:CaptouchSlider_Masked_x8_2pt_12x6x6x0.5mm
- removed J16: CapTouchSlider2, CapTouchSliders:CaptouchSlider_Masked_x8_2pt_12x6x6x1.0mm
- removed J19: SB_slider4_header, Connector_PinSocket_2.54mm:PinSocket_1x06_P2.54mm_Vertical
- removed J21: CapTouchSlider4, CapTouchSliders:CaptouchSlider_Masked_x8_2pt_12x6x6x2.0mm
- removed J7: SB_slider1_header, Connector_PinSocket_2.54mm:PinSocket_1x06_P2.54mm_Vertical
- removed J8: touch_conn_mpr121, Connector_PinSocket_2.54mm:PinSocket_1x08_P2.54mm_Vertical
- removed J9: SB_slider2_header, Connector_PinSocket_2.54mm:PinSocket_1x06_P2.54mm_Vertical
- removed R17, R18, R23, R24, R25, R26, R43, R44: 10k, Resistor_SMD:R_0402_1005Metric
- removed REF**: LHxv1, SamacSys_Parts:B3FS-1000P
- removed REF**: lh_h2, MountingHole:MountingHole_3.2mm_M3_Pad
- removed REF**: LHok, clarinoid2:MB2511S4W01-BC
- removed REF**: PCA9554APW,118, SamacSys_Parts:SOP65P640X110-16N
- removed REF**: LHx2, clarinoid2:MB2511S2G45
- removed REF**: LHxv2, SamacSys_Parts:B3FS-1000P
- removed REF**: LHI2CHdr, clarinoid2:solder point DIP 1x4
- removed REF**: LHx1, clarinoid2:MB2511S2G45
- removed REF**: LHx3, clarinoid2:MB2511S2G45
- removed REF**: LH-BREATHI2CHdr, clarinoid2:solder point DIP 1x4
- removed REF**: lh_h1, MountingHole:MountingHole_3.2mm_M3_Pad
- removed REF**: LHback, clarinoid2:MB2511S4W01-BC
- removed U6: MPR121, 0x5C, Package_DFN_QFN:UQFN-20_3x3mm_P0.4mm
- added BT1: Battery_Cell, Battery:BatteryHolder_Keystone_1042_1x18650, F.Cu at (161.3, 36.3)
- added D12: red, LED_SMD:LED_0402_1005Metric, F.Cu at (125.2, 113.4)
- added D13: red, LED_SMD:LED_0402_1005Metric, F.Cu at (122.7, 113.4)
- added D14: red, LED_SMD:LED_0402_1005Metric, F.Cu at (120.2, 113.4)
- added D15: red, LED_SMD:LED_0402_1005Metric, F.Cu at (117.7, 113.4)
- added D16: green, LED_SMD:LED_0402_1005Metric, F.Cu at (117.7, 114.9)
- added D17: green, LED_SMD:LED_0402_1005Metric, F.Cu at (122.7, 114.9)
- added D18: blue, LED_SMD:LED_0402_1005Metric, F.Cu at (122.7, 116.4)
- added D19: green, LED_SMD:LED_0402_1005Metric, F.Cu at (120.2, 114.9)
- added D20: green, LED_SMD:LED_0402_1005Metric, F.Cu at (125.2, 114.9)
- added D21: green, LED_SMD:LED_0402_1005Metric, F.Cu at (127.7, 114.9)
- added D22: blue, LED_SMD:LED_0402_1005Metric, F.Cu at (117.7, 116.4)
- added D23: blue, LED_SMD:LED_0402_1005Metric, F.Cu at (120.2, 116.4)
- added D24: blue, LED_SMD:LED_0402_1005Metric, F.Cu at (125.2, 116.4)
- added D25: red, LED_SMD:LED_0402_1005Metric, F.Cu at (127.7, 113.4)
- added D26: blue, LED_SMD:LED_0402_1005Metric, F.Cu at (127.7, 116.4)
- added D27: WS2812B, LED_SMD:LED_WS2812B_PLCC4_5.0x5.0mm_P3.2mm, F.Cu at (195.6, 114.4)
- added D28: WS2812B, LED_SMD:LED_WS2812B_PLCC4_5.0x5.0mm_P3.2mm, F.Cu at (195.6, 108.4)
- added D29: WS2812B, LED_SMD:LED_WS2812B_PLCC4_5.0x5.0mm_P3.2mm, F.Cu at (195.6, 102.4)
- added D30: WS2812B, LED_SMD:LED_WS2812B_PLCC4_5.0x5.0mm_P3.2mm, F.Cu at (195.6, 96.4)
- added D31: WS2812B, LED_SMD:LED_WS2812B_PLCC4_5.0x5.0mm_P3.2mm, F.Cu at (195.6, 90.4)
- added D32: WS2812B, LED_SMD:LED_WS2812B_PLCC4_5.0x5.0mm_P3.2mm, F.Cu at (195.6, 84.4)
- added D33: WS2812B, LED_SMD:LED_WS2812B_PLCC4_5.0x5.0mm_P3.2mm, F.Cu at (195.6, 78.4)
- added D34: WS2812B, LED_SMD:LED_WS2812B_PLCC4_5.0x5.0mm_P3.2mm, F.Cu at (195.6, 72.4)
- added D35: WS2812B, LED_SMD:LED_WS2812B_PLCC4_5.0x5.0mm_P3.2mm, F.Cu at (195.7, 66.5)
- added D36: WS2812B, LED_SMD:LED_WS2812B_PLCC4_5.0x5.0mm_P3.2mm, F.Cu at (195.7, 60.5)
- added DS1: Kingbright PDC54-Row1-pins01-09, Connector_PinSocket_2.54mm:PinSocket_1x09_P2.54mm_Vertical, F.Cu at (91.5, 115.9)
- added DS2: Kingbright PDC54-Row2-pins10-18, Connector_PinSocket_2.54mm:PinSocket_1x09_P2.54mm_Vertical, F.Cu at (91.5, 100.7)
- added G***: LOGO, LOGO, B.Cu at (209.0, 94.2)
- added H2: MountingHole, clarinoid2:Wurth Elektronik Reverse SMD Spacer M3, B.Cu at (186.2, 94.4)
- added H3: MountingHole, clarinoid2:Wurth Elektronik Reverse SMD Spacer M3, B.Cu at (117.7, 48.4)
- added H4: MountingHole, clarinoid2:Wurth Elektronik Reverse SMD Spacer M3, B.Cu at (109.7, 91.9)
- added H5: MountingHole, clarinoid2:Wurth Elektronik Reverse SMD Spacer M3, B.Cu at (185.2, 51.4)
- D10, D11: value LED -> red
- D5, D7: value LED -> blue
- D6: value 1N4148 -> 1N4148WS
- D8, D9: value LED -> green
- H1: footprint clarinoid2:Wurth_9774025151_M2.5_spacer_for_micromod -> clarinoid2:Sinhoo SMTSO2530CTJ
- IC3: value PCA9554APW,118 -> IS32FL3240-QWLA3-TR; footprint SamacSys_Parts:SOP65P640X110-16N -> SamacSys_Parts:QFN50P600X600X80-41N-D
- J1: value TRS jack -> AudioOut; footprint clarinoid2:Jack_3.5mm_CUI_SJ-3523-SMT_Horizontal -> clarinoid2:SWITCHCRAFT_35RAPC4BV4
- J10, J11: footprint clarinoid2:Jack_3.5mm_CUI_SJ-3523-SMT_Horizontal -> clarinoid2:SWITCHCRAFT_35RAPC4BV4
- J14: footprint Connector_PinSocket_2.54mm:PinSocket_1x08_P2.54mm_Vertical -> Connector_PinSocket_2.54mm:PinSocket_1x09_P2.54mm_Vertical
- J20: footprint CapTouchSliders:CaptouchSlider_Masked_x8_2pt_12x6x6x1.5mm -> CapTouchSliders:CaptouchSlider_Masked_H3x3_A1.0mm_x12
- J3: value Molex microSD 503398-1892 -> microSD SOFNG TF-15x15; footprint clarinoid2:MOLEX_503398-1892 -> clarinoid2:SOFNG TF-15x15 (LCSC C111196)
- J4: value capsense_subboard_header -> header_spi; footprint Connector_PinSocket_2.54mm:PinSocket_1x04_P2.54mm_Vertical -> Connector_PinSocket_2.54mm:PinSocket_1x07_P2.54mm_Vertical
- J6: value SB_octaves_header -> header_i2c1; footprint Connector_PinSocket_2.54mm:PinSocket_1x06_P2.54mm_Vertical -> Connector_PinSocket_2.54mm:PinSocket_1x04_P2.54mm_Vertical
- R13, R14, R40, R41: value 10k -> 4.7k
- R15: value 10k -> 4.7k; footprint Resistor_SMD:R_0402_1005Metric -> Resistor_THT:R_Axial_DIN0207_L6.3mm_D2.5mm_P7.62mm_Horizontal
- R16: value 75k -> 100k
- SW1: footprint SamacSys_Parts:B3F-4055 -> clarinoid2:XKB switch jlcpcb SW_TS-1187A-B-A-B
- SW6: footprint SamacSys_Parts:TL3305AF160QG -> clarinoid2:XKB switch jlcpcb SW_TS-1187A-B-A-B
- SW7: renamed from SW11; value RotaryEncoder_Switch -> RotaryEncoder_Switch_ABC12; footprint Rotary_Encoder:RotaryEncoder_Alps_EC11E-Switch_Vertical_H20mm -> clarinoid2:Bourns_ENC_PEC11R-4215F-S0024
- U2: value octave_keys_6 -> Micromod outline; footprint clarinoid2:CLARINOID_M6_6OCTAVES_offset -> clarinoid2:Teensy_4.0_MicroMod outline fab
- U3: footprint clarinoid2:Teensy_4.0_MicroMod_nospacer -> SamacSys_Parts:21992304
- U5: value Keystone 1043 -> Placeholder; footprint Battery:BatteryHolder_Keystone_1042_1x18650 -> clarinoid2:Kingbright PDC54 template
- moved C30 174.9 mm to (179.9, 71.6)
- moved J14 174.9 mm to (185.6, 78.4)
- moved IC4 174.9 mm to (178.8, 68.9)
- moved J4 156.9 mm to (207.7, 28.8)
- moved U2 128.9 mm to (142.7, 69.7), turned to 180 degrees
- moved J6 120.8 mm to (207.7, 54.9)
- moved J5 102.7 mm to (207.7, 50.9)
- moved U5 93.2 mm to (91.5, 115.9), turned to 90 degrees
- moved J12 75.0 mm to (160.8, 61.4)
- moved U12 75.0 mm to (154.4, 59.9)
- moved R15 70.1 mm to (122.0, 97.4), turned to 45 degrees
- moved SW2 69.4 mm to (154.7, 98.9)
- moved U9 67.8 mm to (197.3, 53.3)
- moved R16 67.3 mm to (127.0, 100.9), turned to 135 degrees
- moved C1 64.9 mm to (126.3, 101.8), turned to 135 degrees
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Connections:
- C1 pad 1: Net-(C1-Pad1) -> +3V3
- C30 pad 2: capsenseSB_GND -> GND
- IC3 pad 1: +3V3 -> Net-(IC3-Pad1)
- IC3 pad 11: unconnected-(IC3-Pad11) -> Net-(IC3-Pad11)
- IC3 pad 12: unconnected-(IC3-Pad12) -> Net-(IC3-Pad12)
- IC3 pad 13: unconnected-(IC3-Pad13) -> Net-(IC3-Pad13)
- IC3 pad 14: I2C_SCL -> Net-(IC3-Pad14)
- IC3 pad 15: I2C_SDA -> GND
- IC3 pad 16: +3V3 -> GND
- IC3 pad 2: GND -> Net-(IC3-Pad2)
- IC3 pad 3: GND -> Net-(IC3-Pad3)
- IC3 pad 8: GND -> Net-(IC3-Pad8)
- IC4 pad 10: unconnected-(IC4-Pad10) -> Net-(IC4-Pad10)
- IC4 pad 14: capsenseSB_SDA -> I2C_SDA
- IC4 pad 15: capsenseSB_SCL -> I2C_SCL
- IC4 pad 17: capsenseSB_GND -> GND
- IC4 pad 5: capsenseSB_3v3 -> +3V3
- IC4 pad 6: capsenseSB_3v3 -> +3V3
- IC4 pad 7: capsenseSB_GND -> GND
- J1 pad 2: Net-(C12-Pad1) -> Net-(C9-Pad1)
- J1 pad 3: Net-(C9-Pad1) -> unconnected-(J1-Pad3)
- J10 pad 1: Net-(J10-Pad1) -> unconnected-(J10-Pad1)
- J10 pad 2: unconnected-(J10-Pad2) -> Net-(D6-Pad2)
- J10 pad 3: Net-(D6-Pad2) -> unconnected-(J10-Pad3)
- J11 pad 1: Net-(J11-Pad1) -> GND
- J11 pad 2: GND -> Net-(J11-Pad2)
- J11 pad 3: Net-(J11-Pad3) -> unconnected-(J11-Pad3)
- J14 pad 1: capsenseSB_GND -> GND
- J14 pad 8: Net-(IC4-Pad11) -> Net-(IC4-Pad10)
- J20 pad 1: Net-(U4-Pad8) -> GND
- J20 pad 2: Net-(U4-Pad9) -> Net-(J20-Pad2)
- J20 pad 3: Net-(U4-Pad10) -> Net-(J20-Pad3)
- J20 pad 4: Net-(U4-Pad11) -> Net-(J20-Pad4)
- J20 pad 5: Net-(U4-Pad12) -> Net-(J20-Pad5)
- J20 pad 6: Net-(U4-Pad13) -> Net-(J20-Pad6)
- J20 pad 7: GND -> Net-(J20-Pad7)
- J20 pad 8: GND -> Net-(J20-Pad8)
- J4 pad 1: capsenseSB_SCL -> GND
- J4 pad 2: capsenseSB_SDA -> +3V3
- J4 pad 3: capsenseSB_3v3 -> SPI0_MISO
- J4 pad 4: capsenseSB_GND -> SPI0_MOSI
- J6 pad 1: Net-(J6-Pad1) -> GND
- J6 pad 2: Net-(J6-Pad2) -> +3V3
- J6 pad 3: Net-(J6-Pad3) -> I2C1_SDA
- J6 pad 4: Net-(J6-Pad4) -> I2C1_SCL
- R13 pad 1: I2C_SDA -> I2C1_SDA
- R14 pad 1: I2C_SCL -> I2C1_SCL
- R15 pad 1: Net-(R15-Pad1) -> GND
- R15 pad 2: +3V3 -> Net-(IC3-Pad37)
- R16 pad 1: Net-(R16-Pad1) -> enable_led_driver
- R19 pad 1: Net-(J10-Pad1) -> Net-(J10-Pad4)
- R20 pad 1: Net-(J11-Pad1) -> Net-(J11-Pad4)
- R21 pad 1: Net-(J11-Pad3) -> Net-(J11-Pad2)
- R40 pad 1: I2C_SCL -> I2C_SDA
- R41 pad 1: I2C_SDA -> I2C_SCL
- SW7 pad S1: ENC_SWITCH -> (no net)
- SW7 pad S2: GND -> (no net)
- U3 pad 51: unconnected-(U3-Pad51) -> I2C1_SDA
- U3 pad 53: unconnected-(U3-Pad53) -> I2C1_SCL
- U3 pad 61: unconnected-(U3-Pad61) -> SPI0_MISO
- U3 pad 63: unconnected-(U3-Pad63) -> kingbright_dig1
- U3 pad 65: unconnected-(U3-Pad65) -> kingbright_dig0
- U3 pad 67: unconnected-(U3-Pad67) -> SPI0_generic1_cs
- U3 pad 73: unconnected-(U3-Pad73) -> SPI0_generic0_cs
- U3 pad 8: unconnected-(U3-Pad8) -> enable_led_driver
- U4 pad 10: Net-(U4-Pad10) -> Net-(J20-Pad4)
- U4 pad 11: Net-(U4-Pad11) -> Net-(J20-Pad5)
- U4 pad 12: Net-(U4-Pad12) -> Net-(J20-Pad6)
- U4 pad 13: Net-(U4-Pad13) -> Net-(J20-Pad7)
- U4 pad 14: unconnected-(U4-Pad14) -> Net-(J20-Pad8)
- U4 pad 15: unconnected-(U4-Pad15) -> Net-(J20-Pad9)
- U4 pad 16: unconnected-(U4-Pad16) -> Net-(J20-Pad10)
- U4 pad 17: unconnected-(U4-Pad17) -> Net-(J20-Pad11)
- U4 pad 8: Net-(U4-Pad8) -> Net-(J20-Pad2)
- U4 pad 9: Net-(U4-Pad9) -> Net-(J20-Pad3)
- U9 pad 2: WS2812_DATA -> WS2812_DATA2
Routing:
- net +3V3: track 6.83 -> 444.9 mm, vias 0 -> 13
- net I2C_SCL: track 8.24 -> 211.2 mm, vias 0 -> 6
- net GND: track 58.1 -> 251.9 mm, vias 2 -> 33
- net I2C_SDA: track 12.5 -> 203.2 mm, vias 0 -> 7
- net WS2812_DATA: track 0.00 -> 95.0 mm, vias 0 -> 2
- net SPI0_SCK: track 0.00 -> 93.4 mm, vias 0 -> 4
- net SPI0_MISO: track 0.00 -> 92.8 mm, vias 0 -> 2
- net SPI0_generic0_cs: track 0.00 -> 90.2 mm, vias 0 -> 2
- net SPI0_generic1_cs: track 0.00 -> 90.2 mm, vias 0 -> 2
- net SPI0_MOSI: track 0.00 -> 87.0 mm, vias 0 -> 4
- net USB data in -: track 0.00 -> 84.2 mm, vias 0 -> 2
- net USB data in +: track 0.00 -> 82.9 mm, vias 0 -> 2
- net I2C1_SCL: track 0.00 -> 81.4 mm, vias 0 -> 2
- net I2C1_SDA: track 0.00 -> 78.4 mm, vias 0 -> 2
- net kingbright_dig0: track 0.00 -> 75.2 mm, vias 0 -> 1
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- added copper zone on B.Cu, net GND
- added copper zone on F.Cu, net GND
- removed copper zone on B.Cu, net capsenseSB_GND
- removed copper zone on F.Cu, net capsenseSB_GND
Other:
- board size 162 x 230 mm -> 131.5 x 95 mm
- board text added: "CS1 CS0 CLK SI SO 3v3 GND"
- board text added: "G 3v CK DT RS DC CS"
- board text added: "GND 3v3 SDA SCK"
- board text added: "I2C0"
- board text added: "I2C1"
- board text added: "SPI0"
- board text added: "SSD1306"
- board text added: "WS2812b 3v DT G"
- board text added: "clarinoid test device rev 1"
- board text removed: "I2C -scl -sda -3v3 -gnd"
- board text removed: "WS2812b +3v Data GND"
- board text removed: "small (4deg) rotation is possible and gives space between top keys"
