File: CAD/clarinoid3-micromod/clarinoid3.kicad_pcb (KiCad board)
At the start: 2 copper layers, 519 x 63.5 mm, 53 parts, among them IC1 PCA9554APW,118, IC2 PCA9554APW,118, J1 LEDHdr, J10 pitch_pitchhdr, J12 RHI2CHdr, J13 RHencHdr, J16 LHI2CHdr, J18 MIDIin, J19 Molex microSD 503398-1892, J2 OLEDHdr, J20 LH-BREATHI2CHdr, J3 StereoPot_SW, J4 MIDIOut, J5 AudioOut, J7 BREATHI2CHdr, J8 USB_B_Micro, J9 RH_PitchHdr, SW10 LHx1, SW11 LHx2, SW12 LHback, SW13 LHx3, SW14 LHok, SW15 RHx4, SW3 RHx1, SW5 RHx2, SW6 RHx3, SW9 Rotary_Encoder_Switch, U1 Teensy_4.0_MicroMod, U2 AdafruitMPR121, U3 AdafruitMPR121, U5 MH-CD42, U6 PCM5102, U7 HoneywellABPMAND001PG2A3, U8 CLARINOID_OCTAVES

Commit message: incremental progress of clarinoid test device renaming midi performer to prepare for rev2
Parts:
- added REF**: CaptouchSlider_Masked_x8_2pt_12x6x6x1.5mm, CapTouchSliders:CaptouchSlider_Masked_x8_2pt_12x6x6x1.5mm, F.Cu at (152.4, -85.7)
- U8: value CLARINOID_OCTAVES -> octave_keys
- moved U5 129.7 mm to (467.5, -60.3)
- moved J3 97.9 mm to (380.9, -121.7)
- moved U6 81.5 mm to (378.9, -43.2)
- moved U2 70.4 mm to (420.1, -46.6)
- moved J5 68.2 mm to (325.9, -127.5)
- moved U1 58.1 mm to (287.3, -120.4)
- moved H8 58.1 mm to (269.8, -121.7)
- moved S6 53.7 mm to (418.4, -135.2)
- moved R1 23.0 mm to (348.2, -128.2)
- moved J4 23.0 mm to (354.4, -125.2)
- moved R2 23.0 mm to (348.2, -122.2)
- moved J18 21.5 mm to (340.9, -126.7)
- moved H10 7.02 mm to (142.9, -108.7)
- moved H9 7.02 mm to (245.9, -108.7)
- moved J10 7.02 mm to (235.4, -100.2)
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Connections:
- U3 pad 10: Net-(U3-Pad10) -> unconnected-(U3-Pad10)
- U8 pad 1: Net-(U3-Pad10) -> Net-(U3-Pad9)
- U8 pad 2: Net-(U3-Pad9) -> Net-(U3-Pad8)
- U8 pad 3: Net-(U3-Pad8) -> Net-(U3-Pad7)
- U8 pad 4: Net-(U3-Pad7) -> Net-(U3-Pad6)
- U8 pad 5: Net-(U3-Pad6) -> Net-(U3-Pad5)
- U8 pad 6: Net-(U3-Pad5) -> Net-(U3-Pad4)
Other:
- board size 519 x 63.5 mm -> 519 x 63 mm
- board text added: "pitch midpoint @ 1/3 between keys 1&2"
