File: CAD/clarinoid3-bodytest/00/clarinoid-devboard-04/clarinoid-bodytest.kicad_pcb (KiCad board)
At the start: 2 copper layers, 489 x 343 mm, 225 parts, among them IC1 PCA9554APW,118, IC2 Injoinic IP5306 battery charge, IC3 PCA9554APW,118, J1 Switchcraft 35RAPC4BV4, J1 header i2c pressure, J10 MIDI IN, J10 header i2c lh to main, J11 MIDI OUT, J11 microSD SOFNG TF-15x15, J12 I2C HEADER main to LH, J13 ENC_HEADER main to lh, J14 header_i2c_lh to pressure, J15 StereoPot_SW_CommonAudioGND, J16 AudioOut, J17 lh_enc_header, J18 header lh_keys, J19 header_ws2812 main to LH, J2 lh_header_i2c_main, J20 header_ws2812 LH from main, J3 MIDI IN, J4 MIDI OUT, J5 XKB_U262-16XN-4BVC11 USB-C re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, J6 RH touch keys header, J7 I2C HEADER main to PITCH, J8 CapTouchSlider3, J9 OLED_HEADER, SW1 SW_Push, SW8 RotaryEncoder_Switch_ABC12, U1 PCM5102A, U1 Pressure1_0x28_I2C0, U10 MPR121, 0x5A, U11 MPR121, 0x5A, U11 TLV75733PDBV, U12 octave_keys_6, U13 stereo pot w switch sub-board, U14 stereo pot subboard template, U2 APCI0108-P001A Teensy_4.0_Mic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, U3 APCI0136-P001A Teensy_4.0_Mic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, U3 Micromod outline, U4 MPR121, 0x5A, U4 PCM5102A, U5 TLV75533PDBV, U6 6N138, U7 TLV75533PDBV, U7 TLV75733PDBV, U8 6N138, U8 MPR121, 0x5A, U9 WS2812_HEADER LH to external

Commit message: adding a hardware layout sketch to the midi performer device PCB progress on the clarinoid3 body
Parts:
- removed ?: , clipboard:9196e359-7150-4967-9b24-df29c59429f9
- removed the BT1 at (-94.0, 86.4)
- removed D18, D19, D20, D21, D22, D23, D24: WS2812B, LED_SMD:LED_WS2812B_PLCC4_5.0x5.0mm_P3.2mm
- removed J13: ENC_HEADER main to lh, Connector_PinHeader_2.00mm:PinHeader_1x03_P2.00mm_Vertical
- removed J17: lh_enc_header, Connector_PinHeader_2.00mm:PinHeader_1x03_P2.00mm_Vertical
- removed J19: header_ws2812 main to LH, Connector_PinHeader_2.00mm:PinHeader_1x01_P2.00mm_Vertical
- removed J20: header_ws2812 LH from main, Connector_PinHeader_2.00mm:PinHeader_1x01_P2.00mm_Vertical
- removed SW8: RotaryEncoder_Switch_ABC12, clarinoid2:Bourns_ENC_PEC11R-4215F-S0024
- removed the U3 at (-147.4, 83.7)
- added J21: encoder header, Connector_PinHeader_2.54mm:PinHeader_1x05_P2.54mm_Vertical, F.Cu at (-492.0, 226.1)
- added SW10: SW_x1, clarinoid2:MB2511S2G45, F.Cu at (-437.6, 225.8)
- added SW11: SW_x2, clarinoid2:MB2511S2G45, F.Cu at (-464.2, 225.8)
- added SW12: SW_x3, clarinoid2:MB2511S2G45, F.Cu at (-479.0, 225.8)
- added SW2: sw_RHx1, clarinoid2:MB2511S2G45, F.Cu at (-291.4, 226.6)
- added SW3: sw_RHx2, clarinoid2:MB2511S2G45, F.Cu at (-275.4, 223.8)
- added SW4: sw_RHx3, clarinoid2:MB2511S2G45, F.Cu at (-245.4, 223.8)
- added SW5: sw_RHx4, clarinoid2:MB2511S2G45, F.Cu at (-229.4, 226.6)
- added SW7: SW_OK, clarinoid2:solder point DIP 1x2, F.Cu at (-457.5, 235.5)
- added SW9: SW_BACK, clarinoid2:solder point DIP 1x2, F.Cu at (-431.0, 235.4)
- added U15: OK cutout, clarinoid2:MB2511S4W01-BC, F.Cu at (-450.9, 230.7)
- added U16: BACK cutout, clarinoid2:MB2511S4W01-BC, F.Cu at (-424.3, 230.7)
- added U17: OLED graphic, clarinoid2:SSD1306_128x64_approximate, F.Cu at (-471.9, 284.3)
- added U18: encoder cutout, clarinoid2:Bourns_ENC_PEC11R-4215F-S0024 panel cutout shaft downward, F.Cu at (-504.0, 228.2)
- H10, H11, H2, H3, H4, H5, H6, H7, H8, H9: footprint clarinoid2:Wurth Elektronik Reverse SMD Spacer M3 -> MountingHole:MountingHole_2.7mm_M2.5
- J1, J14, J18, J2, J6, J7: footprint Connector_PinHeader_2.00mm:PinHeader_1x04_P2.00mm_Vertical -> Connector_PinHeader_2.54mm:PinHeader_1x04_P2.54mm_Vertical
- J10: value header i2c lh to main -> LH header multi to main; footprint Connector_PinHeader_2.00mm:PinHeader_1x04_P2.00mm_Vertical -> Connector_PinHeader_2.54mm:PinHeader_1x07_P2.54mm_Vertical
- J12: value I2C HEADER main to LH -> main header multi to LH; footprint Connector_PinHeader_2.00mm:PinHeader_1x04_P2.00mm_Vertical -> Connector_PinHeader_2.54mm:PinHeader_1x07_P2.54mm_Vertical
- J16, J3, J4, J8: moved to B.Cu
- J9: footprint Connector_PinHeader_2.00mm:PinHeader_1x07_P2.00mm_Vertical -> Connector_PinHeader_2.54mm:PinHeader_1x07_P2.54mm_Vertical
- U12: footprint clarinoid2:CLARINOID_M6_6OCTAVES_p13.25_offset1.0mm_copy -> clarinoid2:CLARINOID_M6_6OCTAVES_p13.3_offset1.0mm; moved to B.Cu
- U9: footprint Connector_PinHeader_2.00mm:PinHeader_1x03_P2.00mm_Vertical -> Connector_PinHeader_2.54mm:PinHeader_1x03_P2.54mm_Vertical
- moved J9 287.5 mm to (-183.6, 218.2)
- moved D25 284.6 mm to (-486.1, 223.4)
- moved U13 267.0 mm to (-417.1, 267.6)
- moved U14 267.0 mm to (-414.6, 272.6)
- moved J7 260.9 mm to (-210.1, 218.2)
- moved J12 254.7 mm to (-222.6, 218.2)
- moved H11 228.6 mm to (-416.4, 231.2)
- moved H4 227.7 mm to (-283.3, 231.2)
- moved H9 227.5 mm to (-471.6, 231.2)
- moved R35 218.4 mm to (-402.8, 225.5), turned to -90 degrees
- moved H2 212.8 mm to (-289.6, 267.2)
- moved D17 208.6 mm to (-415.6, 223.4)
- moved J14 200.2 mm to (-485.3, 228.7)
- moved J18 193.9 mm to (-383.7, 222.3)
- moved J10 193.2 mm to (-388.7, 222.1)
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Connections:
- D15 pad 2: Net-(D15-Pad2) -> /MainBoard/ws2812 data out to LH
- D16 pad 4: Net-(D16-Pad4) -> /LHBoard/ws2812 data from main
- D17 pad 2: Net-(D17-Pad2) -> Net-(D25-Pad4)
- D25 pad 4: Net-(D24-Pad2) -> Net-(D25-Pad4)
- IC3 pad 12: Net-(IC3-Pad12) -> /LHBoard/encoder SW
- U12 pad 1: Net-(U10-Pad12) -> Net-(U10-Pad17)
- U12 pad 2: Net-(U10-Pad13) -> Net-(U10-Pad16)
- U12 pad 3: Net-(U10-Pad14) -> Net-(U10-Pad15)
- U12 pad 4: Net-(U10-Pad15) -> Net-(U10-Pad14)
- U12 pad 5: Net-(U10-Pad16) -> Net-(U10-Pad13)
- U12 pad 6: Net-(U10-Pad17) -> Net-(U10-Pad12)
- U2 pad 44: /MainBoard/ENC_SW -> unconnected-(U2-Pad44)
Routing:
- net Net-(U10-Pad12): track 0.00 -> 103.3 mm
- net Net-(U10-Pad13): track 0.00 -> 90.3 mm
- net Net-(U10-Pad14): track 0.00 -> 75.5 mm
- net Net-(U10-Pad15): track 0.00 -> 61.2 mm
- net Net-(J8-Pad2): track 0.00 -> 53.6 mm, vias 0 -> 1
- net Net-(D16-Pad2): track 0.00 -> 51.3 mm
- net Net-(J8-Pad3): track 0.00 -> 48.8 mm, vias 0 -> 1
- net Net-(U10-Pad16): track 0.00 -> 46.8 mm
- net Net-(J8-Pad4): track 0.00 -> 43.2 mm, vias 0 -> 1
- net Net-(J18-Pad4): track 0.00 -> 42.0 mm, vias 0 -> 1
- net Net-(J8-Pad5): track 0.00 -> 38.3 mm, vias 0 -> 1
- net /LHBoard/lh_sck: track 0.00 -> 37.3 mm, vias 0 -> 1
- net /LHBoard/lh_sda: track 0.00 -> 35.9 mm
- net Net-(J18-Pad3): track 0.00 -> 35.4 mm, vias 0 -> 1
- net /PressureBoard/pressure_sda: track 0.00 -> 35.4 mm
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Other:
- board size 489 x 343 mm -> 467.9 x 96.5 mm
- board text added: "1"
- board text added: "11mm from bottom to switch panel edge"
- board text added: "2"
- board text added: "3"
- board text added: "4"
- board text added: "4mm longer for octaves"
- board text added: "A"
- board text added: "B"
- board text added: "C"
- board text added: "ENCA"
- board text added: "ENCB"
- board text added: "GND"
- board text added: "I2C to Pr."
- board text added: "LED"
- board text added: "LED EXT"
- board text added: "M6 hole center 4.5mm from bottom"
- board text added: "S1"
- board text added: "S2"
- board text added: "SCK"
- board text added: "SDA"
- board text added: "TODO: - add silkscreen markings for screw positions - add markings for key placements - account for no bottom assembly - add port holes for internal led"
- board text added: "To Main"
- board text added: "enc."
- board text added: "keys"
- board text added: "logo"
- board text added: "no component zone"
- board text added: "pipe"
- board text added: "pitch screw"
- board text added: "~6.6mm from switch panel edge to hole center"
- board text removed: "TODO: add silkscreen markings for screw positions"
