File: CAD/clarinoid3-bodytest/02/MIDI.kicad_sch (KiCad schematic)
At the start: 9 parts, among them J3 MIDI IN, J4 MIDI OUT, U6 6N138

Commit message: created clarinoid presets for Cave Bouncer more clarinoid3 pcb WIP midi performer application WIP; transitioning to Teensy4
Parts:
- J3, J4: footprint clarinoid2:SWITCHCRAFT_35RAPC4BV4 -> clarinoid2:SWITCHCRAFT_35RAPC4BV4_OvalHoles
Changed lines of the file:
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@@
     (property "Reference" "J3" (id 0) (at 73.914 75.565 0))
     (property "Value" "MIDI IN" (id 1) (at 71.374 86.995 0))
-    (property "Footprint" "clarinoid2:SWITCHCRAFT_35RAPC4BV4" (id 2) (at 75.819 83.185 0)
+    (property "Footprint" "clarinoid2:SWITCHCRAFT_35RAPC4BV4_OvalHoles" (id 2) (at 75.819 83.185 0)
       (effects (font (size 1.27 1.27)) (justify left bottom) hide)
     )
@@
     (property "Reference" "J4" (id 0) (at 185.039 73.66 0))
     (property "Value" "MIDI OUT" (id 1) (at 185.039 76.2 0))
-    (property "Footprint" "clarinoid2:SWITCHCRAFT_35RAPC4BV4" (id 2) (at 181.864 92.075 0)
+    (property "Footprint" "clarinoid2:SWITCHCRAFT_35RAPC4BV4_OvalHoles" (id 2) (at 181.864 92.075 0)
       (effects (font (size 1.27 1.27)) (justify left bottom) hide)
     )
