File: CAD/clarinoid3-bodytest/02/MainBoard.kicad_sch (KiCad schematic)
At the start: 15 parts, among them J12 main header multi to LH, J16 AudioOut, J19 clarinoid3 DAC and POT subboa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, J7 I2C HEADER main to PITCH, J9 OLED_HEADER, U2 APCI0108-P001A Teensy_4.0_Mic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, U3 Micromod outline

Commit message: created clarinoid presets for Cave Bouncer more clarinoid3 pcb WIP midi performer application WIP; transitioning to Teensy4
Parts:
- J16: footprint clarinoid2:SWITCHCRAFT_35RAPC4BV4 -> clarinoid2:SWITCHCRAFT_35RAPC4BV4_OvalHoles
Connections:
- net audio_gnd: now reaches J16.1 (S-GND), J19.10 (audio_out_S_gnd)
Changed lines of the file:
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@@
+    (effects (font (size 1.27 1.27)) (justify right bottom))
+  )
+  (label "audio_gnd" (at 222.758 156.21 180)
     (effects (font (size 1.27 1.27)) (justify right bottom))
   )
@@
       (effects (font (size 1.27 1.27)) (justify right))
     )
-    (property "Footprint" "clarinoid2:SWITCHCRAFT_35RAPC4BV4" (id 2) (at 250.698 147.828 0)
+    (property "Footprint" "clarinoid2:SWITCHCRAFT_35RAPC4BV4_OvalHoles" (id 2) (at 250.698 147.828 0)
       (effects (font (size 1.27 1.27)) (justify left bottom) hide)
     )
