File: CAD/clarinoid3-bodytest/03/clarinoid-bodytest.kicad_pcb (KiCad board)
At the start: 2 copper layers, 467.9 x 112.2 mm, 130 parts, among them IC1 PCA9554APW,118, IC2 Injoinic IP5306 battery charge, IC3 PCA9554APW,118, J1 header i2c pressure, J10 LH header multi to main, J11 microSD SOFNG TF-15x15, J12 main header multi to LH, J13 clarinoid3 main usb interconn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, J14 header_i2c_lh to pressure, J15 clarinoid3 DAC and POT subboa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, J16 AudioOut, J17 clarinoid3 main usb interconn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, J18 header lh_keys, J19 clarinoid3 DAC and POT subboa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, J2 lh_header_i2c_main, J21 encoder header, J3 MIDI IN, J4 MIDI OUT, J5 XKB_U262-16XN-4BVC11 USB-C re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, J6 RH touch keys header, J7 I2C HEADER main to PITCH, J8 CapTouchSlider3, J9 OLED_HEADER, SW1 sw_batteryindicator, SW10 SW_x1, SW11 SW_x2, SW12 SW_x3, SW13 SW_y1, SW14 SW_y2, SW2 sw_RHx1, SW3 sw_RHx2, SW4 sw_RHx3, SW5 sw_RHx4, SW6 sw_program, SW7 SW_OK, SW9 SW_BACK, U1 Pressure1_0x28_I2C0, U10 MPR121, 0x5A, U11 MPR121, 0x5A, U12 octave_keys_6, U15 OK cutout, U16 BACK cutout, U17 OLED graphic, U18 encoder cutout, U2 APCI0108-P001A Teensy_4.0_Mic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, U3 Micromod outline, U4 PCM5102A, U5 TLV75533PDBV, U6 6N138, U7 TLV75733PDBV, U8 MPR121, 0x5A, U9 WS2812_HEADER LH to external

Commit message: pcb incremental
Parts:
- moved J14 97.7 mm to (-383.8, 226.9), turned to 0 degrees
- moved U9 79.1 mm to (-391.8, 225.3), turned to 0 degrees
- moved J12 61.0 mm to (-229.3, 232.7)
- moved C2 58.0 mm to (-460.4, 222.5), turned to 90 degrees
- moved R36 57.1 mm to (-461.4, 224.5), turned to 90 degrees
- moved R35 54.5 mm to (-457.2, 222.8), turned to 0 degrees
- moved U10 53.2 mm to (-458.8, 225.7), turned to -90 degrees
- moved C29 52.7 mm to (-455.7, 223.2), turned to 90 degrees
- moved SW14 46.4 mm to (-374.8, 238.9)
- moved IC3 39.7 mm to (-443.3, 225.2), turned to -90 degrees
- moved SW7 35.7 mm to (-424.3, 222.2), turned to 0 degrees
- moved SW13 34.5 mm to (-416.8, 238.2), turned to -90 degrees
- moved R17 33.9 mm to (-254.7, 232.3)
- moved R18 33.9 mm to (-254.7, 231.2)
- moved IC1 33.9 mm to (-249.5, 230.1)
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Routing:
- net /LHBoard/lh_3v3: track 287.0 -> 3.49 mm, vias 7 -> 0
- net /LHBoard/encoder A: track 157.1 -> 0.00 mm
- net /LHBoard/encoder B: track 113.7 -> 0.00 mm, vias 2 -> 0
- net /MainBoard/ws2812 data out to LH: track 107.2 -> 0.00 mm
- net /LHBoard/lh_sck: track 104.7 -> 0.00 mm, vias 2 -> 0
- net /MainBoard/i2c0_sda: track 128.4 -> 23.8 mm, vias 4 -> 2
- net /LHBoard/encoder SW: track 99.6 -> 0.00 mm, vias 2 -> 0
- net /MainBoard/i2c0_scl: track 117.2 -> 22.2 mm, vias 6 -> 2
- net Net-(IC3-Pad9): track 86.5 -> 0.00 mm, vias 2 -> 0
- net Net-(D17-Pad2): track 71.1 -> 0.00 mm
- net Net-(U10-Pad12): track 103.4 -> 46.2 mm
- net Net-(U10-Pad13): track 90.4 -> 33.8 mm
- net Net-(U10-Pad14): track 75.6 -> 22.1 mm
- net Net-(D16-Pad2): track 51.3 -> 0.00 mm
- net Net-(IC3-Pad4): track 71.9 -> 22.9 mm, vias 2 -> 0
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Other:
- board text added: "DAT"
- board text added: "TODO: - find PCB-mount through hole switches for reset (high actuation force) - check clearance of molex vertical keyed SMT header - headers which are to be hand-soldered with wire = use short pins (encoder to board for exmple). this has low clearance to avoid hitting the rivet - headers board-to-board will use molex SL keyed connectors to eliminate polarity confusion."
- board text removed: "FX enable"
- board text removed: "logo"
