File: CAD/clarinoid-devboard/clarinoid-devboard-05/clarinoid-devboard.kicad_sch (KiCad schematic)
At the start: 152 parts, among them IC1 PCA9554APW,118, IC2 Injoinic IP5306 battery charge, J1 AudioOut, J10 MIDI IN, J11 MIDI OUT, J12 SSD1306, J13 captouch 3x3x1 header B, J14 captouch4x4x2 headerA, J15 captouch4x4x2 header B, J16 captouch4x4x2, J17 captouch4x4x3 headerA, J18 captouch4x4x3 header B, J19 captouch4x4x.5 headerA, J2 XKB_U262-16XN-4BVC11 USB-C re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, J20 CapTouchSlider_3x3x1, J21 captouch4x4x.5 header B, J22 captouch4x4x3, J23 captouch4x4x.5, J24 captouch5x5x1 headerA, J25 captouch5x5x1 header B, J26 captouch4x4x1 headerA, J27 captouch4x4x1 header B, J28 captouch5x5x1, J29 captouch4x4x1, J3 header_usbfromteensy, J30 microSD SOFNG TF-15x15, J4 header_spi, J5 header_i2c, J6 Conn_01x06, J7 header_power tap, J8 Conn_01x06, J9 captouch 3x3x1 headerA, SW1 SW_Push, SW10 DIP red power source, SW2 SW_Push, SW3 SW_Push, SW4 SW_Push, SW5 SW_Push, SW6 SW_Push, SW7 RotaryEncoder_Switch_ABC12, SW8 DIP red power source, SW9 DIP red power source, U1 PCM5102A, U10 captouch4x4x2 graphic, U11 captouch4x4x3 graphic, U12 ssd1306_graphic, U13 captouch4x4x.5 graphic, U14 captouch5x5x1 graphic, U15 captouch4x4x1 graphic, U16 APCI0108-P001A Teensy_4.0_Mic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, U17 TLV75733PDBV, U18 Micromod outline, U19 TLV75733PDBV, U2 Teensy4.1_LEFT, U3 Teensy4.1_RIGHT, U4 MPR121, 0x5A, U5 main captouch graphic, U6 Placeholder, U7 TLV75533PDBV, U8 6N138, U9 captouch3x3x1 graphic

Commit message: devboard rev 2 i think is ready for assembly
Parts:
- removed D12, D13, D14, D15: WS2812B, LED_SMD:LED_WS2812B_PLCC4_5.0x5.0mm_P3.2mm, symbol LED:WS2812B
- added C33: 0.1uF, Capacitor_SMD:C_0805_2012Metric, symbol Device:C
- added H5: MountingHole, MountingHole:MountingHole_3.2mm_M3_Pad_Via, symbol Mechanical:MountingHole_Pad
- added IC3: CY8CMBR3108-LQXIT, SamacSys_Parts:QFN50P300X300X60-17N-D, symbol SamacSys_Parts:CY8CMBR3108-LQXIT
- added NT2: I2S tee_LRCK, NetTie:NetTie-3_SMD_Pad0.5mm, symbol Device:NetTie_3_Tee
- added NT3: I2S tee_DIN, NetTie:NetTie-3_SMD_Pad0.5mm, symbol Device:NetTie_3_Tee
- added NT4: I2S tee_BCK, NetTie:NetTie-3_SMD_Pad0.5mm, symbol Device:NetTie_3_Tee
- added U20, U21, U22, U23, U24, U25, U26, U27, U28, U29, U30, U31, U32, U33, U34, U35, U36, U37: mb1, clarinoid2:mouse-bite-2mm-slot, symbol clarinoid2:Placeholder
- added U38: WS2812, Connector_PinSocket_2.54mm:PinSocket_1x03_P2.54mm_Vertical, symbol clarinoid2:WS2812
- BT1, J1, J10, J11, J16, J20, J22, J23, J28, J29, NT1, SW7, U12, U18: LCSC part number - -> (none)
- C1, C10, C11, C15, C16, C3, C5: LCSC (none) -> C15850; LCSC part number C15525 -> C15850
- C12, C7, C8, C9: LCSC (none) -> C49217; LCSC part number C12530 -> C49217
- C13, C14, C23, C24, C25, C27, C28, C4, C6: LCSC (none) -> C49678; LCSC part number C1525 -> C49678
- C17, C18, C19, C20, C21, C22: LCSC (none) -> C602037; LCSC part number C59461 -> C602037
- C2, C30: LCSC (none) -> C5378; LCSC part number C21120 -> C5378
- C26, C31: LCSC (none) -> C49678; LCSC part number C14663 -> C49678
- C29, C32: LCSC (none) -> C28323; LCSC part number C14663 -> C28323
- D1, D2, D3, D4: LCSC (none) -> C264424
- D10, D11: LCSC (none) -> C72044
- D16: LCSC (none) -> C393436; LCSC part number (none) -> C393436; verif (none) -> 1
- D5, D7: LCSC (none) -> C72041
- D6: LCSC (none) -> C2128
- D8, D9: LCSC (none) -> C72043
- H1, H2, H3: LCSC part number - -> (none); now left out of the parts list
- H4: LCSC (none) -> C2915630; verif 1 -> (none)
- IC1: LCSC (none) -> C86803
- IC2: LCSC (none) -> C181692
- J12, J4: LCSC (none) -> C358721
- J13, J14, J15, J17, J18, J19, J21, J24, J25, J26, J27, J9: LCSC (none) -> C492405; LCSC part number - -> C492405; now in the parts list
- J2: LCSC (none) -> C319148; LCSC part number (none) -> C319148; verif (none) -> 1
- J3: LCSC (none) -> C492403; LCSC part number C2718488 -> C492403
- J30: LCSC (none) -> C111196
- J5: LCSC (none) -> C2718488
- J6, J8: footprint Connector_PinSocket_2.54mm:PinSocket_1x06_P2.54mm_Vertical_SMD_Pin1Right -> Connector_PinSocket_2.54mm:PinSocket_1x06_P2.54mm_Vertical; LCSC (none) -> C40877; LCSC part number (none) -> C40877; verif (none) -> 1
- J7: LCSC (none) -> C49661
- L1: LCSC (none) -> C112125; LCSC part number C385251 -> C112125
- R1, R2, R3: LCSC (none) -> C17958; LCSC part number C25092 -> C17958
- R10, R4: LCSC (none) -> C17902; LCSC part number C25744 -> C17902
- R11: LCSC (none) -> C25340; LCSC part number C880273 -> C25340
- R12: LCSC (none) -> C17986; LCSC part number C25798 -> C17986
- R13: verif (none) -> 1; now left out of the parts list
- R14: LCSC (none) -> C17900; LCSC part number C25905 -> C17900
- R15, R16: LCSC (none) -> C17900; LCSC part number C25092 -> C17900
- R19: LCSC (none) -> C17957; LCSC part number C17557 -> C17957
- R20, R21: LCSC (none) -> C17969; LCSC part number C17714 -> C17969
- R22: LCSC (none) -> C4502; LCSC part number C17710 -> C4502
- R34, R35, R36, R37, R38, R39, R5, R6: LCSC (none) -> C4502; LCSC part number C25117 -> C4502
- R40, R41: LCSC (none) -> C17936; LCSC part number C25900 -> C17936
- R7, R8: LCSC (none) -> C26033; LCSC part number C25905 -> C26033
- R9: LCSC (none) -> C17942; LCSC part number C22977 -> C17942
- SW1, SW6: LCSC (none) -> C318884
- SW10, SW8: LCSC (none) -> C319060
- SW2, SW3, SW4, SW5: LCSC (none) -> C84931
- SW9: LCSC (none) -> C319058; LCSC part number C319060 -> C319058
- TP1: value +5v charger output -> CHG>5v; verif (none) -> 1
- TP2, TP3, TP5, TP6, TP7, TP8, U10, U11, U13, U14, U15, U5, U6, U9: verif (none) -> 1
- TP4: value +3v3 peripheral -> +3v3 periph; verif (none) -> 1
- U1: LCSC (none) -> C107671
- U16: LCSC (none) -> C841659; verif 1 -> (none)
- U17, U19: LCSC (none) -> C485517
- U2, U3: footprint Connector_PinSocket_2.54mm:PinSocket_1x24_P2.54mm_Vertical_SMD_Pin1Right -> Connector_PinSocket_2.54mm:PinSocket_1x20_P2.54mm_Vertical; LCSC (none) -> C50984; LCSC part number (none) -> C50984; verif (none) -> 1
- U4: LCSC (none) -> C91322
- U7: value TLV75533PDBV -> TLV75733PDBV; LCSC (none) -> C485517; LCSC part number C404027 -> C485517
- U8: LCSC (none) -> C571211
Connections:
- net +3V3: now also U38.3 (+5v)
- net GEN_LED6: now also U16.49 (22_BATT_VIN_A8), U3.5 (22_A8_CTX1); no longer U16.63 (33_G10_ADCD+), U3.24 (33_MCLK2)
- net GND: now also C33.2, H5.1, IC3.17 (EP), IC3.7 (VSS), U38.1 (gnd)
- net I2C_SCL: now also IC3.15 (I2C_SCL)
- net I2C_SDA: now also IC3.14 (I2C_SDA)
- net I2S_BCK: now also NT4.2; no longer U16.50 (21_BCLK_A7), U3.6 (21_A7_RX5_BCLK1)
- net I2S_DIN: now also NT3.2; no longer U16.56 (7_AUD_OUT), U2.9 (7_RX2_OUT1A)
- net I2S_LRCK: now also NT2.2; no longer U16.52 (20_LRCLK_A6), U3.7 (20_A6_TX5_LRCLK1)
- net Supply+5v: now also C17.1, C20.1, C21.1, C22.1, C23.1
- net WS2812_DATA: now also U38.2 (Data)
- net i2c_3v3: now also IC3.5 (VDDIO), IC3.6 (VDD)
- net captouch_05: now reaches J8.1 (Pin_1), U4.13 (LED1/ELE5)
- net captouch_05: now also IC3.9 (CS5/GPO1)
- net captouch_06: now reaches J8.2 (Pin_2), U4.14 (LED2/ELE6)
- net captouch_06: now also IC3.10 (CS6/GPO2)
- net captouch_07: now reaches J8.3 (Pin_3), U4.15 (LED3/ELE7)
- net captouch_07: now also IC3.11 (CS7/GPO3/SH)
- net captouch_00: now reaches J6.2 (Pin_2), U4.8 (ELE0)
- net captouch_00: now also IC3.1 (CS0/PS0)
- net captouch_01: now reaches J6.3 (Pin_3), U4.9 (ELE1)
- net captouch_01: now also IC3.2 (CS1/PS1)
- net captouch_02: now reaches J6.4 (Pin_4), U4.10 (ELE2)
- net captouch_02: now also IC3.12 (CS2/GUARD)
- net captouch_03: now reaches J6.5 (Pin_5), U4.11 (ELE3)
- net captouch_03: now also IC3.13 (CS3)
- net captouch_04: now reaches J6.6 (Pin_6), U4.12 (LED0/ELE4)
- net captouch_04: now also IC3.8 (CS4/GPO0)
- removed net SPI0_generic0_cs: J4.6 (Pin_6), U16.43 (31_CAN_TX), U2.23 (31_CTX3)
- removed net SPI0_generic1_cs: J4.7 (Pin_7), U16.65 (32_G9_ADCD-), U2.24 (32_OUT1B)
- new net: C33.1, IC3.4 (VCC)
- new net I2S_BCK_MM: NT4.1, U16.50 (21_BCLK_A7)
- new net I2S_BCK_T4: NT4.3, U3.6 (21_A7_RX5_BCLK1)
- new net I2S_DIN_MM: NT3.1, U16.56 (7_AUD_OUT)
- new net I2S_DIN_T4: NT3.3, U2.9 (7_RX2_OUT1A)
- new net I2S_LRCK_MM: NT2.1, U16.52 (20_LRCLK_A6)
- new net I2S_LRCK_T4: NT2.3, U3.7 (20_A6_TX5_LRCLK1)
- new net charger output: IC2.8 (VOUT), SW9.2
- no-connect marks 52 -> 59
Other:
- note added: "CapSense, i2c 0x37"
- note added: "https://cdn.sparkfun.com/assets/5/8/e/f/a/MicroMod_Data_Logging_CB-Schematic.pdf https://cdn.sparkfun.com/assets/5/a/3/6/0/MicroMod-Teensy_V1_3.pdf https://www.pjrc.com/teensy/schematic41.png https://learn.sparkfun.com/tutorials/designing-with-micromod/all"
- note removed: "- use different m.2 (Foxconn?) - no vias under m.2 https://cdn.sparkfun.com/assets/5/8/e/f/a/MicroMod_Data_Logging_CB-Schematic.pdf https://cdn.sparkfun.com/assets/5/a/3/6/0/MicroMod-Teensy_V1_3.pdf https://www.pjrc.com/teensy/schematic41.png https://learn.sparkfun.com/tutorials/designing-with-micromod/all"
- moved on the sheet: C17, C20, C21, C22, C23, J6, J8, U5

Commit message: adding changes leftover from MSI crash. basically a working & tested devboard 5 (same as 6). for some reason, newlines changed.
Parts:
- removed BT1: Battery_Cell, Battery:BatteryHolder_Keystone_1042_1x18650, symbol Device:Battery_Cell
- removed C1, C15, C16: 10uF, Capacitor_SMD:C_0805_2012Metric, symbol Device:C
- removed C18, C19: 22uF, Capacitor_SMD:C_0805_2012Metric, symbol Device:C
- removed C2, C30: 0.22uF, Capacitor_SMD:C_0805_2012Metric, symbol Device:C
- removed C24, C25, C26, C28, C31, C33: 0.1uF, Capacitor_SMD:C_0805_2012Metric, symbol Device:C
- removed C29, C32: 1uF, Capacitor_SMD:C_0805_2012Metric, symbol Device:C
- removed D1: 25%, LED_SMD:LED_0805_2012Metric, symbol Device:LED
- removed D10, D11: red, LED_SMD:LED_0603_1608Metric, symbol Device:LED
- removed D16: 3.3v, Diode_SMD:D_MiniMELF, symbol Device:D_Zener
- removed D2: 50%, LED_SMD:LED_0805_2012Metric, symbol Device:LED
- removed D3: 75%, LED_SMD:LED_0805_2012Metric, symbol Device:LED
- removed D4: 100%, LED_SMD:LED_0805_2012Metric, symbol Device:LED
- removed H4: M.2 riser 2.5mm, clarinoid2:Sinhoo SMTSO2530CTJ, symbol Mechanical:MountingHole_Pad
- removed IC2: Injoinic IP5306 battery charge, SamacSys_Parts:SOIC127P599X155-9N, symbol clarinoid2:Injoinic IP5306 battery charge
- removed IC3: CY8CMBR3108-LQXIT, SamacSys_Parts:QFN50P300X300X60-17N-D, symbol SamacSys_Parts:CY8CMBR3108-LQXIT
- removed J3: header_usbfromteensy, Connector_PinSocket_2.54mm:PinSocket_1x04_P2.54mm_Vertical, symbol Connector_Generic:Conn_01x04
- removed J30: microSD SOFNG TF-15x15, clarinoid2:SOFNG TF-15x15 (LCSC C111196), symbol clarinoid2:microSD SOFNG TF-15x15
- removed J4: header_spi, Connector_PinSocket_2.54mm:PinSocket_1x07_P2.54mm_Vertical, symbol Connector_Generic:Conn_01x07
- removed J7: header_power tap, Connector_PinSocket_2.54mm:PinSocket_1x02_P2.54mm_Vertical, symbol Connector_Generic:Conn_01x02
- removed J8: Conn_01x06, Connector_PinSocket_2.54mm:PinSocket_1x06_P2.54mm_Vertical, symbol Connector_Generic:Conn_01x06
- removed L1: 1uH, clarinoid2:Inductor_MCS0630-1R0MN2, symbol pspice:INDUCTOR
- removed NT2: I2S tee_LRCK, NetTie:NetTie-3_SMD_Pad0.5mm, symbol Device:NetTie_3_Tee
- removed NT3: I2S tee_DIN, NetTie:NetTie-3_SMD_Pad0.5mm, symbol Device:NetTie_3_Tee
- removed NT4: I2S tee_BCK, NetTie:NetTie-3_SMD_Pad0.5mm, symbol Device:NetTie_3_Tee
- removed R10, R4: 10k, Resistor_SMD:R_1206_3216Metric, symbol Device:R
- removed R11: 0.5R, Resistor_SMD:R_1206_3216Metric, symbol Device:R
- removed R12: 75k, Resistor_SMD:R_1206_3216Metric, symbol Device:R
- removed R14, R15, R16: 100k, Resistor_SMD:R_1206_3216Metric, symbol Device:R
- removed R38, R39: 470R, Resistor_SMD:R_1206_3216Metric, symbol Device:R
- removed R9: 2R, Resistor_SMD:R_1206_3216Metric, symbol Device:R
- removed SW1, SW6: SW_Push, clarinoid2:XKB switch jlcpcb SW_TS-1187A-B-A-B, symbol clarinoid2:XKB tactile switch jlcpcb TS-1187A-B-A-B
- removed SW10, SW8: DIP red power source, clarinoid2:dip switch XKB DS-04, symbol Switch:SW_DIP_x04
- removed SW9: DIP red power source, clarinoid2:dip switch XKB DS-06RP, symbol Switch:SW_DIP_x06
- removed TP1: CHG>5v, TestPoint:TestPoint_THTPad_D2.0mm_Drill1.0mm, symbol Connector:TestPoint
- removed TP2: GND, TestPoint:TestPoint_THTPad_D2.0mm_Drill1.0mm, symbol Connector:TestPoint
- removed TP4: +3v3 periph, TestPoint:TestPoint_THTPad_D2.0mm_Drill1.0mm, symbol Connector:TestPoint
- removed TP5: +5v supply, TestPoint:TestPoint_THTPad_D2.0mm_Drill1.0mm, symbol Connector:TestPoint
- removed TP7: 3v3, TestPoint:TestPoint_THTPad_D2.0mm_Drill1.0mm, symbol Connector:TestPoint
- removed U16: APCI0108-P001A Teensy_4.0_MicroMod, SamacSys_Parts:21992304, symbol Teensy_4.0_MicroMod:Teensy_4.0_MicroMod
- removed U17, U19: TLV75733PDBV, Package_TO_SOT_SMD:SOT-23-5, symbol Regulator_Linear:TLV75733PDBV
- removed U18: Micromod outline, clarinoid2:Teensy_4.0_MicroMod outline fab, symbol clarinoid2:Placeholder
- removed U2: Teensy4.1_LEFT, Connector_PinSocket_2.54mm:PinSocket_1x20_P2.54mm_Vertical, symbol clarinoid2:Teensy4.1_LEFT
- removed U3: Teensy4.1_RIGHT, Connector_PinSocket_2.54mm:PinSocket_1x20_P2.54mm_Vertical, symbol clarinoid2:Teensy4.1_RIGHT
- removed U4: MPR121, 0x5A, Package_DFN_QFN:UQFN-20_3x3mm_P0.4mm, symbol Sensor_Touch:MPR121QR2
- removed U5: main captouch graphic, CapTouchSliders:captouch dev board subboard template, symbol clarinoid2:Placeholder
- removed U6: Placeholder, clarinoid2:Teensy41_graphic, symbol clarinoid2:Placeholder
- added H13, H14, H15: MountingHole, MountingHole:MountingHole_3.2mm_M3, symbol Mechanical:MountingHole
- added J31: 4p, Connector_PinSocket_2.54mm:PinSocket_1x04_P2.54mm_Vertical, symbol Connector_Generic:Conn_01x04
- added J32: header_power tap, Connector_PinSocket_2.54mm:PinSocket_1x02_P2.54mm_Vertical, symbol Connector_Generic:Conn_01x02
- added J43: Conn_01x20, Connector_PinSocket_2.54mm:PinSocket_1x20_P2.54mm_Vertical, symbol Connector_Generic:Conn_01x20
- added J44: Conn_01x08, Connector_PinSocket_2.54mm:PinSocket_1x08_P2.54mm_Vertical, symbol Connector_Generic:Conn_01x08
- added J45, J52, J53: female 1x6, Connector_PinSocket_2.54mm:PinSocket_1x06_P2.54mm_Vertical, symbol Connector_Generic:Conn_01x06
- added J8: female 1x4, Connector_PinSocket_2.54mm:PinSocket_1x04_P2.54mm_Vertical, symbol Connector_Generic:Conn_01x04
- added U16: power template, clarinoid2:dev board power board template, symbol clarinoid2:Placeholder
- added U4: captouch board template, clarinoid2:dev board captouch board template, symbol clarinoid2:Placeholder
- added U44: processor board template, clarinoid2:dev board processor subboard template, symbol clarinoid2:Placeholder
- added U48, U49, U50, U51, U52, U53, U54, U55, U56, U57, U58, U59, U60, U61, U62, U63, U64, U65, U66, U67, U68: mb1, clarinoid2:mouse-bite-2mm-slot, symbol clarinoid2:Placeholder
- H1: footprint MountingHole:MountingHole_3.2mm_M3_Pad_Via -> clarinoid2:MountingHole_3.2mm_M3_Pad_SQUARE
- J6: value Conn_01x06 -> female 1x6; LCSC C40877 -> C358720; LCSC part number C40877 -> C358720
Connections:
- net I2S_BCK is gone; now on net I2S_BCK_MM: R3.1
- net I2S_DIN is gone; now on net I2S_DIN_MM: R2.1
- net I2S_LRCK is gone; now on net I2S_LRCK_MM: R1.1
- net dac_3v3 is gone; now on net +3.3v regulator output: C5.1, C6.1, NT1.1
- net i2c_3v3 is gone; now on net +3.3v regulator output: IC1.16 (VDD), J5.2 (Pin_2), R40.1, R41.1
- net spi_3v3 is gone; now on net +3.3v regulator output: J12.2 (VDD)
- net ENC_A: now also J43.19 (Pin_19)
- net ENC_B: now also J43.20 (Pin_20)
- net ENC_SWITCH: now also J43.18 (Pin_18)
- net GEN_LED1: now also J44.5 (Pin_5)
- net GEN_LED2: now also J44.6 (Pin_6)
- net GEN_LED3: now also J44.7 (Pin_7)
- net GEN_LED4: now also J44.8 (Pin_8)
- net I2C_SCL: now also J43.4 (Pin_4), J8.4 (Pin_4)
- net I2C_SDA: now also J43.5 (Pin_5), J8.3 (Pin_3)
- net I2S_BCK_MM: now also J43.6 (Pin_6)
- net I2S_DIN_MM: now also J43.8 (Pin_8)
- net I2S_LRCK_MM: now also J43.7 (Pin_7)
- net OLED_CS: now also J43.15 (Pin_15)
- net OLED_DC: now also J43.17 (Pin_17)
- net OLED_RES: now also J43.16 (Pin_16)
- net SPI0_MISO: now also J43.14 (Pin_14)
- net SPI0_MOSI: now also J43.13 (Pin_13)
- net SPI0_SCK: now also J43.12 (Pin_12)
- net T00 MIDI IN: now also J43.9 (Pin_9)
- net T01=MIDI OUT: now also J43.10 (Pin_10)
- net WS2812_DATA: now also J43.11 (Pin_11)
- net at IC1.6 (IO2): now also SW4.1; no longer SW4.2
- net at IC1.7 (IO3): now also SW5.1; no longer SW5.2
- net at IC1.5 (IO1): now also SW3.1; no longer SW3.2
- net at IC1.4 (IO0): now also SW2.1; no longer SW2.2
- net +3V3 renamed +3.3v regulator output
- net +3.3v regulator output: now also J43.2 (Pin_2), J8.2 (Pin_2)
- net +5v before power switch renamed Power board output +5v
- net Power board output +5v: now also J32.2 (Pin_2)
- net GND renamed gnd from processor
- net gnd from processor: now also SW2.2, SW3.2, SW4.2, SW5.2, J43.1 (Pin_1), J8.1 (Pin_1); no longer C17.2, C20.2, C21.2, C22.2, C23.2, J2.A1 (GND), J2.A12 (GND), J2.B1 (GND), J2.B12 (GND), J2.S1 (SHIELD), J6.1 (Pin_1), R7.1, R8.1, SW2.1, SW3.1, SW4.1, SW5.1
- net Supply+5v renamed 5v regulated
- net 5v regulated: now also J44.4 (Pin_4); no longer C27.1, U8.8 (VCC)
- net USB data in + renamed USB D+
- net USB D+: now also J31.2 (Pin_2), J44.2 (Pin_2)
- net USB data in - renamed USB D-
- net USB D-: now also J31.3 (Pin_3), J44.3 (Pin_3)
- net USB_Vin5v renamed USB VIN 5v
- net USB VIN 5v: now also J31.4 (Pin_4)
- net captouch_00: no longer names the net of J6.2 (Pin_2)
- net captouch_00: now also J52.2 (Pin_2)
- net captouch_01: no longer names the net of J6.3 (Pin_3)
- net captouch_01: now also J52.3 (Pin_3)
- net captouch_02: no longer names the net of J6.4 (Pin_4)
- net captouch_02: now also J52.4 (Pin_4)
- net captouch_03: no longer names the net of J6.5 (Pin_5)
- net captouch_03: now also J52.5 (Pin_5)
- net captouch_04: no longer names the net of J6.6 (Pin_6)
- net captouch_04: now also J52.6 (Pin_6)
- new net: J45.1 (Pin_1), J53.1 (Pin_1)
- new net: J45.2 (Pin_2), J53.2 (Pin_2)
- new net: J45.3 (Pin_3), J53.3 (Pin_3)
- new net: J45.4 (Pin_4), J53.4 (Pin_4)
- new net: J45.5 (Pin_5), J53.5 (Pin_5)
- new net: J45.6 (Pin_6), J53.6 (Pin_6)
- new net: J52.1 (Pin_1), J6.1 (Pin_1)
- new net 5v from processor: C27.1, J43.3 (Pin_3), U8.8 (VCC)
- new net powerboard outp GND: C17.2, C20.2, C21.2, C22.2, C23.2, J32.1 (Pin_1), J44.1 (Pin_1)
- new net usb gnd: J2.A1 (GND), J2.A12 (GND), J2.B1 (GND), J2.B12 (GND), J2.S1 (SHIELD), J31.1 (Pin_1), R7.1, R8.1
- no-connect marks 59 -> 14
Other:
- added sheet captouch_capsense (captouch_capsense.kicad_sch)
- added sheet captouch_mpr121 (captouch_mpr121.kicad_sch)
- added sheet power_battery (power_battery.kicad_sch)
- added sheet power_header (power_header.kicad_sch)
- added sheet power_usb (power_usb.kicad_sch)
- added sheet processor_mm (processor_mm.kicad_sch)
- added sheet processor_t4 (processor_t4.kicad_sch)
- note added: "PCA9554APW,118 0x38"
- note added: "todo: x length match x silkscreen, drc, erc x switch footprints x exclude backside headers from BOM as needed - JLCPCB part numbers for headers"
- note removed: "1 = [USB power] 2 = [BATT power] 3 = [HDR power] 4 = USB to charger 5 = HDR to charger 6 = enable 3v3 reg (Micromod), or use internal teensy 3v3"
- note removed: "3.3v REG"
- note removed: "CapSense, i2c 0x37"
- note removed: "MPR121, 0x5A i2c built-in slider"
- note removed: "PCA9554APW,118 0x38 built-in"
- note removed: "battery charge and 5v reg"
- note removed: "https://cdn.sparkfun.com/assets/5/8/e/f/a/MicroMod_Data_Logging_CB-Schematic.pdf https://cdn.sparkfun.com/assets/5/a/3/6/0/MicroMod-Teensy_V1_3.pdf https://www.pjrc.com/teensy/schematic41.png https://learn.sparkfun.com/tutorials/designing-with-micromod/all"
- note removed: "microSD"
- note removed: "peripheral power 3v3"
- moved on the sheet: C17, C20, C21, C22, C23, C3, C4, C5, C6, D5, D7, D8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
