File: CAD/bommanoid/bommanoid00/bommanoid00.kicad_pcb (KiCad board)
At the start: 2 copper layers, 56 parts

Commit message: bomma design progress
Parts:
- removed the REF** at (-292.4, 68.3)
- removed the REF** at (-468.8, 85.0)
- removed the REF** at (-275.4, 85.3)
- removed the REF** at (-281.1, 79.7)
- removed the REF** at (-286.8, 74.0)
- added REF**: LED_RGB_5050-6, LED_SMD:LED_RGB_5050-6, F.Cu at (-335.8, 82.7)
- added REF**: LED_RGB_5050-6, LED_SMD:LED_RGB_5050-6, F.Cu at (-341.4, 77.0)
- added REF**: LED_RGB_5050-6, LED_SMD:LED_RGB_5050-6, F.Cu at (-347.1, 71.3)
- added REF**: LED_RGB_5050-6, LED_SMD:LED_RGB_5050-6, F.Cu at (-352.8, 65.7)
- moved REF** 42.2 mm to (-68.8, 76.0)
- moved REF** 35.2 mm to (-326.8, 90.0), turned to 0 degrees
- moved REF** 25.0 mm to (-57.8, 152.0)
- moved REF** 25.0 mm to (-57.8, 136.0)
- moved REF** 25.0 mm to (-57.8, 128.0)
- moved REF** 25.0 mm to (-57.8, 144.0)
- moved REF** 18.0 mm to (-430.8, 79.0)
- moved REF** 18.0 mm to (-408.8, 79.0)
- moved REF** 12.0 mm to (-122.8, 76.0)
- moved REF** 12.0 mm to (-100.8, 76.0)
- moved REF** 11.4 mm to (-207.8, 72.0)
- moved REF** 7.66 mm to (-151.8, 90.3), turned to 180 degrees
- moved REF** 7.36 mm to (-161.3, 80.5), turned to 45 degrees
- moved REF** 7.29 mm to (-169.8, 72.0), turned to 45 degrees
- moved REF** 5.92 mm to (-164.1, 77.7), turned to 45 degrees
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Other:
- board text added: "BATTERY PCB also needs 2 levels, because we need LEDs to be close to the case, but we also want the battery holder to be visible. this also allows us to put the on-off pot on the back panel JST-PH vertical requires 20mm clearance with wires. that means interconnects will go under."
- board text removed: "BATTERY PCB also needs 2 levels, because we need LEDs to be close to the case, but we also want the battery holder to be visible. this also allows us to put the on-off pot on the back panel"
