File: CAD/bommanoid/bommanoid01/bell.kicad_sch (KiCad schematic)
At the start: 0 parts

Commit message: progress on bommanoid pcb design adding some winisd simulations
Parts:
- added D25, D26, D29, D30, D32, D34: LED, LED_THT:LED_D5.0mm, symbol Device:LED
- added D27, D28, D31, D33, D35, D36, D37, D38: WS2812B, LED_SMD:LED_WS2812B_PLCC4_5.0x5.0mm_P3.2mm, symbol LED:WS2812B
- added H15, H16: MountingHole_Pad, MountingHole:MountingHole_3.2mm_M3, symbol Mechanical:MountingHole_Pad
- added J31: RJ45_LED_Shielded, Connector_RJ:RJ45_Amphenol_RJHSE538X, symbol Connector:RJ45_LED_Shielded
- added R38, R39, R40, R41, R42, R43, R44, R45: R, Resistor_THT:R_Axial_DIN0207_L6.3mm_D2.5mm_P10.16mm_Horizontal, symbol Device:R
Connections:
- new net: D29.1 (K), R40.1
- new net: D25.1 (K), R38.1
- new net: D27.2 (DOUT), D28.4 (DIN)
- new net: D32.1 (K), R42.1
- new net: D37.2 (DOUT), D38.4 (DIN)
- new net: D31.2 (DOUT), D33.4 (DIN)
- new net: D28.2 (DOUT), D31.4 (DIN)
- new net: D26.1 (K), R39.1
- new net: D35.2 (DOUT), D36.4 (DIN)
- new net: D33.2 (DOUT), D35.4 (DIN)
- new net: J31.9, R44.2
- new net: D30.1 (K), R41.1
- new net: D36.2 (DOUT), D37.4 (DIN)
- new net: D34.1 (K), R43.1
- new net: J31.11, R45.2
- new net amp_5v: D25.2 (A), J31.8
- new net gnd: D27.3 (VSS), D28.3 (VSS), D31.3 (VSS), D33.3 (VSS), D35.3 (VSS), D36.3 (VSS), D37.3 (VSS), D38.3 (VSS), H15.1, H16.1, J31.1, J31.SH, R38.2, R39.2, R40.2, R41.2, R42.2, R43.2, R44.1, R45.1
- new net led_act1_5v: D29.2 (A), J31.12, J31.5
- new net led_act2_5v: D30.2 (A), J31.6
- new net led_act3_5v: D32.2 (A), J31.7
- new net led_blink_5v: D34.2 (A), J31.10, J31.4
- new net sys_5v: D26.2 (A), D27.1 (VDD), D28.1 (VDD), D31.1 (VDD), D33.1 (VDD), D35.1 (VDD), D36.1 (VDD), D37.1 (VDD), D38.1 (VDD), J31.2
- new net ws2812_data: D27.4 (DIN), J31.3
- no-connect marks 0 -> 1
Other:
- note added: "LED 20ma / 1.9 @ 2ma https://cdn.amphenol-cs.com/media/wysiwyg/files/documentation/datasheet/inputoutput/io-modjack-rjhse.pdf"
- note added: "RJ45"
- note added: "led lighting"
