File: CAD/bommanoid/bommanoid01/bommanoid_batt_top.kicad_sch (KiCad schematic)
At the start: 25 parts, among them J8 korg female oct

Commit message: progress on bommanoid pcb design adding some winisd simulations
Parts:
- removed D10, D13, D14, D9: blue, LED_SMD:LED_0603_1608Metric, symbol Device:LED
- removed D11, D12, D15, D4, D6: green, LED_SMD:LED_0603_1608Metric, symbol Device:LED
- removed D3, D5, D7, D8: WS2812B, LED_SMD:LED_WS2812B_PLCC4_5.0x5.0mm_P3.2mm, symbol LED:WS2812B
- removed J8: korg female oct, symbol Connector_Generic:Conn_01x09
- removed R16, R17, R18, R19, R20, R21, R22, R23, R24, R25: 470R, Resistor_SMD:R_1206_3216Metric, symbol Device:R
- added C16, C26: 10uF, Capacitor_SMD:C_1206_3216Metric, symbol Device:C
- added C27, C28, C29, C30: 22uF, Capacitor_SMD:C_1206_3216Metric, symbol Device:C
- added C31, C32: 22uF, Capacitor_SMD:C_0603_1608Metric, symbol Device:C
- added C33: 0.1uF, Capacitor_SMD:C_1206_3216Metric, symbol Device:C
- added H8, H9: MountingHole_Pad, MountingHole:MountingHole_3.2mm_M3, symbol Mechanical:MountingHole_Pad
- added IC3: Injoinic IP5306 battery charge, clarinoid2:SOIC127P599X155-9N (IP5306), symbol clarinoid2:Injoinic IP5306 battery charge
- added J20: Conn_01x07, Connector_PinSocket_2.54mm:PinSocket_1x07_P2.54mm_Vertical, symbol Connector_Generic:Conn_01x05
- added J21: Conn_01x05, Connector_PinSocket_2.54mm:PinSocket_1x05_P2.54mm_Vertical, symbol Connector_Generic:Conn_01x05
- added L1: 1uH-psa, clarinoid2:Inductor_MCS0630-1R0MN2, symbol pspice:INDUCTOR
- added R27: 2R, Resistor_SMD:R_0603_1608Metric, symbol Device:R
- added R28: 10k, Resistor_SMD:R_0603_1608Metric, symbol Device:R
- added R29: 0.5R, Resistor_SMD:R_0603_1608Metric, symbol Device:R
- D16: value green -> korgpwr; footprint LED_SMD:LED_0603_1608Metric -> LED_SMD:LED_0805_2012Metric; LCSC C72043 -> C264424; LCSC part number C72043 -> C264424
Connections:
- net gnd: now also C16.2, C26.2, C27.2, C28.2, C29.2, C30.2, C31.2, C32.2, C33.2, H8.1, H9.1, IC3.9 (PWR-GND), J20.1 (Pin_1)
- net korg_power_led_cathode: now reaches D16.1 (K)
- net korg_power_led_cathode: now also J21.5 (Pin_5)
- net GEN_LED4 renamed korg_power_led_anode
- net korg_power_led_anode: now also J21.4 (Pin_4)
- new net: C16.1, R27.2
- new net: IC3.7 (SW-inductor), L1.1
- new net: IC3.5 (KEY), R28.1
- new net: C27.1, IC3.6 (BAT), R29.2
- new net batt+: C29.1, J20.2 (Pin_2), L1.2, R29.1
- new net chargeled_1: IC3.2 (LED1), J21.1 (Pin_1)
- new net chargeled_2: IC3.3 (LED2), J21.2 (Pin_2)
- new net chargeled_3: IC3.4 (LED3), J21.3 (Pin_3)
- new net charger output +5v: C28.1, C30.1, C31.1, C32.1, C33.1, IC3.8 (VOUT), J20.4 (Pin_4)
- new net key: J20.5 (Pin_5), R28.2
- new net usb_5v: C26.1, IC3.1 (VIN), J20.3 (Pin_3), R27.1
- no-connect marks 0 -> 2
Other:
- note added: "add test points"
- note added: "charge"
- note added: "korg.pwr"
- note added: "to bottom"
- note removed: "smt leds"
- note removed: "todo: - color of LEDs / part numbers"
