File: CAD/bommanoid/bommanoid01/bommanoid_main_bottom.kicad_sch (KiCad schematic)
At the start: 5 parts, among them J6 XKB_U262-16XN-4BVC11 USB-C re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, J7 SSD1306, U8 ssd1306_graphic

Commit message: progress on bommanoid pcb design adding some winisd simulations
Parts:
- removed J7: SSD1306, Connector_PinSocket_2.54mm:PinSocket_1x07_P2.54mm_Vertical, symbol clarinoid2:SSD1306
- added D10, D11, D12, D13, D14, D15, D7, D8, D9: LED, LED_THT:LED_D5.0mm, symbol Device:LED
- added H5, H6, H7: MountingHole_Pad, MountingHole:MountingHole_3.2mm_M3, symbol Mechanical:MountingHole_Pad
- added J10, J13, J19: Conn_01x07, Connector_PinSocket_2.54mm:PinSocket_1x07_P2.54mm_Vertical, symbol Connector_Generic:Conn_01x07
- added J11, J12, J14: Amphenol ACJS-MHOM, SamacSys_Parts:ACJSMHOM, symbol clarinoid2:Amphenol ACJS-MHOM
- added J15, J16: Conn_01x12, Connector_PinSocket_2.54mm:PinSocket_1x12_P2.54mm_Vertical, symbol Connector_Generic:Conn_01x12
- added J17: RJ45_LED_Shielded, Connector_RJ:RJ45_Amphenol_RJHSE538X, symbol Connector:RJ45_LED_Shielded
- added J18: Conn_01x03, Connector_PinSocket_2.54mm:PinSocket_1x03_P2.54mm_Vertical, symbol Connector_Generic:Conn_01x03
- added J7: Conn_02x10_Odd_Even, Connector_PinHeader_2.54mm:PinHeader_2x10_P2.54mm_Vertical, symbol Connector_Generic:Conn_02x10_Odd_Even
- added J8: Conn_01x08, Connector_PinSocket_2.54mm:PinSocket_1x08_P2.54mm_Vertical, symbol Connector_Generic:Conn_01x08
- added J9: Conn_02x04_Odd_Even, Connector_PinHeader_2.54mm:PinHeader_2x07_P2.54mm_Vertical, symbol Connector_Generic:Conn_02x07_Odd_Even
- added R16, R17, R18, R19, R20, R21, R22, R23, R24, R9: R, Resistor_THT:R_Axial_DIN0207_L6.3mm_D2.5mm_P10.16mm_Horizontal, symbol Device:R
- added R25: 5.1k, Resistor_SMD:R_1206_3216Metric, symbol Device:R
- R15: value 5.1k -> R; footprint Resistor_SMD:R_1206_3216Metric -> Resistor_THT:R_Axial_DIN0207_L6.3mm_D2.5mm_P10.16mm_Horizontal; LCSC C26033 -> (none); LCSC part number C26033 -> (none); verif 1 -> (none); now left out of the parts list
Connections:
- net gnd: now also J6.A1 (GND), J6.A12 (GND), J6.B1 (GND), J6.B12 (GND), J6.S1 (SHIELD), R14.1, R15.2, H5.1, H6.1, H7.1, J10.1 (Pin_1), J11.3 (S_1), J11.4 (S_2), J13.1 (Pin_1), J14.3 (S_1), J14.4 (S_2), J15.1 (Pin_1), J16.1 (Pin_1), J17.1, J17.SH, J19.1 (Pin_1), J7.10 (Pin_10), J7.12 (Pin_12), J7.14 (Pin_14), J7.16 (Pin_16), J7.18 (Pin_18), J7.2 (Pin_2), J7.4 (Pin_4), J7.6 (Pin_6), J7.8 (Pin_8), J8.1 (Pin_1), J9.10 (Pin_10), J9.12 (Pin_12), J9.14 (Pin_14), J9.2 (Pin_2), J9.4 (Pin_4), J9.6 (Pin_6), J9.8 (Pin_8), R16.2, R17.2, R18.2, R19.2, R20.2, R21.1, R22.1, R23.2, R24.2, R25.1, R9.2
- net at J6.A5 (CC): now also R25.2; no longer R15.2
- net USB D+ renamed usb_data_+
- net usb_data_+: now also J13.5 (Pin_5)
- net USB D- renamed usb_data_-
- net usb_data_-: now also J13.6 (Pin_6)
- net USB VIN 5v renamed usb_5v
- net usb_5v: now also D8.2 (A), J13.7 (Pin_7), J8.2 (Pin_2), J9.3 (Pin_3)
- removed net usb gnd: J6.A1 (GND), J6.A12 (GND), J6.B1 (GND), J6.B12 (GND), J6.S1 (SHIELD), R14.1, R15.1
- new net: D13.1 (K), R20.1
- new net: D11.1 (K), R18.1
- new net: D15.1 (K), R24.1
- new net: D8.1 (K), R15.1
- new net: D12.1 (K), R19.1
- new net: D10.1 (K), R17.1
- new net: J17.11, R22.2
- new net: J17.9, R21.2
- new net: D14.1 (K), R23.1
- new net: D9.1 (K), R16.1
- new net: D7.1 (K), R9.1
- new net 3v3: J10.2 (Pin_2), J13.4 (Pin_4), J19.2 (Pin_2)
- new net agnd: J12.3 (S_1), J12.4 (S_2), J18.1 (Pin_1), J8.4 (Pin_4)
- new net aleft_post_pot: J12.6 (T), J8.7 (Pin_7)
- new net aleft_pre_pot: J18.2 (Pin_2), J8.5 (Pin_5)
- new net amp_5v: D7.2 (A), J17.8, J9.1 (Pin_1)
- new net aright_post_pot: J12.5 (R), J8.8 (Pin_8)
- new net aright_pre_pot: J18.3 (Pin_3), J8.6 (Pin_6)
- new net btn_x1: J16.2 (Pin_2), J7.1 (Pin_1)
- new net btn_x2: J16.3 (Pin_3), J7.3 (Pin_3)
- new net btn_x3: J16.4 (Pin_4), J7.5 (Pin_5)
- new net btn_x4: J16.5 (Pin_5), J7.7 (Pin_7)
- new net btn_x5: J16.6 (Pin_6), J7.9 (Pin_9)
- new net btn_x6: J16.7 (Pin_7), J7.11 (Pin_11)
- new net btn_x7: J16.8 (Pin_8), J7.13 (Pin_13)
- new net btn_x8: J16.9 (Pin_9), J7.15 (Pin_15)
- new net enc_a: J16.11 (Pin_11), J7.19 (Pin_19)
- new net enc_b: J16.12 (Pin_12), J7.20 (Pin_20)
- new net enc_btn: J16.10 (Pin_10), J7.17 (Pin_17)
- new net led_act1_5v: D11.2 (A), J15.3 (Pin_3), J17.5, J9.9 (Pin_9)
- new net led_act2_5v: D12.2 (A), J15.4 (Pin_4), J17.6, J9.11 (Pin_11)
- new net led_act3_5v: D13.2 (A), J15.5 (Pin_5), J17.7, J9.13 (Pin_13)
- new net led_blink_5v: D10.2 (A), J15.2 (Pin_2), J17.4, J9.7 (Pin_7)
- new net led_rj45_green_5v: J15.7 (Pin_7), J17.12
- new net led_rj45_yellow_5v: J15.6 (Pin_6), J17.10
- new net midi_in_ring: J14.5 (R), J15.9 (Pin_9)
- new net midi_in_tip: J14.6 (T), J15.10 (Pin_10)
- new net midi_out_ring: J11.5 (R), J15.11 (Pin_11)
- new net midi_out_tip: J11.6 (T), J15.12 (Pin_12)
- new net oled_cs: J10.7 (Pin_7), J19.7 (Pin_7)
- new net oled_data: J10.4 (Pin_4), J19.4 (Pin_4)
- new net oled_dc: J10.6 (Pin_6), J19.6 (Pin_6)
- new net oled_rst: J10.5 (Pin_5), J19.5 (Pin_5)
- new net oled_sck: J10.3 (Pin_3), J19.3 (Pin_3)
- new net prg: J13.2 (Pin_2)
- new net sys_5v: D14.2 (A), D15.2 (A), D9.2 (A), J13.3 (Pin_3), J17.2, J8.3 (Pin_3), J9.5 (Pin_5)
- new net ws2812_data_5v: J15.8 (Pin_8), J17.3
- no-connect marks 0 -> 6
Other:
- note added: "LED 20ma / 1.9 @ 2ma https://cdn.amphenol-cs.com/media/wysiwyg/files/documentation/datasheet/inputoutput/io-modjack-rjhse.pdf"
- note added: "MAIN BOTTOM add test points"
- note added: "RJ45"
- note added: "audio"
- note added: "audio out"
- note added: "buttons"
- note added: "led+midi"
- note added: "midi in"
- note added: "midi out"
- note added: "oled"
- note added: "oled from top"
- note added: "pwr+usb"
- note added: "status leds (all 5v input!)"
- note added: "to batt"
- note added: "to top"
- note added: "under lighting"
- note added: "wire"
- moved on the sheet: J6, R14, U8
