File: CAD/bommanoid/bommanoid01/bommanoid_main_top.kicad_sch (KiCad schematic)
At the start: 52 parts, among them J1 header_i2c, J2 AudioOut, J4 MIDI IN, J5 MIDI OUT, SW1 SW_Push, SW2 RotaryEncoder_Switch_ABC12, U1 PCM5102A, U2 TLV75733PDBV, U3 TLV75733PDBV, U4 APCI0108-P001A Teensy_4.0_Mic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, U5 processor board template, U6 Micromod outline, U7 6N138

Commit message: progress on bommanoid pcb design adding some winisd simulations
Parts:
- removed H2: MountingHole, MountingHole:MountingHole_3.2mm_M3, symbol Mechanical:MountingHole
- removed J1: header_i2c, Connector_PinSocket_2.54mm:PinSocket_1x04_P2.54mm_Vertical, symbol Connector_Generic:Conn_01x04
- removed J2: AudioOut, clarinoid2:SWITCHCRAFT_35RAPC4BV4_OvalHoles, symbol clarinoid2:Switchcraft 35RAPC4BV4
- removed J4: MIDI IN, clarinoid2:SWITCHCRAFT_35RAPC4BV4_OvalHoles, symbol clarinoid2:Switchcraft 35RAPC4BV4
- removed J5: MIDI OUT, clarinoid2:SWITCHCRAFT_35RAPC4BV4_OvalHoles, symbol clarinoid2:Switchcraft 35RAPC4BV4
- removed SW1: SW_Push, clarinoid2:XKB switch jlcpcb SW_TS-1187A-B-A-B, symbol clarinoid2:XKB tactile switch jlcpcb TS-1187A-B-A-B
- removed SW2: RotaryEncoder_Switch_ABC12, clarinoid2:Bourns_ENC_PEC11R-4215F-S0024, symbol clarinoid2:RotaryEncoder_Switch_ABC12
- removed TP1: D3v3, TestPoint:TestPoint_THTPad_D2.0mm_Drill1.0mm, symbol Connector:TestPoint
- removed TP2: A3v3, TestPoint:TestPoint_THTPad_D2.0mm_Drill1.0mm, symbol Connector:TestPoint
- removed TP3: AGND, TestPoint:TestPoint_THTPad_D2.0mm_Drill1.0mm, symbol Connector:TestPoint
- removed U5: processor board template, clarinoid2:dev board processor subboard template, symbol clarinoid2:Placeholder
- added D3, D4, D5, D6: WS2812B, LED_SMD:LED_WS2812B_PLCC4_5.0x5.0mm_P3.2mm, symbol LED:WS2812B
- added H2, H3, H4: MountingHole_Pad, MountingHole:MountingHole_3.2mm_M3, symbol Mechanical:MountingHole_Pad
- added IC1, IC2: SN74AHCT125N, SamacSys_Parts:DIP794W53P254L1930H508Q14N, symbol SamacSys_Parts:SN74AHCT125N
- added J1, J2: Conn_01x07, Connector_PinHeader_2.54mm:PinHeader_1x07_P2.54mm_Vertical, symbol Connector_Generic:Conn_01x07
- added J3, J4: Conn_01x12, Connector_PinHeader_2.54mm:PinHeader_1x12_P2.54mm_Vertical, symbol Connector_Generic:Conn_01x12
- added J5: Conn_01x03, Connector_PinHeader_2.54mm:PinHeader_1x03_P2.54mm_Vertical, symbol Connector_Generic:Conn_01x03
- added U5: MCP23017_SP, Package_DIP:DIP-28_W7.62mm, symbol Interface_Expansion:MCP23017_SP
- C20: symbol Device:C -> Device:C_Small
Connections:
- net 5v input is gone; now on net sys_5v: C13.1, C14.1, C15.1, R8.2, U3.1 (IN), U4.9 (VUSB)
- net gnd from processor is gone; now on net gnd: C1.2, C10.1, C2.2, C20.2, C6.2, C7.1, C9.2, U1.10 (DEMP), U1.11 (FLT), U1.16 (FMT), U1.19 (DGND), U2.2 (GND), U7.5 (GND)
- net I2C_SCL: now also R6.1, U5.12 (SCK); no longer R6.2
- net I2C_SDA: now also R7.1, U5.13 (SDA); no longer R7.2
- net gnd: now also D3.3 (VSS), D4.3 (VSS), D5.3 (VSS), D6.3 (VSS), H2.1, H3.1, H4.1, IC1.1 (1~{OE}), IC1.10 (3~{OE}), IC1.13 (4~{OE}), IC1.4 (2~{OE}), IC1.7 (GND), IC2.1 (1~{OE}), IC2.13 (4~{OE}), IC2.4 (2~{OE}), IC2.7 (GND), J1.1 (Pin_1), J2.1 (Pin_1), J3.1 (Pin_1), J4.1 (Pin_1), U5.10 (VSS), U5.15 (A0), U5.16 (A1), U5.17 (A2)
- net prg: now reaches U4.11 (PROGRAM)
- net prg: now also J2.2 (Pin_2)
- net led_blink_3v3: now reaches U4.44 (42_G2)
- net led_blink_3v3: now also IC1.5 (2A)
- net led_act1_3v3: now reaches U4.46 (43_G3)
- net led_act1_3v3: now also IC1.12 (4A)
- net led_act2_3v3: now reaches U4.48 (44_G4)
- net led_act2_3v3: now also IC1.9 (3A)
- net enc_b: now reaches U4.65 (32_G9_ADCD-)
- net enc_b: now also J4.12 (Pin_12)
- net led_act3_3v3: now reaches U4.73 (45_G5)
- net led_act3_3v3: now also IC2.2 (1A)
- net midi_out_tip: now reaches R13.1
- net midi_out_tip: now also J3.12 (Pin_12)
- net midi_in_tip: now reaches D2.2 (A), U7.3 (C2)
- net midi_in_tip: now also J3.10 (Pin_10)
- net midi_in_ring: now reaches R10.1
- net midi_in_ring: now also J3.9 (Pin_9)
- net midi_out_ring: now reaches R12.1
- net midi_out_ring: now also J3.11 (Pin_11)
- net +3.3v regulator output renamed 3v3
- net 3v3: now also R6.2, R7.2, J1.2 (Pin_2), J2.4 (Pin_4), U5.18 (~{RESET}), U5.9 (VDD); no longer R6.1, R7.1
- net 5v from processor renamed sys_5v
- net sys_5v: now also D3.1 (VDD), D4.1 (VDD), D5.1 (VDD), D6.1 (VDD), IC1.14 (VCC), IC2.14 (VCC), J2.3 (Pin_3)
- net A3v3 renamed a3v3
- net AGND renamed agnd
- net agnd: now also J5.1 (Pin_1)
- net D3v3 renamed d3v3
- net ENC_A renamed led_rj45_green_3v3
- net led_rj45_green_3v3: now also IC2.12 (4A)
- net ENC_B renamed enc_a
- net enc_a: now also J4.11 (Pin_11)
- net ENC_SWITCH renamed led_rj45_yellow_3v3
- net led_rj45_yellow_3v3: now also IC2.5 (2A)
- net GEN_LED1: no longer names the net of U4.47 (2_PWM1)
- net GEN_LED2: no longer names the net of U4.32 (3_PWM0)
- net GEN_LED3: no longer names the net of U4.10 (4_D0)
- net GEN_LED4: no longer names the net of U4.18 (5_D1)
- net OLED_CS renamed oled_cs
- net oled_cs: now also J1.7 (Pin_7)
- net OLED_DC renamed oled_dc
- net oled_dc: now also J1.6 (Pin_6)
- net OLED_RES renamed oled_rst
- net oled_rst: now also J1.5 (Pin_5)
- net SDIO_CLOCK: no longer names the net of U4.60 (36_SDIO_CLK)
- net SDIO_CS: no longer names the net of U4.70 (39_SDIO_DATA3)
- net SDIO_DAT2: no longer names the net of U4.68 (38_SDIO_DATA2)
- net SDIO_MISO: no longer names the net of U4.64 (35_SDIO_DATA0)
- net SDIO_MOSI: no longer names the net of U4.62 (37_SDIO_CMD)
- net SPI0_MISO: no longer names the net of U4.61 (12_SPI_SDI)
- net SPI0_MOSI renamed oled_data
- net oled_data: now also J1.4 (Pin_4)
- net SPI0_SCK renamed oled_sck
- net oled_sck: now also J1.3 (Pin_3)
- net WS2812_DATA renamed ws2812_data_3v3
- net ws2812_data_3v3: now also IC1.2 (1A)
- net dac output L renamed aleft
- net aleft: now also J5.2 (Pin_2)
- net dac output R renamed aright
- net aright: now also J5.3 (Pin_3)
- net sdio_dat1: no longer names the net of U4.66 (34_SDIO_DATA1)
- net usb data + renamed usb_data_+
- net usb_data_+: now also J2.5 (Pin_5)
- net usb data - renamed usb_data_-
- net usb_data_-: now also J2.6 (Pin_6)
- new net: D4.2 (DOUT), D5.4 (DIN)
- new net: D3.2 (DOUT), D4.4 (DIN)
- new net: D5.2 (DOUT), D6.4 (DIN)
- new net btn_x1: J4.2 (Pin_2), U5.21 (GPA0)
- new net btn_x2: J4.3 (Pin_3), U5.22 (GPA1)
- new net btn_x3: J4.4 (Pin_4), U5.23 (GPA2)
- new net btn_x4: J4.5 (Pin_5), U5.24 (GPA3)
- new net btn_x5: J4.6 (Pin_6), U5.25 (GPA4)
- new net btn_x6: J4.7 (Pin_7), U5.26 (GPA5)
- new net btn_x7: J4.8 (Pin_8), U5.27 (GPA6)
- new net btn_x8: J4.9 (Pin_9), U5.28 (GPA7)
- new net enc_btn: J4.10 (Pin_10), U5.1 (GPB0)
- new net led_act1_5v: IC1.11 (4Y), J3.3 (Pin_3)
- new net led_act2_5v: IC1.8 (3Y), J3.4 (Pin_4)
- new net led_act3_5v: IC2.3 (1Y), J3.5 (Pin_5)
- new net led_blink_5v: IC1.6 (2Y), J3.2 (Pin_2)
- new net led_rj45_green_5v: IC2.11 (4Y), J3.7 (Pin_7)
- new net led_rj45_yellow_5v: IC2.6 (2Y), J3.6 (Pin_6)
- new net usb_5v: J2.7 (Pin_7)
- new net ws2812_data_1: D3.4 (DIN), IC1.3 (1Y)
- new net ws2812_data_2: D6.2 (DOUT), J3.8 (Pin_8)
- no-connect marks 32 -> 45
Other:
- note added: "GND DIN pin is NC"
- note added: "MAIN TOP add test points double-check"
- note added: "audio"
- note added: "buttons"
- note added: "led+midi"
- note added: "oled"
- note added: "power nets: - gnd - 3v3 - sys_5v - usb_5v - agnd - a3v3"
- note added: "pwr+usb"
- note added: "to bottom"
- note added: "ws2812b flow: teensy3v3 > 125n >_1-> onboard leds >_2>tobottom"
- note removed: "encoder"
- moved on the sheet: C1, C10, C11, C12, C13, C14, C15, C17, C18, C19, C2, C20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
