File: CAD/bommanoid/bommanoid01/cab.kicad_sch (KiCad schematic)
At the start: 0 parts

Commit message: progress on bommanoid pcb design adding some winisd simulations
Parts:
- added D23, D24: LED, LED_THT:LED_D5.0mm, symbol Device:LED
- added H13, H14: MountingHole_Pad, MountingHole:MountingHole_3.2mm_M3, symbol Mechanical:MountingHole_Pad
- added J27: Amphenol ACJS-MHOM, SamacSys_Parts:ACJSMHOM, symbol clarinoid2:Amphenol ACJS-MHOM
- added J28: Conn_02x10_Odd_Even, Connector_PinHeader_2.54mm:PinHeader_2x14_P2.54mm_Vertical, symbol Connector_Generic:Conn_02x14_Odd_Even
- added J29, J30: RJ45_LED_Shielded, Connector_RJ:RJ45_Amphenol_RJHSE538X, symbol Connector:RJ45_LED_Shielded
- added R32, R33, R34, R35, R36, R37: R, Resistor_THT:R_Axial_DIN0207_L6.3mm_D2.5mm_P10.16mm_Horizontal, symbol Device:R
Connections:
- new net: J30.11, R36.2
- new net: D23.1 (K), R34.1
- new net: J30.9, R35.2
- new net: J29.11, R33.2
- new net: J29.9, R32.2
- new net: D24.1 (K), R37.1
- new net agnd: J27.3 (S_1), J27.4 (S_2), J28.26 (Pin_26), J28.28 (Pin_28)
- new net aleft: J27.6 (T), J28.27 (Pin_27)
- new net amp_5v: J28.11 (Pin_11), J28.7 (Pin_7), J28.9 (Pin_9), J29.8, J30.8
- new net aright: J27.5 (R), J28.25 (Pin_25)
- new net gnd: H13.1, H14.1, J28.10 (Pin_10), J28.12 (Pin_12), J28.14 (Pin_14), J28.16 (Pin_16), J28.18 (Pin_18), J28.2 (Pin_2), J28.20 (Pin_20), J28.22 (Pin_22), J28.4 (Pin_4), J28.6 (Pin_6), J28.8 (Pin_8), J29.1, J29.SH, J30.1, J30.SH, R32.1, R33.1, R34.2, R35.1, R36.1, R37.2
- new net led_act1_5v: J28.17 (Pin_17), J29.12, J29.5, J30.5
- new net led_act2_5v: J28.19 (Pin_19), J29.6, J30.10, J30.6
- new net led_act3_5v: J28.21 (Pin_21), J29.7, J30.12, J30.7
- new net led_blink_5v: J28.15 (Pin_15), J29.10, J29.4, J30.4
- new net powerbank_5v: J28.1 (Pin_1), J28.3 (Pin_3), J28.5 (Pin_5)
- new net sys_5v: D23.2 (A), D24.2 (A), J28.13 (Pin_13), J29.2, J30.2
- new net ws2812_data_a: J28.23 (Pin_23), J29.3
- new net ws2812_data_b: J28.24 (Pin_24), J30.3
- no-connect marks 0 -> 2
Other:
- note added: "<-- for relay"
- note added: "<-- requires jumper if no case ws2812 leds"
- note added: "<-- toggle switch output then to LED and relay"
- note added: "RJ45 in"
- note added: "RJ45 thru"
- note added: "WIRE"
- note added: "audio in"
- note added: "under lighting"
- note added: "ws2812 flow A (case) => B (bell)"
