File: CAD/bommanoid/bommanoid01/clarinoid-devboard.kicad_pcb (KiCad board)
At the start: 2 copper layers, 1273.3 x 654.2 mm, 356 parts, among them J1 AudioOut, J1 header_i2c, J10 MIDI IN, J11 MIDI OUT, J12 SSD1306, J13 captouch 3x3x1 header B, J2 AudioOut, J2 XKB_U262-16XN-4BVC11 USB-C re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, J20 CapTouchSlider_3x3x1, J3 microSD SOFNG TF-15x15, J38 microSD SOFNG TF-15x15, J39 Conn_01x20 MANUAL, J4 MIDI IN, J40 Conn_01x08 MANUAL, J45 female 1x6, J5 MIDI OUT, J5 header_i2c, J6 XKB_U262-16XN-4BVC11 USB-C re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, J6 female 1x6, J7 SSD1306, SW1 SW_Push, SW2 RotaryEncoder_Switch_ABC12, SW6 SW_Push, U1 PCM5102A, U12 ssd1306_graphic, U19 TLV75733PDBV, U2 TLV75733PDBV, U21 mb1, U22 mb1, U23 mb1, U24 mb1, U26 mb1, U27 mb1, U3 TLV75733PDBV, U30 mb1, U32 mb1, U40 APCI0108-P001A Teensy_4.0_Mic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, U41 Micromod outline, U43 processor board template, U49 mb1, U5 main captouch graphic, U5 processor board template, U53 mb1, U54 mb1, U55 mb1, U6 Micromod outline, U60 mb1, U65 mb1, U7 6N138, U7 TLV75733PDBV, U8 6N138, U8 ssd1306_graphic, U9 captouch3x3x1 graphic

Commit message: progress on bommanoid pcb design adding some winisd simulations
Parts:
- removed the C17 at (418.6, 71.2)
- removed the C17 at (342.4, 431.5)
- removed the C20 at (420.7, 71.2)
- removed the C21 at (422.8, 71.2)
- removed the C21 at (353.2, 462.2)
- removed the C22 at (357.6, 465.2)
- removed the C22 at (424.9, 71.2)
- removed the C23 at (427.0, 71.2)
- removed the C23 at (357.6, 462.2)
- removed the D5 at (384.7, 96.4)
- removed the D5 at (270.1, 470.6)
- removed the D7 at (383.1, 96.4)
- removed the D7 at (278.5, 464.0)
- removed the D8 at (270.1, 477.3)
- removed the D8 at (381.5, 96.4)
- removed the D9 at (379.9, 96.4)
- removed the D9 at (281.9, 471.9)
- removed the H1 at (336.4, 426.3)
- removed the H1 at (374.1, -50.1)
- removed the H2 at (358.1, -114.1)
- removed the H2 at (305.2, 436.2)
- removed the H5 at (171.3, -36.9)
- removed the H5 at (77.1, -27.3)
- removed the H5 at (126.3, -144.6)
- removed the H5 at (349.1, -129.1)
- removed the H5 at (-602.2, 322.1)
- removed the J** at (12.8, 375.4)
- removed the J** at (380.4, -66.8)
- removed the J** at (338.4, -66.8)
- removed the J** at (359.4, -66.8)
- removed the J1 at (298.9, 434.5)
- removed the J1 at (336.2, 27.4)
- removed the J2 at (275.6, 450.5)
- removed the J2 at (436.1, -80.1)
- removed J38: microSD SOFNG TF-15x15, clarinoid2:SOFNG TF-15x15 (LCSC C111196)
- removed J39: Conn_01x20 MANUAL, Connector_PinHeader_2.54mm:PinHeader_1x20_P2.54mm_Vertical
- removed J40: Conn_01x08 MANUAL, Connector_PinHeader_2.54mm:PinHeader_1x08_P2.54mm_Vertical
- removed J45: female 1x6, Connector_PinSocket_2.54mm:PinSocket_1x06_P2.54mm_Vertical
- removed the J5 at (341.5, 63.3)
- removed the J5 at (306.4, 427.4)
- removed the J6 at (425.4, 414.6)
- removed the J6 at (451.0, 8.85)
- removed the R13 at (304.0, 441.8)
- removed the R13 at (159.1, -62.1)
- removed the R15 at (525.3, 163.7)
- removed the R15 at (432.6, 391.1)
- removed the R20 at (291.1, 462.4)
- removed the R20 at (326.5, 8.40)
- removed the R21 at (326.5, 10.8)
- removed the R21 at (268.6, 485.5)
- removed the R8 at (433.9, -71.1)
- removed the REF** at (414.7, -76.0)
- removed the REF** at (-600.2, 336.1)
- removed the REF** at (-579.2, 335.1)
- removed the REF** at (-579.2, 443.1)
- removed the REF** at (-614.2, 311.1)
- removed the REF** at (-583.2, 335.1)
- removed the REF** at (-575.2, 335.1)
- removed the REF** at (-587.2, 335.1)
- removed SW2: RotaryEncoder_Switch_ABC12, clarinoid2:Bourns_ENC_PEC11R-4215F-S0024
- removed TP1, TP6: D3v3, TestPoint:TestPoint_THTPad_D2.0mm_Drill1.0mm
- removed TP2: A3v3, TestPoint:TestPoint_THTPad_D2.0mm_Drill1.0mm
- removed TP3 (x2): AGND, TestPoint:TestPoint_THTPad_D2.0mm_Drill1.0mm
- removed the U12 at (469.9, -125.1)
- removed U21, U22, U23, U24, U26, U27, U30, U32, U49, U53, U54, U55, U60, U65: mb1, clarinoid2:mouse-bite-2mm-slot
- removed the U40 at (390.8, -123.1)
- removed the U41 at (386.6, -125.8)
- removed U43: processor board template, clarinoid2:dev board processor subboard template
- removed the U5 at (270.1, 393.6)
- removed the U5 at (451.0, 8.85)
- removed U9: captouch3x3x1 graphic, CapTouchSliders:captouch dev board subboard template
- added C17: 1uF, Capacitor_SMD:C_0805_2012Metric, F.Cu at (415.6, 781.0)
- added C21: 22uF, Capacitor_SMD:C_0805_2012Metric, F.Cu at (431.2, 775.0)
- added C22: 22uF, Capacitor_SMD:C_0805_2012Metric, F.Cu at (431.2, 784.1)
- added C23: 22uF, Capacitor_SMD:C_0805_2012Metric, F.Cu at (435.6, 778.1)
- added C26: 10uF, Capacitor_SMD:C_1206_3216Metric, F.Cu at (447.6, 737.4)
- added C27: 22uF, Capacitor_SMD:C_1206_3216Metric, F.Cu at (459.6, 722.6)
- added C29: 22uF, Capacitor_SMD:C_1206_3216Metric, F.Cu at (441.9, 737.4)
- added C30: 22uF, Capacitor_SMD:C_1206_3216Metric, F.Cu at (450.4, 729.3)
- added C31: 22uF, Capacitor_SMD:C_0603_1608Metric, F.Cu at (446.7, 740.3)
- added C32: 22uF, Capacitor_SMD:C_0603_1608Metric, F.Cu at (445.1, 743.7)
- added C33: 0.1uF, Capacitor_SMD:C_1206_3216Metric, F.Cu at (456.0, 729.1)
- added D17: 25%, LED_SMD:LED_0805_2012Metric, F.Cu at (435.7, 781.1)
- added D18: 50%, LED_SMD:LED_0805_2012Metric, F.Cu at (440.1, 778.0)
- added D19: 75%, LED_SMD:LED_0805_2012Metric, F.Cu at (435.7, 775.0)
- added D20: 100%, LED_SMD:LED_0805_2012Metric, F.Cu at (431.2, 781.1)
- added D21: LED, LED_THT:LED_D5.0mm, F.Cu at (526.4, 709.5)
- added D22: LED, LED_THT:LED_D5.0mm, F.Cu at (557.0, 698.9)
- added D23: LED, LED_THT:LED_D5.0mm, F.Cu at (539.0, 742.9)
- added D24: LED, LED_THT:LED_D5.0mm, F.Cu at (531.0, 750.8)
- added D25: LED, LED_THT:LED_D5.0mm, F.Cu at (544.4, 772.1)
- added D26: LED, LED_THT:LED_D5.0mm, F.Cu at (539.3, 788.1)
- added D27: WS2812B, LED_SMD:LED_WS2812B_PLCC4_5.0x5.0mm_P3.2mm, F.Cu at (393.1, 691.1)
- added D28: WS2812B, LED_SMD:LED_WS2812B_PLCC4_5.0x5.0mm_P3.2mm, F.Cu at (409.9, 697.7)
- added D29: LED, LED_THT:LED_D5.0mm, F.Cu at (531.8, 789.9)
- added D30: LED, LED_THT:LED_D5.0mm, F.Cu at (545.1, 779.6)
- added D31: WS2812B, LED_SMD:LED_WS2812B_PLCC4_5.0x5.0mm_P3.2mm, F.Cu at (401.5, 691.1)
- added D32: LED, LED_THT:LED_D5.0mm, F.Cu at (557.7, 768.0)
- added D33: WS2812B, LED_SMD:LED_WS2812B_PLCC4_5.0x5.0mm_P3.2mm, F.Cu at (418.4, 697.7)
- added D34: LED, LED_THT:LED_D5.0mm, F.Cu at (552.6, 775.6)
- added D35: WS2812B, LED_SMD:LED_WS2812B_PLCC4_5.0x5.0mm_P3.2mm, F.Cu at (401.5, 697.7)
- added D36: WS2812B, LED_SMD:LED_WS2812B_PLCC4_5.0x5.0mm_P3.2mm, F.Cu at (418.4, 691.1)
- added D37: WS2812B, LED_SMD:LED_WS2812B_PLCC4_5.0x5.0mm_P3.2mm, F.Cu at (409.9, 691.1)
- added D38: WS2812B, LED_SMD:LED_WS2812B_PLCC4_5.0x5.0mm_P3.2mm, F.Cu at (393.1, 697.7)
- added D5: WS2812B, LED_SMD:LED_WS2812B_PLCC4_5.0x5.0mm_P3.2mm, F.Cu at (404.7, 776.8)
- added D7: LED, LED_THT:LED_D5.0mm, F.Cu at (672.1, 692.4)
- added D8: LED, LED_THT:LED_D5.0mm, F.Cu at (680.8, 676.7)
- added D9: LED, LED_THT:LED_D5.0mm, F.Cu at (656.5, 712.1)
- added DS**: Kingbright PDC54, clarinoid2:Kingbright PDC54 template, F.Cu at (-278.6, 326.2)
- added H1: M.2 riser 2.5mm, clarinoid2:Sinhoo SMTSO2530CTJ, F.Cu at (381.8, 800.4)
- added H10: MountingHole_Pad, MountingHole:MountingHole_3.2mm_M3, F.Cu at (520.0, 709.7)
- added H11: MountingHole_Pad, MountingHole:MountingHole_3.2mm_M3, F.Cu at (538.6, 705.7)
- added H12: MountingHole_Pad, MountingHole:MountingHole_3.2mm_M3, F.Cu at (512.0, 709.7)
- added H13: MountingHole_Pad, MountingHole:MountingHole_3.2mm_M3, F.Cu at (560.4, 721.2)
- added H14: MountingHole_Pad, MountingHole:MountingHole_3.2mm_M3, F.Cu at (532.5, 743.1)
- added H15: MountingHole_Pad, MountingHole:MountingHole_3.2mm_M3, F.Cu at (538.6, 780.4)
- added H16: MountingHole_Pad, MountingHole:MountingHole_3.2mm_M3, F.Cu at (525.3, 790.1)
- added H2: MountingHole_Pad, MountingHole:MountingHole_3.2mm_M3, F.Cu at (636.8, 734.8)
- added H5: MountingHole, MountingHole:MountingHole_3.2mm_M3_Pad_Via, F.Cu at (-590.7, 330.6)
- added H5: MountingHole_Pad, MountingHole:MountingHole_3.2mm_M3, F.Cu at (663.8, 696.8)
- added H5: MountingHole, MountingHole:MountingHole_3.2mm_M3_Pad_Via, F.Cu at (-590.7, 437.1)
- added H5: MountingHole, MountingHole:MountingHole_3.2mm_M3_Pad_Via, F.Cu at (-608.2, 315.1)
- added H6: MountingHole_Pad, MountingHole:MountingHole_3.2mm_M3, F.Cu at (650.5, 700.8)
- added H7: MountingHole_Pad, MountingHole:MountingHole_3.2mm_M3, F.Cu at (637.1, 715.0)
- added H8: MountingHole_Pad, MountingHole:MountingHole_3.2mm_M3, F.Cu at (709.2, 676.9)
- added IC1: SN74AHCT125N, SamacSys_Parts:DIP794W53P254L1930H508Q14N, F.Cu at (395.0, 805.4)
- added IC2: SN74AHCT125N, SamacSys_Parts:DIP794W53P254L1930H508Q14N, F.Cu at (395.0, 784.1)
- added IC3: Injoinic IP5306 battery charge, clarinoid2:SOIC127P599X155-9N (IP5306), F.Cu at (452.5, 724.2)
- added J1: Conn_01x07, Connector_PinHeader_2.54mm:PinHeader_1x07_P2.54mm_Vertical, F.Cu at (625.8, 725.2)
- added J14: Amphenol ACJS-MHOM, SamacSys_Parts:ACJSMHOM, F.Cu at (356.5, 736.1)
- added J15: Conn_01x12, Connector_PinSocket_2.54mm:PinSocket_1x12_P2.54mm_Vertical, F.Cu at (611.9, 675.3)
- added J16: Conn_01x12, Connector_PinSocket_2.54mm:PinSocket_1x12_P2.54mm_Vertical, F.Cu at (616.5, 675.3)
- added J17: RJ45_LED_Shielded, Connector_RJ:RJ45_Amphenol_RJHSE538X, F.Cu at (637.3, 682.0)
- added J18: Conn_01x03, Connector_PinSocket_2.54mm:PinSocket_1x03_P2.54mm_Vertical, F.Cu at (667.3, 683.4)
- added J19: Conn_01x07, Connector_PinSocket_2.54mm:PinSocket_1x07_P2.54mm_Vertical, F.Cu at (662.7, 675.3)
- added J2: Conn_01x07, Connector_PinHeader_2.54mm:PinHeader_1x07_P2.54mm_Vertical, F.Cu at (621.2, 725.2)
- added J21: Conn_01x05, Connector_PinSocket_2.54mm:PinSocket_1x05_P2.54mm_Vertical, F.Cu at (703.0, 675.3)
- added J22: Conn_01x08, Connector_JST:JST_PH_B8B-PH-K_1x08_P2.00mm_Vertical, F.Cu at (533.0, 697.9)
- added J23: Conn_01x05, Connector_PinSocket_2.54mm:PinSocket_1x05_P2.54mm_Vertical, F.Cu at (600.7, 675.3)
- added J24: Conn_01x05, Connector_PinSocket_2.54mm:PinSocket_1x05_P2.54mm_Vertical, F.Cu at (552.3, 697.7)
- added J25: Conn_01x09, Connector_JST:JST_PH_B9B-PH-K_1x09_P2.00mm_Vertical, F.Cu at (511.0, 697.9)
- added J26: Conn_02x06_Odd_Even, Connector_PinHeader_2.54mm:PinHeader_2x08_P2.54mm_Vertical, F.Cu at (593.5, 675.3)
- added J27: Amphenol ACJS-MHOM, SamacSys_Parts:ACJSMHOM, F.Cu at (352.7, 702.9)
- added J28: Conn_02x10_Odd_Even, Connector_PinHeader_2.54mm:PinHeader_2x14_P2.54mm_Vertical, F.Cu at (510.4, 719.6)
- added J29: RJ45_LED_Shielded, Connector_RJ:RJ45_Amphenol_RJHSE538X, F.Cu at (542.6, 726.3)
- added J30: RJ45_LED_Shielded, Connector_RJ:RJ45_Amphenol_RJHSE538X, F.Cu at (522.0, 726.3)
- added J31: RJ45_LED_Shielded, Connector_RJ:RJ45_Amphenol_RJHSE538X, F.Cu at (514.8, 773.3)
- added J5: Conn_01x03, Connector_PinHeader_2.54mm:PinHeader_1x03_P2.54mm_Vertical, F.Cu at (630.5, 725.2)
- added J6: XKB_U262-16XN-4BVC11 USB-C recept, clarinoid2:USB_C_Receptacle_XKB_U262-16XN-4BVC11, F.Cu at (353.8, 763.9)
- added J8: Conn_01x08, Connector_PinSocket_2.54mm:PinSocket_1x08_P2.54mm_Vertical, F.Cu at (628.3, 675.3)
- added J9: Conn_02x04_Odd_Even, Connector_PinHeader_2.54mm:PinHeader_2x07_P2.54mm_Vertical, F.Cu at (628.3, 697.7)
- added L1: 1uH-psa, clarinoid2:Inductor_MCS0630-1R0MN2, F.Cu at (443.3, 735.0)
- added R13: 47R, Resistor_SMD:R_1206_3216Metric, F.Cu at (384.4, 805.8)
- added R15: R, Resistor_THT:R_Axial_DIN0207_L6.3mm_D2.5mm_P10.16mm_Horizontal, F.Cu at (634.7, 709.0)
- added R20: R, Resistor_THT:R_Axial_DIN0207_L6.3mm_D2.5mm_P10.16mm_Horizontal, F.Cu at (611.1, 707.5)
- added R21: R, Resistor_THT:R_Axial_DIN0207_L6.3mm_D2.5mm_P10.16mm_Horizontal, F.Cu at (648.1, 694.8)
- added R27: 2R, Resistor_SMD:R_0603_1608Metric, F.Cu at (464.4, 722.2)
- added R28: 10k, Resistor_SMD:R_0603_1608Metric, F.Cu at (441.1, 743.7)
- added R29: 0.5R, Resistor_SMD:R_0603_1608Metric, F.Cu at (452.4, 735.5)
- added R30: R, Resistor_THT:R_Axial_DIN0207_L6.3mm_D2.5mm_P10.16mm_Horizontal, F.Cu at (522.9, 703.7)
- added R31: R, Resistor_THT:R_Axial_DIN0207_L6.3mm_D2.5mm_P10.16mm_Horizontal, F.Cu at (509.6, 703.7)
- added R32: R, Resistor_THT:R_Axial_DIN0207_L6.3mm_D2.5mm_P10.16mm_Horizontal, F.Cu at (516.8, 745.2)
- added R33: R, Resistor_THT:R_Axial_DIN0207_L6.3mm_D2.5mm_P10.16mm_Horizontal, F.Cu at (516.8, 741.1)
- added R38: R, Resistor_THT:R_Axial_DIN0207_L6.3mm_D2.5mm_P10.16mm_Horizontal, F.Cu at (509.6, 784.1)
- added R39: R, Resistor_THT:R_Axial_DIN0207_L6.3mm_D2.5mm_P10.16mm_Horizontal, F.Cu at (509.6, 788.1)
- added R42: R, Resistor_THT:R_Axial_DIN0207_L6.3mm_D2.5mm_P10.16mm_Horizontal, F.Cu at (530.2, 766.3)
- added R43: R, Resistor_THT:R_Axial_DIN0207_L6.3mm_D2.5mm_P10.16mm_Horizontal, F.Cu at (530.2, 770.3)
- added R44: R, Resistor_THT:R_Axial_DIN0207_L6.3mm_D2.5mm_P10.16mm_Horizontal, F.Cu at (509.6, 792.2)
- added R45: R, Resistor_THT:R_Axial_DIN0207_L6.3mm_D2.5mm_P10.16mm_Horizontal, F.Cu at (530.2, 774.4)
- added R6: 4.7k, Resistor_SMD:R_1206_3216Metric, F.Cu at (383.6, 809.1)
- added R9: R, Resistor_THT:R_Axial_DIN0207_L6.3mm_D2.5mm_P10.16mm_Horizontal, F.Cu at (611.1, 711.6)
- added REF**: DIP-14_W7.62mm, Package_DIP:DIP-14_W7.62mm, F.Cu at (-299.9, 310.1)
- added REF**: PinHeader_1x03_P2.54mm_Vertical, Connector_PinHeader_2.54mm:PinHeader_1x03_P2.54mm_Vertical, F.Cu at (-5.38, 389.1)
- added REF**: PinHeader_1x05_P2.54mm_Vertical, Connector_PinHeader_2.54mm:PinHeader_1x05_P2.54mm_Vertical, F.Cu at (-599.2, 336.6)
- added REF**: PinHeader_1x05_P2.54mm_Vertical, Connector_PinHeader_2.54mm:PinHeader_1x05_P2.54mm_Vertical, F.Cu at (-614.2, 322.5)
- added REF**: PinHeader_1x03_P2.54mm_Vertical, Connector_PinHeader_2.54mm:PinHeader_1x03_P2.54mm_Vertical, F.Cu at (-4.91, 341.6)
- added REF**: PinHeader_2x06_P2.54mm_Vertical, Connector_PinHeader_2.54mm:PinHeader_2x06_P2.54mm_Vertical, F.Cu at (-584.7, 445.1)
- added U5: MCP23017_SP, Package_DIP:DIP-28_W7.62mm, F.Cu at (349.5, 775.6)
- BT1: footprint Battery:BatteryHolder_Keystone_1042_1x18650 -> clarinoid2:KEYSTONE_1043
- C16: value 0.1uF -> 10uF; footprint Capacitor_SMD:C_0805_2012Metric -> Capacitor_SMD:C_1206_3216Metric
- C28: value 0.1uF -> 22uF; footprint Capacitor_SMD:C_0805_2012Metric -> Capacitor_SMD:C_1206_3216Metric
- D10, D13, D14: value blue -> LED; footprint LED_SMD:LED_0603_1608Metric -> LED_THT:LED_D5.0mm
- D11, D12, D15: value green -> LED; footprint LED_SMD:LED_0603_1608Metric -> LED_THT:LED_D5.0mm
- D16: value green -> korgpwr; footprint LED_SMD:LED_0603_1608Metric -> LED_SMD:LED_0805_2012Metric
- D4, D6: value green -> WS2812B; footprint LED_SMD:LED_0603_1608Metric -> LED_SMD:LED_WS2812B_PLCC4_5.0x5.0mm_P3.2mm
- H3: value MountingHole -> MountingHole_Pad; footprint MountingHole:MountingHole_3.2mm_M3_Pad_Via -> MountingHole:MountingHole_3.2mm_M3
- H4: value M.2 riser 2.5mm -> MountingHole_Pad; footprint clarinoid2:Sinhoo SMTSO2530CTJ -> MountingHole:MountingHole_3.2mm_M3
- H9: value MountingHole -> MountingHole_Pad
- J10: value MIDI IN -> Conn_01x07; footprint clarinoid2:SWITCHCRAFT_35RAPC4BV4_OvalHoles -> Connector_PinSocket_2.54mm:PinSocket_1x07_P2.54mm_Vertical
- J11: value MIDI OUT -> Amphenol ACJS-MHOM; footprint clarinoid2:SWITCHCRAFT_35RAPC4BV4_OvalHoles -> SamacSys_Parts:ACJSMHOM
- J12: value SSD1306 -> Amphenol ACJS-MHOM; footprint Connector_PinSocket_2.54mm:PinSocket_1x07_P2.54mm_Vertical -> SamacSys_Parts:ACJSMHOM
- J13: value captouch 3x3x1 header B -> Conn_01x07; footprint Connector_PinHeader_2.54mm:PinHeader_1x06_P2.54mm_Vertical -> Connector_PinSocket_2.54mm:PinSocket_1x07_P2.54mm_Vertical
- J20: value CapTouchSlider_3x3x1 -> Conn_01x07; footprint CapTouchSliders:CaptouchSlider_Masked_H3x3_A1.0mm_x12 -> Connector_PinSocket_2.54mm:PinSocket_1x07_P2.54mm_Vertical; moved to F.Cu
- J3: value microSD SOFNG TF-15x15 -> Conn_01x12; footprint clarinoid2:SOFNG TF-15x15 (LCSC C111196) -> Connector_PinHeader_2.54mm:PinHeader_1x12_P2.54mm_Vertical
- J4: value MIDI IN -> Conn_01x12; footprint clarinoid2:SWITCHCRAFT_35RAPC4BV4_OvalHoles -> Connector_PinHeader_2.54mm:PinHeader_1x12_P2.54mm_Vertical
- J7: value SSD1306 -> Conn_02x10_Odd_Even; footprint Connector_PinSocket_2.54mm:PinSocket_1x07_P2.54mm_Vertical -> Connector_PinHeader_2.54mm:PinHeader_2x10_P2.54mm_Vertical
- R16, R17, R18, R19, R22, R23, R24, R34, R35, R36, R37: value 470R -> R; footprint Resistor_SMD:R_1206_3216Metric -> Resistor_THT:R_Axial_DIN0207_L6.3mm_D2.5mm_P10.16mm_Horizontal
- R25: value 470R -> 5.1k
- R40, R41: value 4.7k -> R; footprint Resistor_SMD:R_1206_3216Metric -> Resistor_THT:R_Axial_DIN0207_L6.3mm_D2.5mm_P10.16mm_Horizontal
- R7: value 5.1k -> 4.7k; moved to F.Cu
- moved H4 897.4 mm to (644.7, 726.9)
- moved R7 886.4 mm to (367.6, 812.4), turned to 0 degrees
- moved J12 863.8 mm to (392.3, 736.1), turned to 0 degrees
- moved H3 860.0 mm to (636.8, 726.9)
- moved BT1 855.7 mm to (549.6, 684.1)
- moved R40 745.2 mm to (522.9, 784.1)
- moved R41 731.0 mm to (543.5, 766.3)
- moved J11 715.7 mm to (356.5, 754.9)
- moved J10 701.8 mm to (658.1, 675.3)
- moved J20 682.5 mm to (698.4, 675.3), turned to 0 degrees
- moved R36 676.7 mm to (509.6, 756.9), turned to 0 degrees
- moved R37 671.0 mm to (516.8, 749.2), turned to 0 degrees
- moved R35 661.0 mm to (530.1, 737.1), turned to 0 degrees
- moved R34 657.7 mm to (516.8, 737.1), turned to 0 degrees
- moved J13 596.1 mm to (653.5, 675.3), turned to 0 degrees
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Connections:
- net /bommanoid_batt_bottom/5v regulated renamed /bommanoid_batt_bottom/sys_5v
- BT1 pad 1: /power_battery/battery + 5v -> /bommanoid_batt_bottom/batt+
- BT1 pad 2: /power_battery/gnd -> /bommanoid_batt_bottom/gnd
- C1 pad 1: /bommanoid_main_top/+3.3v regulator output -> /bommanoid_main_top/3v3
- C1 pad 2: /bommanoid_main_top/gnd from processor -> /bommanoid_main_top/gnd
- C10 pad 1: /bommanoid_main_top/gnd from processor -> /bommanoid_main_top/gnd
- C10 pad 2: D3v3 -> /bommanoid_main_top/d3v3
- C11 pad 1: A3v3 -> /bommanoid_main_top/a3v3
- C11 pad 2: AGND -> /bommanoid_main_top/agnd
- C12 pad 1: A3v3 -> /bommanoid_main_top/a3v3
- C12 pad 2: AGND -> /bommanoid_main_top/agnd
- C13 pad 1: /bommanoid_main_top/5v input -> /bommanoid_main_top/sys_5v
- C14 pad 1: /bommanoid_main_top/5v input -> /bommanoid_main_top/sys_5v
- C15 pad 1: /bommanoid_main_top/5v input -> /bommanoid_main_top/sys_5v
- C16 pad 1: /bommanoid_main_top/+3.3v regulator output -> Net-(C16-Pad1)
- C16 pad 2: /bommanoid_main_top/gnd -> /bommanoid_batt_top/gnd
- C18 pad 1: /bommanoid_main_top/+3.3v regulator output -> /bommanoid_main_top/3v3
- C19 pad 1: /bommanoid_main_top/+3.3v regulator output -> /bommanoid_main_top/3v3
- C2 pad 1: /bommanoid_main_top/+3.3v regulator output -> /bommanoid_main_top/3v3
- C2 pad 2: /bommanoid_main_top/gnd from processor -> /bommanoid_main_top/gnd
- C20 pad 1: /bommanoid_main_top/5v from processor -> /bommanoid_main_top/sys_5v
- C20 pad 2: /bommanoid_main_top/gnd from processor -> /bommanoid_main_top/gnd
- C28 pad 1: /processor_mm/+3.3v regulator output -> /bommanoid_batt_top/charger output +5v
- C28 pad 2: /processor_mm/gnd -> /bommanoid_batt_top/gnd
- C5 pad 1: dac output L -> /bommanoid_main_top/aleft
- C5 pad 2: AGND -> /bommanoid_main_top/agnd
- C6 pad 2: /bommanoid_main_top/gnd from processor -> /bommanoid_main_top/gnd
- C7 pad 1: /bommanoid_main_top/gnd from processor -> /bommanoid_main_top/gnd
- C7 pad 2: D3v3 -> /bommanoid_main_top/d3v3
- C8 pad 1: dac output R -> /bommanoid_main_top/aright
- C8 pad 2: AGND -> /bommanoid_main_top/agnd
- C9 pad 2: /bommanoid_main_top/gnd from processor -> /bommanoid_main_top/gnd
- D10 pad 2: /bommanoid_batt_top/GEN_LED2 -> /bommanoid_main_bottom/led_blink_5v
- D11 pad 2: /bommanoid_batt_top/GEN_LED3 -> /bommanoid_main_bottom/led_act1_5v
- D12 pad 2: /bommanoid_batt_top/GEN_LED4 -> /bommanoid_main_bottom/led_act2_5v
- D13 pad 2: /bommanoid_batt_top/GEN_LED1 -> /bommanoid_main_bottom/led_act3_5v
- D14 pad 2: /bommanoid_batt_top/GEN_LED2 -> /bommanoid_main_bottom/sys_5v
- D15 pad 2: /bommanoid_batt_top/GEN_LED3 -> /bommanoid_main_bottom/sys_5v
- D16 pad 1: Net-(D16-Pad1) -> /bommanoid_batt_top/korg_power_led_cathode
- D16 pad 2: /bommanoid_batt_top/GEN_LED4 -> /bommanoid_batt_top/korg_power_led_anode
- D2 pad 2: Net-(D2-Pad2) -> /bommanoid_main_top/midi_in_tip
- D3 pad 1: unconnected-(D3-Pad1) -> /bommanoid_main_top/sys_5v
- D3 pad 2: unconnected-(D3-Pad2) -> Net-(D3-Pad2)
- D3 pad 3: unconnected-(D3-Pad3) -> /bommanoid_main_top/gnd
- D3 pad 4: unconnected-(D3-Pad4) -> /bommanoid_main_top/ws2812_data_1
- D4 pad 1: Net-(D4-Pad1) -> /bommanoid_main_top/sys_5v
- D4 pad 2: /bommanoid_batt_top/GEN_LED4 -> Net-(D4-Pad2)
- D6 pad 1: Net-(D6-Pad1) -> /bommanoid_main_top/sys_5v
- D6 pad 2: /bommanoid_batt_top/GEN_LED4 -> /bommanoid_main_top/ws2812_data_2
- J10 pad 1: unconnected-(J10-Pad1) -> /bommanoid_main_bottom/gnd
- J10 pad 2: Net-(D6-Pad2) -> /bommanoid_main_bottom/3v3
- J10 pad 3: unconnected-(J10-Pad3) -> /bommanoid_main_bottom/oled_sck
- J10 pad 4: Net-(J10-Pad4) -> /bommanoid_main_bottom/oled_data
- J10 pad 5: unconnected-(J10-Pad5) -> /bommanoid_main_bottom/oled_rst
- J11 pad 1: /gnd from processor -> unconnected-(J11-Pad1)
- J11 pad 2: Net-(J11-Pad2) -> unconnected-(J11-Pad2)
- J11 pad 3: unconnected-(J11-Pad3) -> /bommanoid_main_bottom/gnd
- J11 pad 4: Net-(J11-Pad4) -> /bommanoid_main_bottom/gnd
- J11 pad 5: unconnected-(J11-Pad5) -> /bommanoid_main_bottom/midi_out_ring
- J12 pad 1: /gnd from processor -> unconnected-(J12-Pad1)
- J12 pad 2: /+3.3v regulator output -> unconnected-(J12-Pad2)
- J12 pad 3: /SPI0_SCK -> /bommanoid_main_bottom/agnd
- J12 pad 4: /SPI0_MOSI -> /bommanoid_main_bottom/agnd
- J12 pad 5: /OLED_RES -> /bommanoid_main_bottom/aright_post_pot
- J12 pad 6: /OLED_DC -> /bommanoid_main_bottom/aleft_post_pot
- J13 pad 1: Net-(J13-Pad1) -> /bommanoid_main_bottom/gnd
- J13 pad 2: Net-(J13-Pad2) -> /bommanoid_main_bottom/prg
- J13 pad 3: Net-(J13-Pad3) -> /bommanoid_main_bottom/sys_5v
- J13 pad 4: Net-(J13-Pad4) -> /bommanoid_main_bottom/3v3
- J13 pad 5: Net-(J13-Pad5) -> /bommanoid_main_bottom/usb_data_+
- J13 pad 6: Net-(J13-Pad6) -> /bommanoid_main_bottom/usb_data_-
- J20 pad 1: /captouch 3x3x1 GND -> /bommanoid_batt_top/gnd
- J20 pad 2: Net-(J20-Pad2) -> /bommanoid_batt_top/batt+
- J20 pad 3: Net-(J20-Pad3) -> /bommanoid_batt_top/usb_5v
- J20 pad 4: Net-(J20-Pad4) -> /bommanoid_batt_top/charger output +5v
- J20 pad 5: Net-(J20-Pad5) -> /bommanoid_batt_top/key
- J20 pad 6: Net-(J20-Pad6) -> (no net)
- J20 pad 7: Net-(J13-Pad1) -> (no net)
- J3 pad 1: /bommanoid_main_top/SDIO_DAT2 -> /bommanoid_main_top/gnd
- J3 pad 2: /bommanoid_main_top/SDIO_CS -> /bommanoid_main_top/led_blink_5v
- J3 pad 3: /bommanoid_main_top/SDIO_MOSI -> /bommanoid_main_top/led_act1_5v
- J3 pad 4: /bommanoid_main_top/+3.3v regulator output -> /bommanoid_main_top/led_act2_5v
- J3 pad 5: /bommanoid_main_top/SDIO_CLOCK -> /bommanoid_main_top/led_act3_5v
- J3 pad 6: /bommanoid_main_top/gnd -> /bommanoid_main_top/led_rj45_yellow_5v
- J3 pad 7: /bommanoid_main_top/SDIO_MISO -> /bommanoid_main_top/led_rj45_green_5v
- J3 pad 8: /bommanoid_main_top/sdio_dat1 -> /bommanoid_main_top/ws2812_data_2
- J4 pad 1: unconnected-(J4-Pad1) -> /bommanoid_main_top/gnd
- J4 pad 2: Net-(D2-Pad2) -> /bommanoid_main_top/btn_x1
- J4 pad 3: unconnected-(J4-Pad3) -> /bommanoid_main_top/btn_x2
- J4 pad 4: Net-(J4-Pad4) -> /bommanoid_main_top/btn_x3
- J4 pad 5: unconnected-(J4-Pad5) -> /bommanoid_main_top/btn_x4
- J7 pad 1: /bommanoid_main_bottom/gnd -> /bommanoid_main_bottom/btn_x1
- J7 pad 2: /bommanoid_main_bottom/+3.3v regulator output -> /bommanoid_main_bottom/gnd
- J7 pad 3: /bommanoid_main_bottom/SPI0_SCK -> /bommanoid_main_bottom/btn_x2
- J7 pad 4: /bommanoid_main_bottom/SPI0_MOSI -> /bommanoid_main_bottom/gnd
- J7 pad 5: /bommanoid_main_bottom/OLED_RES -> /bommanoid_main_bottom/btn_x3
- J7 pad 6: /bommanoid_main_bottom/OLED_DC -> /bommanoid_main_bottom/gnd
- J7 pad 7: /bommanoid_main_bottom/OLED_CS -> /bommanoid_main_bottom/btn_x4
- NT1 pad 1: /bommanoid_main_top/+3.3v regulator output -> /bommanoid_main_top/3v3
- NT1 pad 2: D3v3 -> /bommanoid_main_top/d3v3
- R10 pad 1: Net-(J4-Pad4) -> /bommanoid_main_top/midi_in_ring
- R11 pad 1: /bommanoid_main_top/+3.3v regulator output -> /bommanoid_main_top/3v3
- R12 pad 1: Net-(J5-Pad4) -> /bommanoid_main_top/midi_out_ring
- R12 pad 2: /bommanoid_main_top/+3.3v regulator output -> /bommanoid_main_top/3v3
- R14 pad 1: /bommanoid_main_bottom/usb gnd -> /bommanoid_main_bottom/gnd
- R16 pad 1: Net-(D4-Pad1) -> Net-(D9-Pad1)
- R16 pad 2: /bommanoid_batt_top/gnd -> /bommanoid_main_bottom/gnd
- R17 pad 1: Net-(D6-Pad1) -> Net-(D10-Pad1)
- R17 pad 2: unconnected-(R17-Pad2) -> /bommanoid_main_bottom/gnd
- R18 pad 1: Net-(D9-Pad1) -> Net-(D11-Pad1)
- R18 pad 2: unconnected-(R18-Pad2) -> /bommanoid_main_bottom/gnd
- R19 pad 1: Net-(D10-Pad1) -> Net-(D12-Pad1)
- R19 pad 2: unconnected-(R19-Pad2) -> /bommanoid_main_bottom/gnd
- R22 pad 1: Net-(D13-Pad1) -> /bommanoid_main_bottom/gnd
- R22 pad 2: /bommanoid_batt_top/gnd from processor -> Net-(J17-Pad11)
- R23 pad 2: /bommanoid_batt_top/gnd from processor -> /bommanoid_main_bottom/gnd
- R24 pad 2: /bommanoid_batt_top/gnd from processor -> /bommanoid_main_bottom/gnd
- R25 pad 1: Net-(D16-Pad1) -> /bommanoid_main_bottom/gnd
- R25 pad 2: /bommanoid_batt_top/gnd from processor -> Net-(J6-PadA5)
- R34 pad 2: /gnd from processor -> /cab/gnd
- R35 pad 1: Net-(D7-Pad1) -> /cab/gnd
- R35 pad 2: /gnd from processor -> Net-(J30-Pad9)
- R36 pad 1: Net-(D8-Pad1) -> /cab/gnd
- R36 pad 2: /gnd from processor -> Net-(J30-Pad11)
- R37 pad 1: Net-(D9-Pad1) -> Net-(D24-Pad1)
- R37 pad 2: /gnd from processor -> /cab/gnd
- R4 pad 2: dac output L -> /bommanoid_main_top/aleft
- R40 pad 1: /+3.3v regulator output -> Net-(D29-Pad1)
- R40 pad 2: /I2C_SDA -> /bell/gnd
- R41 pad 1: /+3.3v regulator output -> Net-(D30-Pad1)
- R41 pad 2: /I2C_SCL -> /bell/gnd
- R5 pad 2: dac output R -> /bommanoid_main_top/aright
- R7 pad 1: /usb gnd -> /bommanoid_main_top/I2C_SDA
- R7 pad 2: Net-(J2-PadB5) -> /bommanoid_main_top/3v3
- R8 pad 2: /bommanoid_main_top/5v input -> /bommanoid_main_top/sys_5v
- SW1 pad 1: Net-(SW1-Pad1) -> /bommanoid_batt_top/gnd
- SW1 pad 2: /bommanoid_main_top/gnd -> Net-(R28-Pad2)
- U1 pad 1: A3v3 -> /bommanoid_main_top/a3v3
- U1 pad 10: /bommanoid_main_top/gnd from processor -> /bommanoid_main_top/gnd
- U1 pad 11: /bommanoid_main_top/gnd from processor -> /bommanoid_main_top/gnd
- U1 pad 16: /bommanoid_main_top/gnd from processor -> /bommanoid_main_top/gnd
- U1 pad 17: D3v3 -> /bommanoid_main_top/d3v3
- U1 pad 19: /bommanoid_main_top/gnd from processor -> /bommanoid_main_top/gnd
- U1 pad 20: D3v3 -> /bommanoid_main_top/d3v3
- U1 pad 8: A3v3 -> /bommanoid_main_top/a3v3
- U1 pad 9: AGND -> /bommanoid_main_top/agnd
- U2 pad 1: D3v3 -> /bommanoid_main_top/d3v3
- U2 pad 2: /bommanoid_main_top/gnd from processor -> /bommanoid_main_top/gnd
- U2 pad 3: D3v3 -> /bommanoid_main_top/d3v3
- U2 pad 5: A3v3 -> /bommanoid_main_top/a3v3
- U3 pad 1: /bommanoid_main_top/5v input -> /bommanoid_main_top/sys_5v
- U3 pad 5: /bommanoid_main_top/+3.3v regulator output -> /bommanoid_main_top/3v3
- U7 pad 3: Net-(D2-Pad2) -> /bommanoid_main_top/midi_in_tip
- U7 pad 5: /bommanoid_main_top/gnd from processor -> /bommanoid_main_top/gnd
- U7 pad 8: /bommanoid_main_top/5v from processor -> /bommanoid_main_top/sys_5v
Routing:
- net (no net): track 323.5 -> 0.00 mm, vias 10 -> 16
- net /+3.3v regulator output: track 229.9 -> 21.7 mm, vias 4 -> 2
- net /I2C_SCL: track 208.0 -> 0.00 mm, vias 4 -> 0
- net /I2C_SDA: track 203.3 -> 0.00 mm, vias 4 -> 0
- net /USB D-: track 137.2 -> 0.00 mm, vias 1 -> 0
- net /USB D+: track 137.0 -> 0.00 mm, vias 1 -> 0
- net /5v regulated: track 135.7 -> 0.00 mm, vias 4 -> 0
- net /Power board output +5v: track 115.2 -> 0.00 mm, vias 2 -> 0
- net Net-(J52-Pad6): track 93.4 -> 0.00 mm
- net Net-(J52-Pad5): track 92.3 -> 0.00 mm
- net /processor_mm/5v input: track 104.9 -> 12.8 mm
- net Net-(J52-Pad4): track 91.1 -> 0.00 mm
- net Net-(J52-Pad3): track 90.0 -> 0.00 mm
- net Net-(J52-Pad2): track 89.5 -> 0.00 mm
- net Net-(J52-Pad1): track 89.5 -> 0.00 mm
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- added copper zone on B.Cu, net (none)
- added copper zone on F.Cu, net (none)
- removed copper zone on B.Cu, net /captouch 3x3x1 GND
- removed copper zone on F.Cu, net /captouch 3x3x1 GND
- removed copper zone on B.Cu, net /gnd from processor
- removed copper zone on F.Cu, net /gnd from processor
- removed copper zone on B.Cu, net /processor_mm/gnd
- removed copper zone on F.Cu, net /processor_mm/gnd
- removed copper zone on B.Cu, net /usb gnd
- removed copper zone on F.Cu, net /usb gnd
- removed copper zone on B.Cu, net AGND
- removed copper zone on F.Cu, net AGND
Other:
- board size 1273.3 x 654.2 mm -> 1817.8 x 281.5 mm
- board text added: "+5v GND IN"
- board text added: "53x18 relay from tinytronics."
- board text added: "HDR to top - GND - bat + - usb 5v in - charge output 5v - key - charge led 1 - charge led 2 - charge led 3 - korg pwr led anode - korg oct led cathode"
- board text added: "LEDs ---------- amp power usb power 5v 5v post charger, post pot blink act1 act2 act3"
- board text added: "MOD"
- board text added: "NC COMM ON"
- board text added: "PITCH"
- board text added: "RJ45 thru"
- board text added: "TO TOP (pwr, 7p) - gnd - prg - 5v system (to top) - 3v3 (from top) - USB data + - USB data - - USB 5v (btn, 12p) - gnd - btn 1 - btn 2 - btn 3 - btn 4 - btn 5 - btn 6 - btn 7 - btn 8 - enc a - enc b - enc btn (led,midi,11p) - gnd - led1 (blink) - led2 (act1) - led3 (act2) - led4 (act3) - rj45_led_yellow - rj45_led_green - ws2812b data - midi out a - midi in a - midi in b (audio, 3p) - agnd - alef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"
- board text added: "WIRE: - korg oct -, gnd - korg oct +, gnd - korg oct-2 led, gnd - korg oct-1 led, gnd - korg oct+1 led, gnd - korg oct+2 led, gnd"
- board text added: "audio in"
- board text added: "holes enlarged by .5 M3 screws"
- board text added: "korg pwr"
- board text added: "to main: - gnd - USB 5v in - charge 5v out - AGND - Aleft-prepot - Aright-prepot - Aleft-postpot - Aright-postpot"
- board text removed: "1"
- board text removed: "10"
- board text removed: "11"
- board text removed: "12"
- board text removed: "13"
- board text removed: "14"
- board text removed: "2"
- board text removed: "3"
- board text removed: "3x3x1"
- board text removed: "4"
- board text removed: "5"
- board text removed: "6"
- board text removed: "7"
- board text removed: "8"
- board text removed: "9"
- board text removed: "AGND"
- board text removed: "AUDIO OUT"
- board text removed: "BATT BOTTOM"
- board text removed: "BATT TOP (top assembly)"
- board text removed: "D3v3"
- board text removed: "HDR to top - GND - bat + - charge led 1 - charge led 2 - charge led 3 - amp power +5v - korg oct led gnd - korg oct led 1 - korg oct led 2 - korg oct led 3 - korg oct led 4"
- board text removed: "I2C"
- board text removed: "KEY"
- board text removed: "LEDs usb power 5v 5v amp pwr 5v ws2812 system status"
- board text removed: "MIDI IN"
- board text removed: "MIDI OUT"
- board text removed: "PRG"
- board text removed: "SCL SDA +3v GND"
- board text removed: "TO TOP - gnd - prg - 5v system - 3v3 (from top) - USB data + - USB data - - USB 5v - gnd - btn 1 - btn 2 - btn 3 - btn 4 - enc a - enc b - enc btn - gnd - led3 - led4 - ws2812b data from top - midi out a - midi in a - midi in b - agnd - aleft-prepot - aright-prepot 7x OLED"
- board text removed: "WIRE: - korg gnd - korg oct - - korg oct +"
- board text removed: "amp pwr"
- board text removed: "bottom"
- board text removed: "clarinoid test device 2 3x3x1"
- board text removed: "clarinoid test device 2 4x4x3"
- board text removed: "gnd 3v3 5v scl sda BCK LRCK DIN MidiIn Midiout ws2812b SPI_SCK SPI_MOSI SPI_MISO oled_cs oled_res oled_dc enc_sw enc_a enc_b"
- board text removed: "gnd 3v3 sda scl"
- board text removed: "gnd usb+ usb- 5v led1 led2 led3 led4"
- board text removed: "octave leds"
- board text removed: "to main: - gnd - USB 5v in - 5v out - AGND - Aleft-prepot - Aright-prepot - Aleft-postpot - Aright-postpot"
- board text removed: "top"
- board text removed: "wire:key"
