File: CAD/bommanoid/bommanoid05/PH_breakout.kicad_sch (KiCad schematic)
At the start: 20 parts, among them J65 Conn_01x02, J66 Conn_01x03, J67 Conn_01x04, J68 Conn_01x02, J69 Conn_01x02, J70 Conn_01x03, J71 Conn_01x03, J72 Conn_01x04, J73 Conn_01x04, J74 Conn_01x05, J75 Conn_01x06, J76 Conn_01x08, J77 Conn_01x05, J78 Conn_01x05, J79 Conn_01x06, J80 Conn_01x06, J81 Conn_01x08, J82 Conn_01x08

Commit message: bommanoid05 sent to production
Parts:
- H21, H22, J65, J66, J67, J68, J70, J72, J74, J75, J76, J77, J79, J81: now left out of the parts list
- J69: LCSC (none) -> C49661; LCSC part number (none) -> C49661
- J71: LCSC (none) -> C146243; LCSC part number (none) -> C146243
- J73: LCSC (none) -> C2718488; LCSC part number (none) -> C2718488
- J78: LCSC (none) -> C50950; LCSC part number (none) -> C50950
- J80: LCSC (none) -> C40877; LCSC part number (none) -> C40877
- J82: LCSC (none) -> C27438; LCSC part number (none) -> C27438
Changed lines of the file:
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@@
   )
   (symbol (lib_id "Connector_Generic:Conn_01x05") (at 162.56 26.67 0) (unit 1)
-    (in_bom yes) (on_board yes) (fields_autoplaced)
+    (in_bom no) (on_board yes) (fields_autoplaced)
     (property "Reference" "J77" (id 0) (at 165.1 26.6699 0)
       (effects (font (size 1.27 1.27)) (justify left))
@@
   )
   (symbol (lib_id "Connector_Generic:Conn_01x02") (at 80.01 24.13 0) (unit 1)
-    (in_bom yes) (on_board yes) (fields_autoplaced)
+    (in_bom no) (on_board yes) (fields_autoplaced)
     (property "Reference" "J68" (id 0) (at 82.55 24.1299 0)
       (effects (font (size 1.27 1.27)) (justify left))
@@
     )
     (property "Datasheet" "~" (id 3) (at 162.56 129.54 0)
+      (effects (font (size 1.27 1.27)) hide)
+    )
+    (property "LCSC" "C27438" (id 4) (at 162.56 129.54 0)
+      (effects (font (size 1.27 1.27)) hide)
+    )
+    (property "LCSC part number" "C27438" (id 5) (at 162.56 129.54 0)
       (effects (font (size 1.27 1.27)) hide)
     )
@@
   )
   (symbol (lib_id "Connector_Generic:Conn_01x03") (at 80.01 52.07 0) (unit 1)
-    (in_bom yes) (on_board yes) (fields_autoplaced)
+    (in_bom no) (on_board yes) (fields_autoplaced)
     (property "Reference" "J70" (id 0) (at 82.55 52.0699 0)
       (effects (font (size 1.27 1.27)) (justify left))
@@
       (effects (font (size 1.27 1.27)) hide)
     )
+    (property "verif" "" (id 4) (at 80.01 31.75 0)
+      (effects (font (size 1.27 1.27)) hide)
+    )
+    (property "LCSC" "C49661" (id 5) (at 80.01 31.75 0)
+      (effects (font (size 1.27 1.27)) hide)
+    )
+    (property "LCSC part number" "C49661" (id 6) (at 80.01 31.75 0)
+      (effects (font (size 1.27 1.27)) hide)
+    )
     (pin "1")
     (pin "2")
@@
       (effects (font (size 1.27 1.27)) hide)
     )
+    (property "LCSC" "C40877" (id 4) (at 162.56 80.01 0)
+      (effects (font (size 1.27 1.27)) hide)
+    )
+    (property "LCSC part number" "C40877" (id 5) (at 162.56 80.01 0)
+      (effects (font (size 1.27 1.27)) hide)
+    )
     (pin "1")
     (pin "2")
@@
   )
   (symbol (lib_id "Connector_Generic:Conn_01x03") (at 29.21 62.23 0) (mirror y) (unit 1)
-    (in_bom yes) (on_board yes)
+    (in_bom no) (on_board yes)
     (property "Reference" "J66" (id 0) (at 29.21 49.53 0))
     (property "Value" "Conn_01x03" (id 1) (at 29.21 53.34 0))
@@
   )
   (symbol (lib_id "Connector_Generic:Conn_01x05") (at 111.76 43.18 0) (mirror y) (unit 1)
-    (in_bom yes) (on_board yes) (fields_autoplaced)
+    (in_bom no) (on_board yes) (fields_autoplaced)
     (property "Reference" "J74" (id 0) (at 111.76 31.75 0))
     (property "Value" "Conn_01x05" (id 1) (at 111.76 34.29 0))
@@
   )
   (symbol (lib_id "Connector_Generic:Conn_01x02") (at 29.21 31.75 0) (mirror y) (unit 1)
-    (in_bom yes) (on_board yes) (fields_autoplaced)
+    (in_bom no) (on_board yes) (fields_autoplaced)
     (property "Reference" "J65" (id 0) (at 29.21 25.4 0))
     (property "Value" "Conn_01x02" (id 1) (at 29.21 27.94 0))
@@
   )
   (symbol (lib_id "Connector_Generic:Conn_01x04") (at 29.21 90.17 0) (mirror y) (unit 1)
-    (in_bom yes) (on_board yes) (fields_autoplaced)
+    (in_bom no) (on_board yes) (fields_autoplaced)
     (property "Reference" "J67" (id 0) (at 29.21 81.28 0))
     (property "Value" "Conn_01x04" (id 1) (at 29.21 83.82 0))
@@
   )
   (symbol (lib_id "Connector_Generic:Conn_01x08") (at 162.56 105.41 0) (unit 1)
-    (in_bom yes) (on_board yes) (fields_autoplaced)
+    (in_bom no) (on_board yes) (fields_autoplaced)
     (property "Reference" "J81" (id 0) (at 165.1 104.1399 0)
       (effects (font (size 1.27 1.27)) (justify left))
@@
   )
   (symbol (lib_id "Connector_Generic:Conn_01x08") (at 111.76 129.54 0) (mirror y) (unit 1)
-    (in_bom yes) (on_board yes) (fields_autoplaced)
+    (in_bom no) (on_board yes) (fields_autoplaced)
     (property "Reference" "J76" (id 0) (at 111.76 115.57 0))
     (property "Value" "Conn_01x08" (id 1) (at 111.76 118.11 0))
@@
       (effects (font (size 1.27 1.27)) hide)
     )
+    (property "LCSC" "C50950" (id 4) (at 162.56 43.18 0)
+      (effects (font (size 1.27 1.27)) hide)
+    )
+    (property "LCSC part number" "C50950" (id 5) (at 162.56 43.18 0)
+      (effects (font (size 1.27 1.27)) hide)
+    )
     (pin "1")
     (pin "2")
@@
   )
   (symbol (lib_id "Connector_Generic:Conn_01x04") (at 80.01 77.47 0) (unit 1)
-    (in_bom yes) (on_board yes) (fields_autoplaced)
+    (in_bom no) (on_board yes) (fields_autoplaced)
     (property "Reference" "J72" (id 0) (at 82.55 77.4699 0)
       (effects (font (size 1.27 1.27)) (justify left))
@@
   )
   (symbol (lib_id "Connector_Generic:Conn_01x06") (at 111.76 80.01 0) (mirror y) (unit 1)
-    (in_bom yes) (on_board yes) (fields_autoplaced)
+    (in_bom no) (on_board yes) (fields_autoplaced)
     (property "Reference" "J75" (id 0) (at 111.76 68.58 0))
     (property "Value" "Conn_01x06" (id 1) (at 111.76 71.12 0))
@@
   )
   (symbol (lib_id "Mechanical:MountingHole") (at 198.12 24.13 0) (unit 1)
-    (in_bom yes) (on_board yes) (fields_autoplaced)
+    (in_bom no) (on_board yes) (fields_autoplaced)
     (property "Reference" "H21" (id 0) (at 200.66 21.5899 0)
       (effects (font (size 1.27 1.27)) (justify left))
@@
   )
   (symbol (lib_id "Mechanical:MountingHole") (at 201.93 39.37 0) (unit 1)
-    (in_bom yes) (on_board yes) (fields_autoplaced)
+    (in_bom no) (on_board yes) (fields_autoplaced)
     (property "Reference" "H22" (id 0) (at 204.47 36.8299 0)
       (effects (font (size 1.27 1.27)) (justify left))
@@
       (effects (font (size 1.27 1.27)) hide)
     )
+    (property "LCSC" "C146243" (id 4) (at 80.01 62.23 0)
+      (effects (font (size 1.27 1.27)) hide)
+    )
+    (property "LCSC part number" "C146243" (id 5) (at 80.01 62.23 0)
+      (effects (font (size 1.27 1.27)) hide)
+    )
     (pin "1")
     (pin "2")
@@
   )
   (symbol (lib_id "Connector_Generic:Conn_01x06") (at 162.56 60.96 0) (unit 1)
-    (in_bom yes) (on_board yes) (fields_autoplaced)
+    (in_bom no) (on_board yes) (fields_autoplaced)
     (property "Reference" "J79" (id 0) (at 165.1 60.9599 0)
       (effects (font (size 1.27 1.27)) (justify left))
@@
       (effects (font (size 1.27 1.27)) hide)
     )
+    (property "LCSC" "C2718488" (id 4) (at 80.01 90.17 0)
+      (effects (font (size 1.27 1.27)) hide)
+    )
+    (property "LCSC part number" "C2718488" (id 5) (at 80.01 90.17 0)
+      (effects (font (size 1.27 1.27)) hide)
+    )
