File: CAD/bommanoid/bommanoid05/bell.kicad_sch (KiCad schematic)
At the start: 25 parts, among them J31 RJ45_LED_Shielded

Commit message: bommanoid05 sent to production
Parts:
- D27, D28, D31, D33, D35, D36, D37, D38: LCSC (none) -> C2761795; LCSC part number (none) -> C2761795
- H15, H16: now left out of the parts list
- J31: LCSC (none) -> C464587; LCSC part number (none) -> C464587
Changed lines of the file:
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@@
       (effects (font (size 1.27 1.27)) (justify left top) hide)
+    )
+    (property "verif" "" (id 4) (at 76.2 152.4 0)
+      (effects (font (size 1.27 1.27)) hide)
+    )
+    (property "LCSC" "C2761795" (id 5) (at 76.2 152.4 0)
+      (effects (font (size 1.27 1.27)) hide)
+    )
+    (property "LCSC part number" "C2761795" (id 6) (at 76.2 152.4 0)
+      (effects (font (size 1.27 1.27)) hide)
     )
     (pin "1")
@@
       (effects (font (size 1.27 1.27)) (justify left top) hide)
     )
+    (property "verif" "" (id 4) (at 182.88 152.4 0)
+      (effects (font (size 1.27 1.27)) hide)
+    )
+    (property "LCSC" "C2761795" (id 5) (at 182.88 152.4 0)
+      (effects (font (size 1.27 1.27)) hide)
+    )
+    (property "LCSC part number" "C2761795" (id 6) (at 182.88 152.4 0)
+      (effects (font (size 1.27 1.27)) hide)
+    )
     (pin "1")
     (pin "2")
@@
       (effects (font (size 1.27 1.27)) (justify left top) hide)
     )
+    (property "verif" "" (id 4) (at 106.68 152.4 0)
+      (effects (font (size 1.27 1.27)) hide)
+    )
+    (property "LCSC" "C2761795" (id 5) (at 106.68 152.4 0)
+      (effects (font (size 1.27 1.27)) hide)
+    )
+    (property "LCSC part number" "C2761795" (id 6) (at 106.68 152.4 0)
+      (effects (font (size 1.27 1.27)) hide)
+    )
     (pin "1")
     (pin "2")
@@
       (effects (font (size 1.27 1.27)) (justify left top) hide)
     )
+    (property "verif" "" (id 4) (at 137.16 152.4 0)
+      (effects (font (size 1.27 1.27)) hide)
+    )
+    (property "LCSC" "C2761795" (id 5) (at 137.16 152.4 0)
+      (effects (font (size 1.27 1.27)) hide)
+    )
+    (property "LCSC part number" "C2761795" (id 6) (at 137.16 152.4 0)
+      (effects (font (size 1.27 1.27)) hide)
+    )
     (pin "1")
     (pin "2")
@@
   )
   (symbol (lib_id "Mechanical:MountingHole") (at 87.63 52.07 0) (unit 1)
-    (in_bom yes) (on_board yes) (fields_autoplaced)
+    (in_bom no) (on_board yes) (fields_autoplaced)
     (property "Reference" "H16" (id 0) (at 90.17 49.5299 0)
       (effects (font (size 1.27 1.27)) (justify left))
@@
   )
   (symbol (lib_id "Mechanical:MountingHole") (at 62.23 52.07 0) (unit 1)
-    (in_bom yes) (on_board yes) (fields_autoplaced)
+    (in_bom no) (on_board yes) (fields_autoplaced)
     (property "Reference" "H15" (id 0) (at 64.77 49.5299 0)
       (effects (font (size 1.27 1.27)) (justify left))
@@
       (effects (font (size 1.27 1.27)) (justify left top) hide)
     )
+    (property "verif" "" (id 4) (at 167.64 152.4 0)
+      (effects (font (size 1.27 1.27)) hide)
+    )
+    (property "LCSC" "C2761795" (id 5) (at 167.64 152.4 0)
+      (effects (font (size 1.27 1.27)) hide)
+    )
+    (property "LCSC part number" "C2761795" (id 6) (at 167.64 152.4 0)
+      (effects (font (size 1.27 1.27)) hide)
+    )
     (pin "1")
     (pin "2")
@@
       (effects (font (size 1.27 1.27)) (justify left top) hide)
     )
+    (property "verif" "" (id 4) (at 91.44 152.4 0)
+      (effects (font (size 1.27 1.27)) hide)
+    )
+    (property "LCSC" "C2761795" (id 5) (at 91.44 152.4 0)
+      (effects (font (size 1.27 1.27)) hide)
+    )
+    (property "LCSC part number" "C2761795" (id 6) (at 91.44 152.4 0)
+      (effects (font (size 1.27 1.27)) hide)
+    )
     (pin "1")
     (pin "2")
@@
       (effects (font (size 1.27 1.27)) (justify left top) hide)
     )
+    (property "verif" "" (id 4) (at 152.4 152.4 0)
+      (effects (font (size 1.27 1.27)) hide)
+    )
+    (property "LCSC" "C2761795" (id 5) (at 152.4 152.4 0)
+      (effects (font (size 1.27 1.27)) hide)
+    )
+    (property "LCSC part number" "C2761795" (id 6) (at 152.4 152.4 0)
+      (effects (font (size 1.27 1.27)) hide)
+    )
     (pin "1")
     (pin "2")
@@
       (effects (font (size 1.27 1.27)) (justify left top) hide)
     )
+    (property "verif" "" (id 4) (at 121.92 152.4 0)
+      (effects (font (size 1.27 1.27)) hide)
+    )
+    (property "LCSC" "C2761795" (id 5) (at 121.92 152.4 0)
+      (effects (font (size 1.27 1.27)) hide)
+    )
+    (property "LCSC part number" "C2761795" (id 6) (at 121.92 152.4 0)
+      (effects (font (size 1.27 1.27)) hide)
+    )
     (pin "1")
     (pin "2")
@@
       (effects (font (size 1.27 1.27)) hide)
     )
+    (property "LCSC" "C464587" (id 4) (at 195.58 48.26 0)
+      (effects (font (size 1.27 1.27)) hide)
+    )
+    (property "LCSC part number" "C464587" (id 5) (at 195.58 48.26 0)
+      (effects (font (size 1.27 1.27)) hide)
+    )
