File: CAD/bommanoid/bommanoid05/bommanoid_batt_bottom.kicad_sch (KiCad schematic)
At the start: 22 parts, among them J23 Conn_01x05, J24 Conn_01x05, J25 Conn_01x09, J26 Conn_01x02, J34 Conn_01x04, J53 Conn_01x04, J54 Conn_01x02, J55 Conn_01x04, J58 Conn_01x04

Commit message: bommanoid05 sent to production
Parts:
- D17: value 25% -> red; verif 1 -> (none)
- D18: value 50% -> red; verif 1 -> (none)
- D19: value 75% -> red; verif 1 -> (none)
- D20: value 100% -> red; verif 1 -> (none)
- D21, D22, H23, J26, J34, J53, J54, J55, J58: now left out of the parts list
- J23, J24: LCSC (none) -> C50950; LCSC part number (none) -> C50950
Changed lines of the file:
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@@
+      (effects (font (size 1.27 1.27)) hide)
+    )
+    (property "LCSC" "C50950" (id 4) (at 132.08 152.4 0)
+      (effects (font (size 1.27 1.27)) hide)
+    )
+    (property "LCSC part number" "C50950" (id 5) (at 132.08 152.4 0)
       (effects (font (size 1.27 1.27)) hide)
     )
@@
   )
   (symbol (lib_id "Mechanical:MountingHole") (at 102.87 113.03 0) (unit 1)
-    (in_bom yes) (on_board yes) (fields_autoplaced)
+    (in_bom no) (on_board yes) (fields_autoplaced)
     (property "Reference" "H23" (id 0) (at 105.41 111.7599 0)
       (effects (font (size 1.27 1.27)) (justify left))
@@
   )
   (symbol (lib_id "Connector_Generic:Conn_01x04") (at 257.81 162.56 0) (unit 1)
-    (in_bom yes) (on_board yes) (fields_autoplaced)
+    (in_bom no) (on_board yes) (fields_autoplaced)
     (property "Reference" "J55" (id 0) (at 260.35 162.5599 0)
       (effects (font (size 1.27 1.27)) (justify left))
@@
   )
   (symbol (lib_id "Connector_Generic:Conn_01x02") (at 257.81 125.73 0) (unit 1)
-    (in_bom yes) (on_board yes) (fields_autoplaced)
+    (in_bom no) (on_board yes) (fields_autoplaced)
     (property "Reference" "J26" (id 0) (at 260.35 125.7299 0)
       (effects (font (size 1.27 1.27)) (justify left))
@@
       (effects (font (size 1.27 1.27)) hide)
     )
+    (property "LCSC" "C50950" (id 4) (at 85.09 149.86 0)
+      (effects (font (size 1.27 1.27)) hide)
+    )
+    (property "LCSC part number" "C50950" (id 5) (at 85.09 149.86 0)
+      (effects (font (size 1.27 1.27)) hide)
+    )
     (pin "1")
     (pin "2")
@@
   )
   (symbol (lib_id "Connector_Generic:Conn_01x04") (at 34.29 154.94 0) (unit 1)
-    (in_bom yes) (on_board yes) (fields_autoplaced)
+    (in_bom no) (on_board yes) (fields_autoplaced)
     (property "Reference" "J34" (id 0) (at 36.83 153.6699 0)
       (effects (font (size 1.27 1.27)) (justify left))
@@
   )
   (symbol (lib_id "Device:LED") (at 191.77 96.52 90) (unit 1)
-    (in_bom yes) (on_board yes) (fields_autoplaced)
+    (in_bom no) (on_board yes) (fields_autoplaced)
     (property "Reference" "D21" (id 0) (at 195.58 96.8374 90)
       (effects (font (size 1.27 1.27)) (justify right))
@@
   )
   (symbol (lib_id "Connector_Generic:Conn_01x02") (at 257.81 152.4 0) (unit 1)
-    (in_bom yes) (on_board yes) (fields_autoplaced)
+    (in_bom no) (on_board yes) (fields_autoplaced)
     (property "Reference" "J54" (id 0) (at 260.35 152.3999 0)
       (effects (font (size 1.27 1.27)) (justify left))
@@
   )
   (symbol (lib_id "Connector_Generic:Conn_01x04") (at 257.81 175.26 0) (unit 1)
-    (in_bom yes) (on_board yes) (fields_autoplaced)
+    (in_bom no) (on_board yes) (fields_autoplaced)
     (property "Reference" "J58" (id 0) (at 260.35 175.2599 0)
       (effects (font (size 1.27 1.27)) (justify left))
@@
       (effects (font (size 1.27 1.27)) (justify right))
     )
-    (property "Value" "75%" (id 1) (at 124.46 86.6774 90)
+    (property "Value" "red" (id 1) (at 124.46 86.6774 90)
       (effects (font (size 1.27 1.27)) (justify right))
     )
@@
       (effects (font (size 1.27 1.27)) hide)
     )
-    (property "verif" "1" (id 5) (at 119.38 83.82 0)
+    (property "verif" "" (id 5) (at 119.38 83.82 0)
       (effects (font (size 1.27 1.27)) hide)
     )
@@
       (effects (font (size 1.27 1.27)) (justify left))
     )
-    (property "Value" "100%" (id 1) (at 134.62 84.7724 90)
+    (property "Value" "red" (id 1) (at 134.62 84.7724 90)
       (effects (font (size 1.27 1.27)) (justify left))
     )
@@
       (effects (font (size 1.27 1.27)) hide)
     )
-    (property "verif" "1" (id 5) (at 130.81 85.09 0)
+    (property "verif" "" (id 5) (at 130.81 85.09 0)
       (effects (font (size 1.27 1.27)) hide)
     )
@@
   )
   (symbol (lib_id "Device:LED") (at 201.93 96.52 90) (unit 1)
-    (in_bom yes) (on_board yes) (fields_autoplaced)
+    (in_bom no) (on_board yes) (fields_autoplaced)
     (property "Reference" "D22" (id 0) (at 205.74 96.8374 90)
       (effects (font (size 1.27 1.27)) (justify right))
@@
   )
   (symbol (lib_id "Connector_Generic:Conn_01x04") (at 257.81 135.89 0) (unit 1)
-    (in_bom yes) (on_board yes) (fields_autoplaced)
+    (in_bom no) (on_board yes) (fields_autoplaced)
     (property "Reference" "J53" (id 0) (at 260.35 135.8899 0)
       (effects (font (size 1.27 1.27)) (justify left))
@@
       (effects (font (size 1.27 1.27)) (justify right))
     )
-    (property "Value" "25%" (id 1) (at 102.235 86.6774 90)
+    (property "Value" "red" (id 1) (at 102.235 86.6774 90)
       (effects (font (size 1.27 1.27)) (justify right))
     )
@@
       (effects (font (size 1.27 1.27)) hide)
     )
-    (property "verif" "1" (id 5) (at 97.79 83.82 0)
+    (property "verif" "" (id 5) (at 97.79 83.82 0)
       (effects (font (size 1.27 1.27)) hide)
     )
@@
       (effects (font (size 1.27 1.27)) (justify left))
     )
-    (property "Value" "50%" (id 1) (at 114.3 83.5024 90)
+    (property "Value" "red" (id 1) (at 114.3 83.5024 90)
       (effects (font (size 1.27 1.27)) (justify left))
     )
@@
       (effects (font (size 1.27 1.27)) hide)
     )
-    (property "verif" "1" (id 5) (at 109.22 83.82 0)
-      (effects (font (size 1.27 1.27)) hide)
-    )
+    (property "verif" "" (id 5) (at 109.22 83.82 0)
+      (effects (font (size 1.27 1.27)) hide)
+    )
