File: CAD/bommanoid/bommanoid05/bommanoid_batt_top.kicad_sch (KiCad schematic)
At the start: 19 parts, among them IC3 Injoinic IP5306 battery charge, J20 Conn_01x05, J21 Conn_01x05

Commit message: bommanoid05 sent to production
Parts:
- C16, C26, C27, C28, C29, C30, C33, IC3, L1: verif 1 -> (none)
- C31, C32: LCSC (none) -> C12891; LCSC part number (none) -> C12891; verif 1 -> (none)
- D16: value korgpwr -> red; verif 1 -> (none)
- J20, J21: LCSC (none) -> C50950; LCSC part number (none) -> C50950
- R27: LCSC (none) -> C17942; LCSC part number (none) -> C17942; verif 1 -> (none)
- R28: LCSC (none) -> C17902; LCSC part number (none) -> C17902; verif 1 -> (none)
- R29: LCSC (none) -> C25340; LCSC part number (none) -> C25340; verif 1 -> (none)
Changed lines of the file:
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@@
       (effects (font (size 1.27 1.27)) hide)
     )
-    (property "LCSC part number" "" (id 4) (at 38.1 50.8 0)
-      (effects (font (size 1.27 1.27)) hide)
-    )
-    (property "verif" "1" (id 5) (at 38.1 50.8 0)
-      (effects (font (size 1.27 1.27)) hide)
-    )
-    (property "LCSC" "" (id 6) (at 38.1 50.8 0)
+    (property "LCSC part number" "C17942" (id 4) (at 38.1 50.8 0)
+      (effects (font (size 1.27 1.27)) hide)
+    )
+    (property "verif" "" (id 5) (at 38.1 50.8 0)
+      (effects (font (size 1.27 1.27)) hide)
+    )
+    (property "LCSC" "C17942" (id 6) (at 38.1 50.8 0)
       (effects (font (size 1.27 1.27)) hide)
     )
@@
       (effects (font (size 1.27 1.27)) hide)
     )
-    (property "verif" "1" (id 5) (at 106.68 50.8 0)
+    (property "verif" "" (id 5) (at 106.68 50.8 0)
       (effects (font (size 1.27 1.27)) hide)
     )
@@
       (effects (font (size 1.27 1.27)) hide)
     )
-    (property "verif" "1" (id 5) (at 83.82 50.8 0)
+    (property "verif" "" (id 5) (at 83.82 50.8 0)
       (effects (font (size 1.27 1.27)) hide)
     )
@@
       (effects (font (size 1.27 1.27)) hide)
     )
+    (property "LCSC" "C50950" (id 4) (at 201.93 142.24 0)
+      (effects (font (size 1.27 1.27)) hide)
+    )
+    (property "LCSC part number" "C50950" (id 5) (at 201.93 142.24 0)
+      (effects (font (size 1.27 1.27)) hide)
+    )
     (pin "1")
     (pin "2")
@@
       (effects (font (size 1.27 1.27)) (justify left))
     )
-    (property "Value" "korgpwr" (id 1) (at 175.26 98.7424 90)
+    (property "Value" "red" (id 1) (at 175.26 98.7424 90)
       (effects (font (size 1.27 1.27)) (justify left))
     )
@@
       (effects (font (size 1.27 1.27)) hide)
     )
-    (property "verif" "1" (id 5) (at 172.72 99.06 0)
+    (property "verif" "" (id 5) (at 172.72 99.06 0)
       (effects (font (size 1.27 1.27)) hide)
     )
@@
       (effects (font (size 1.27 1.27)) hide)
     )
-    (property "LCSC part number" "" (id 4) (at 101.6 60.96 0)
-      (effects (font (size 1.27 1.27)) hide)
-    )
-    (property "verif" "1" (id 5) (at 101.6 60.96 0)
-      (effects (font (size 1.27 1.27)) hide)
-    )
-    (property "LCSC" "" (id 6) (at 101.6 60.96 0)
+    (property "LCSC part number" "C17902" (id 4) (at 101.6 60.96 0)
+      (effects (font (size 1.27 1.27)) hide)
+    )
+    (property "verif" "" (id 5) (at 101.6 60.96 0)
+      (effects (font (size 1.27 1.27)) hide)
+    )
+    (property "LCSC" "C17902" (id 6) (at 101.6 60.96 0)
       (effects (font (size 1.27 1.27)) hide)
     )
@@
       (effects (font (size 1.27 1.27)) hide)
     )
-    (property "verif" "1" (id 5) (at 127 54.61 0)
+    (property "verif" "" (id 5) (at 127 54.61 0)
       (effects (font (size 1.27 1.27)) hide)
     )
@@
       (effects (font (size 1.27 1.27)) hide)
     )
-    (property "verif" "1" (id 5) (at 141.605 35.56 0)
+    (property "verif" "" (id 5) (at 141.605 35.56 0)
       (effects (font (size 1.27 1.27)) hide)
     )
@@
       (effects (font (size 1.27 1.27)) hide)
     )
-    (property "LCSC part number" "" (id 4) (at 154.94 35.56 0)
-      (effects (font (size 1.27 1.27)) hide)
-    )
-    (property "verif" "1" (id 5) (at 154.94 35.56 0)
-      (effects (font (size 1.27 1.27)) hide)
-    )
-    (property "LCSC" "" (id 6) (at 154.94 35.56 0)
+    (property "LCSC part number" "C12891" (id 4) (at 154.94 35.56 0)
+      (effects (font (size 1.27 1.27)) hide)
+    )
+    (property "verif" "" (id 5) (at 154.94 35.56 0)
+      (effects (font (size 1.27 1.27)) hide)
+    )
+    (property "LCSC" "C12891" (id 6) (at 154.94 35.56 0)
       (effects (font (size 1.27 1.27)) hide)
     )
@@
       (effects (font (size 1.27 1.27)) hide)
     )
+    (property "LCSC" "C50950" (id 4) (at 245.11 142.24 0)
+      (effects (font (size 1.27 1.27)) hide)
+    )
+    (property "LCSC part number" "C50950" (id 5) (at 245.11 142.24 0)
+      (effects (font (size 1.27 1.27)) hide)
+    )
     (pin "1")
     (pin "2")
@@
       (effects (font (size 1.27 1.27)) hide)
     )
-    (property "verif" "1" (id 5) (at 114.935 62.23 0)
+    (property "verif" "" (id 5) (at 114.935 62.23 0)
       (effects (font (size 1.27 1.27)) hide)
     )
@@
       (effects (font (size 1.27 1.27)) hide)
     )
-    (property "verif" "1" (id 5) (at 127 35.56 0)
+    (property "verif" "" (id 5) (at 127 35.56 0)
       (effects (font (size 1.27 1.27)) hide)
     )
@@
       (effects (font (size 1.27 1.27)) hide)
     )
-    (property "verif" "1" (id 5) (at 47.625 50.8 0)
+    (property "verif" "" (id 5) (at 47.625 50.8 0)
       (effects (font (size 1.27 1.27)) hide)
     )
@@
       (effects (font (size 1.27 1.27)) hide)
     )
-    (property "verif" "1" (id 5) (at 38.1 58.42 0)
+    (property "verif" "" (id 5) (at 38.1 58.42 0)
       (effects (font (size 1.27 1.27)) hide)
     )
@@
       (effects (font (size 1.27 1.27)) hide)
     )
-    (property "verif" "1" (id 5) (at 182.88 35.56 0)
+    (property "verif" "" (id 5) (at 182.88 35.56 0)
       (effects (font (size 1.27 1.27)) hide)
     )
@@
       (effects (font (size 1.27 1.27)) hide)
     )
-    (property "LCSC part number" "" (id 4) (at 114.935 54.61 0)
-      (effects (font (size 1.27 1.27)) hide)
-    )
-    (property "verif" "1" (id 5) (at 114.935 54.61 0)
-      (effects (font (size 1.27 1.27)) hide)
-    )
-    (property "LCSC" "" (id 6) (at 114.935 54.61 0)
+    (property "LCSC part number" "C25340" (id 4) (at 114.935 54.61 0)
+      (effects (font (size 1.27 1.27)) hide)
+    )
+    (property "verif" "" (id 5) (at 114.935 54.61 0)
+      (effects (font (size 1.27 1.27)) hide)
+    )
+    (property "LCSC" "C25340" (id 6) (at 114.935 54.61 0)
       (effects (font (size 1.27 1.27)) hide)
     )
@@
       (effects (font (size 1.27 1.27)) hide)
     )
-    (property "LCSC part number" "" (id 4) (at 170.18 35.56 0)
-      (effects (font (size 1.27 1.27)) hide)
-    )
-    (property "verif" "1" (id 5) (at 170.18 35.56 0)
-      (effects (font (size 1.27 1.27)) hide)
-    )
-    (property "LCSC" "" (id 6) (at 170.18 35.56 0)
-      (effects (font (size 1.27 1.27)) hide)
-    )
+    (property "LCSC part number" "C12891" (id 4) (at 170.18 35.56 0)
+      (effects (font (size 1.27 1.27)) hide)
+    )
+    (property "verif" "" (id 5) (at 170.18 35.56 0)
+      (effects (font (size 1.27 1.27)) hide)
+    )
+    (property "LCSC" "C12891" (id 6) (at 170.18 35.56 0)
+      (effects (font (size 1.27 1.27)) hide)
+    )
