File: CAD/bommanoid/bommanoid05/bommanoid_main_bottom.kicad_sch (KiCad schematic)
At the start: 52 parts, among them J10 Conn_01x07, J11 Amphenol ACJS-MHOM, J12 Amphenol ACJS-MHOM, J13 Conn_01x09, J14 Amphenol ACJS-MHOM, J15 Conn_01x12, J16 Conn_01x12, J18 Conn_01x03, J19 Conn_01x07, J22 Conn_01x06, J32 USB_A, J33 Conn_01x08, J49 Conn_01x04, J50 Conn_01x04, J51 Conn_01x04, J52 Conn_01x04, J56 Conn_01x02, J57 Conn_01x06, J7 Conn_01x04, J8 Conn_01x04, J83 Conn_01x15, J9 Conn_01x02, U8 ssd1306_graphic

Commit message: bommanoid05 sent to production
Parts:
- added H37: MountingHole_M3, MountingHole:MountingHole_3.2mm_M3, symbol Mechanical:MountingHole
- C21, C22, C23, C24: LCSC (none) -> C12891; LCSC part number (none) -> C12891; verif 1 -> (none)
- C25, U8: verif 1 -> (none)
- H24, J22, J32, J33, J49, J50, J51, J52, J56, J57, J7, J8, J83, J9, NT4, NT5: now left out of the parts list
- J10, J19: LCSC (none) -> C358721; LCSC part number (none) -> C358721
- J13: LCSC (none) -> C39576; LCSC part number (none) -> C39576
- J15, J16: LCSC (none) -> C350303; LCSC part number (none) -> C350303
- J18: LCSC (none) -> C146243; LCSC part number (none) -> C146243
