File: CAD/bommanoid/bommanoid05/bommanoid_main_top.kicad_sch (KiCad schematic)
At the start: 70 parts, among them IC1 SN74AHCT125N, IC2 SN74AHCT125N, J1 Conn_01x07, J2 Conn_01x09, J3 Conn_01x12, J4 Conn_01x12, J5 Conn_01x03, U1 PCM5102A, U2 TLV75733PDBV, U3 TLV75733PDBV, U4 APCI0108-P001A Teensy_4.0_Mic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, U5 TCA9554PW, U6 Micromod outline, U7 6N138

Commit message: bommanoid05 sent to production
Parts:
- C1, C10, C11, C12, C13, C14, C15, C17, C18, C19, C2, C3, C4, C5, C6, C7, C8, C9, D1, D2, H1, NT1, R1, R10, R11, R12, R13, R2, R3, R4, R5, R6, R7, R8, U1, U2, U3, U4, U6, U7: verif 1 -> (none)
- C20: LCSC C49678 -> C24497; LCSC part number C49678 -> C24497; verif 1 -> (none)
- DS1, J1, J2, J3, J4, J5: now left out of the parts list
- R47, R48, R49, R50, R51, R52, R53, R54, R57, R58, R59, R60, R61, R62, R63: LCSC (none) -> C17557; LCSC part number (none) -> C17557
- U5: LCSC (none) -> C477924; LCSC part number (none) -> C477924
