File: CAD/bommanoid/bommanoid05/cab.kicad_sch (KiCad schematic)
At the start: 32 parts, among them J27 Amphenol ACJS-MHOM, J28 Conn_01x02, J29 RJ45_LED_Shielded, J30 RJ45_LED_Shielded, J35 Conn_02x02_Odd_Even, J36 Conn_01x02, J37 Conn_01x02, J38 Barrel_Jack_MountingPin, J39 Conn_01x03, J40 Conn_01x02, J41 Conn_01x02, J42 Conn_01x02, J43 Conn_01x04, J44 Conn_01x02, J45 Conn_01x02, J46 Conn_01x02, J47 Conn_01x02, J48 Conn_01x02, U9 LM7809_TO220

Commit message: bommanoid05 sent to production
Parts:
- removed J35: Conn_02x02_Odd_Even, Connector_PinHeader_2.54mm:PinHeader_2x02_P2.54mm_Vertical, symbol Connector_Generic:Conn_02x02_Odd_Even
- added C34: 0.33uF, Capacitor_SMD:C_1206_3216Metric, symbol Device:C
- added C35: 0.1uF, Capacitor_SMD:C_1206_3216Metric, symbol Device:C
- added H33, H34, H35, H36: MountingHole_M3, MountingHole:MountingHole_3.2mm_M3, symbol Mechanical:MountingHole
- added J17, J35, J6: AudioOut, clarinoid2:SWITCHCRAFT_35RAPC4BV4_OvalHoles, symbol clarinoid2:Switchcraft 35RAPC4BV4
- H13, H14, H17, J28, J36, J37, J38, J39, J40, J41, J42, J43, J44, J45, J46, J47, J48, NT2, NT3: now left out of the parts list
- J29, J30: LCSC (none) -> C464587; LCSC part number (none) -> C464587
- R34: footprint Resistor_THT:R_Axial_Power_L25.0mm_W9.0mm_P27.94mm -> Resistor_THT:R_Axial_DIN0207_L6.3mm_D2.5mm_P10.16mm_Horizontal
Connections:
- net agnd: now also J17.1 (S-GND), J35.1 (S-GND), J6.1 (S-GND)
- net ain_postpot: now also J17.5, J6.2 (Tip)
- net amp_9v: now also C35.1
- net gnd: now also C34.2, C35.2
- net powerbank_12v+: now also C34.1
- new net ain_postfx: J17.2 (Tip), J35.2 (Tip)
- no-connect marks 4 -> 12
Other:
- note added: "audioin"
- note added: "fxin"
- note added: "fxout"
- note added: "pot"
- note added: "toamp"
- note removed: "audio"
- note removed: "audio in"
- note removed: "pot connector"
- moved on the sheet: J27, J38, J39, J48
