File: CAD/bommanoid/bommanoid05/clarinoid-devboard.kicad_sch (KiCad schematic)
At the start: 13 parts, among them U11 mousebite2mm, U12 mousebite2mm, U13 mousebite2mm, U14 mousebite2mm, U15 mousebite2mm

Commit message: bommanoid05 sent to production
Parts:
- added U16, U17, U21, U24: mousebite2mm_45deg, clarinoid2:mouse-bite-2mm-45deg, symbol clarinoid2:Placeholder
- added U18, U19, U20, U22, U23, U25, U26, U27, U28, U29, U30, U31, U32, U33, U34, U35, U36, U37, U38, U39: mousebite2mm, clarinoid2:mouse-bite-2mm-slot, symbol clarinoid2:Placeholder
- H25, H26, H27, H28, H29, H30, H31, H32: now left out of the parts list
Other:
- note added: "main assembly"
- moved on the sheet: U14
