File: CAD/clarinoid3-bodytest/04/clarinoid-bodytest.kicad_pcb (KiCad board)
At the start: 2 copper layers, 467.9 x 112.2 mm, 131 parts, among them IC1 PCA9554APW,118, IC2 Injoinic IP5306 battery charge, IC3 PCA9554APW,118, J1 header i2c pressure, J10 LH header multi to main, J11 microSD SOFNG TF-15x15, J12 main header multi to LH, J13 clarinoid3 main usb interconn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, J14 header_i2c_lh to pressure, J15 clarinoid3 DAC and POT subboa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, J16 AudioOut, J17 clarinoid3 main usb interconn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, J18 header lh_keys, J19 clarinoid3 DAC and POT subboa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, J2 lh_header_i2c_main, J21 encoder header, J3 MIDI IN, J4 MIDI OUT, J5 XKB_U262-16XN-4BVC11 USB-C re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, J6 RH touch keys header, J7 I2C HEADER main to PITCH, J8 CapTouchSlider3, J9 OLED_HEADER, SW1 sw_batteryindicator, SW10 SW_x1, SW11 SW_x2, SW12 SW_x3, SW13 SW_y1, SW14 SW_y2, SW2 sw_RHx1, SW3 sw_RHx2, SW4 sw_RHx3, SW5 sw_RHx4, SW6 sw_program, SW7 SW_OK, SW9 SW_BACK, U1 Pressure1_0x28_I2C0, U10 MPR121, 0x5A, U11 MPR121, 0x5A, U12 octave_keys_6, U15 OK cutout, U16 BACK cutout, U17 OLED graphic, U18 encoder cutout, U2 APCI0108-P001A Teensy_4.0_Mic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, U3 Micromod outline, U4 PCM5102A, U5 TLV75533PDBV, U6 6N138, U7 TLV75733PDBV, U8 MPR121, 0x5A, U9 WS2812_HEADER LH to external

Commit message: c3 cad sketches
Parts:
- added BT1: Battery_Cell, Battery:BatteryHolder_Keystone_1042_1x18650, B.Cu at (229.9, 382.9)
- added C1: 10uF, Capacitor_SMD:C_0402_1005Metric, F.Cu at (149.9, 419.9)
- added C10: 0.1uF, Capacitor_SMD:C_0402_1005Metric, F.Cu at (150.1, 417.1)
- added C11: 0.1uF, Capacitor_SMD:C_0402_1005Metric, F.Cu at (150.1, 414.9)
- added C12: 10uF, Capacitor_SMD:C_0402_1005Metric, F.Cu at (162.1, 418.9)
- added C13: 0.1uF, Capacitor_SMD:C_0402_1005Metric, F.Cu at (161.0, 418.9)
- added C3: 0.1uF, Capacitor_SMD:C_0402_1005Metric, F.Cu at (151.0, 419.9)
- added C4: 2.2uF, Capacitor_SMD:C_0402_1005Metric, F.Cu at (161.7, 416.5)
- added C5: 2.2uF, Capacitor_SMD:C_0402_1005Metric, F.Cu at (156.1, 420.7)
- added C6: 2.2uF, Capacitor_SMD:C_0402_1005Metric, F.Cu at (156.0, 431.7)
- added C7: 10uF, Capacitor_SMD:C_0402_1005Metric, F.Cu at (150.1, 418.2)
- added C8: 10uF, Capacitor_SMD:C_0402_1005Metric, F.Cu at (150.1, 416.0)
- added C9: 2.2uF, Capacitor_SMD:C_0402_1005Metric, F.Cu at (163.0, 424.5)
- added D2: 25%, LED_SMD:LED_0402_1005Metric, F.Cu at (222.2, 419.0)
- added D3: 50%, LED_SMD:LED_0402_1005Metric, F.Cu at (222.2, 417.5)
- added D4: 75%, LED_SMD:LED_0402_1005Metric, F.Cu at (222.2, 416.0)
- added D5: 100%, LED_SMD:LED_0402_1005Metric, F.Cu at (222.2, 414.5)
- added J11: microSD SOFNG TF-15x15, clarinoid2:SOFNG TF-15x15 (LCSC C111196), F.Cu at (208.7, 421.6)
- added J13: clarinoid3 main usb interconnect 12p, clarinoid2:clarinoid3-sd subboard castellated, F.Cu at (180.7, 414.0)
- added J15: clarinoid3 DAC and POT subboard interconnect, clarinoid2:Bourns_POT_PTR902-2020K-A103 Panel subboard castellated header, B.Cu at (158.5, 429.4)
- added J16: AudioOut, clarinoid2:SWITCHCRAFT_35RAPC4BV4_OvalHoles, B.Cu at (150.9, 385.9)
- added J19: clarinoid3 DAC and POT subboard interconnect, clarinoid2:Bourns_POT_PTR902-2020K-A103 Panel interconnect, F.Cu at (131.2, 373.3)
- added J3: MIDI IN, clarinoid2:SWITCHCRAFT_35RAPC4BV4_OvalHoles, B.Cu at (117.9, 385.9)
- added J4: MIDI OUT, clarinoid2:SWITCHCRAFT_35RAPC4BV4_OvalHoles, B.Cu at (100.4, 385.9)
- added J5: XKB_U262-16XN-4BVC11 USB-C recept, clarinoid2:USB_C_Receptacle_XKB_U262-16XN-4BVC11, F.Cu at (184.6, 425.8)
- added NT1: NetTie_2, NetTie:NetTie-2_SMD_Pad0.5mm, F.Cu at (150.5, 421.4)
- added R1: 22R, Resistor_SMD:R_0402_1005Metric, F.Cu at (149.6, 429.1)
- added R11: 10k, Resistor_SMD:R_0402_1005Metric, F.Cu at (217.8, 423.8)
- added R13: 5.1k, Resistor_SMD:R_0805_2012Metric, F.Cu at (186.8, 418.5)
- added R14: 5.1k, Resistor_SMD:R_0805_2012Metric, F.Cu at (182.7, 418.5)
- added R2: 22R, Resistor_SMD:R_0402_1005Metric, F.Cu at (148.5, 429.1)
- added R21: PTR902-2020K-A103, SamacSys_Parts:PTR902-2020K-A103, B.Cu at (156.0, 434.4)
- added R3: 22R, Resistor_SMD:R_0402_1005Metric, F.Cu at (150.7, 429.1)
- added R4: 470R, Resistor_SMD:R_0402_1005Metric, F.Cu at (158.1, 432.0)
- added R5: 470R, Resistor_SMD:R_0402_1005Metric, F.Cu at (161.5, 424.0)
- added SW1: sw_batteryindicator, clarinoid2:XKB switch jlcpcb SW_TS-1187A-B-A-B, F.Cu at (222.2, 424.0)
- added SW12: SW_x3, clarinoid2:MB2511S2G45, F.Cu at (5.12, 389.5)
- added SW12: SW_x3, clarinoid2:MB2511S2G45, F.Cu at (-98.9, 389.5)
- added SW12: SW_x3, clarinoid2:MB2511S2G45, F.Cu at (-112.9, 389.5)
- added SW12: SW_x3, clarinoid2:MB2511S2G45, F.Cu at (20.1, 389.5)
- added SW12: SW_x3, clarinoid2:MB2511S2G45, F.Cu at (59.1, 389.5)
- added SW12: SW_x3, clarinoid2:MB2511S2G45, F.Cu at (74.1, 389.5)
- added SW12: SW_x3, clarinoid2:MB2511S2G45, F.Cu at (-139.3, 389.5)
- added SW12: SW_x3, clarinoid2:MB2511S2G45, F.Cu at (-152.9, 389.5)
- added SW6: sw_program, clarinoid2:XKB switch jlcpcb SW_TS-1187A-B-A-B, F.Cu at (195.2, 424.0)
- added U15: OK cutout, clarinoid2:MB2511S4W01-BC, F.Cu at (-126.1, 393.4)
- added U15: OK cutout, clarinoid2:MB2511S4W01-BC, F.Cu at (-162.1, 393.4)
- added U18: encoder cutout, clarinoid2:Bourns_ENC_PEC11R-4215F-S0024 panel cutout shaft downward, F.Cu at (-71.1, 390.9)
- added U4: PCM5102A, Package_SO:TSSOP-20_4.4x6.5mm_P0.65mm, F.Cu at (156.0, 416.3)
- added U5: TLV75533PDBV, Package_TO_SOT_SMD:SOT-23-5, F.Cu at (151.3, 423.8)
Routing:
- net Net-(D2-Pad1): track 28.1 -> 56.2 mm
- net Net-(J13-Pad14): track 27.4 -> 54.8 mm, vias 1 -> 2
- net /DAC/a3v3: track 27.2 -> 54.4 mm
- net /DAC/dac_gnd: track 22.4 -> 44.9 mm, vias 12 -> 24
- net Net-(J13-Pad13): track 22.3 -> 44.5 mm, vias 1 -> 2
- net Net-(R2-Pad2): track 20.4 -> 40.9 mm
- net /DAC/dac_sw2: track 20.4 -> 40.8 mm
- net Net-(R1-Pad2): track 20.1 -> 40.2 mm
- net Net-(D4-Pad2): track 20.1 -> 40.1 mm
- net Net-(R4-Pad1): track 20.0 -> 40.0 mm, vias 2 -> 4
- net /USBSocket/usb bus 5v in: track 19.9 -> 39.8 mm
- net Net-(R3-Pad2): track 19.6 -> 39.2 mm, vias 2 -> 4
- net /DAC/D3v3: track 15.8 -> 31.6 mm
- net /DAC/dac_sw1: track 15.3 -> 30.6 mm
- net Net-(J13-Pad11): track 14.8 -> 29.7 mm
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Other:
- board size 467.9 x 112.2 mm -> 739 x 217.2 mm
- board text added: "- 41mm top key to bottom of octave key - c2 nutserts extend 5mm over top of pipe"
- board text added: "34/30"
- board text added: "34/30 pipe 3mm clearance from M6 top key to PCB yields 25mm assembly area for PCB"
- board text added: "34/30 pipe assuming 3d printed inner skeleton placing a 12mm OD air hose in the chamber and floating the PCB inside the chamber 5mm assembly clearance yeilds max 27mm height assemblable with NO body breach"
- board text added: "34/30 pipe inner skeleton, let's maximize space between tube & pcb"
- board text added: "roughly 42mm from top of key to bottom of oct"

Commit message: c3 pcb iteration
Parts:
- removed the U15 at (-126.1, 393.4)
- removed the U15 at (-162.1, 393.4)
- added SW12: SW_x3, clarinoid2:MB2511S2G45, F.Cu at (-477.6, 24.8)
- added SW12: SW_x3, clarinoid2:MB2511S2G45, F.Cu at (-440.6, 24.8)
- moved C10 485.7 mm to (-163.4, 46.1)
- moved C4 485.7 mm to (-151.8, 45.5)
- moved C8 485.7 mm to (-163.4, 45.0)
- moved D2 485.7 mm to (-91.3, 48.0)
- moved D3 485.7 mm to (-91.3, 46.5)
- moved D4 485.7 mm to (-91.3, 45.0)
- moved D5 485.7 mm to (-91.3, 43.5)
- moved J11 485.7 mm to (-104.8, 50.6)
- moved J13 485.7 mm to (-132.8, 43.0)
- moved J19 485.7 mm to (-182.3, 2.31)
- moved J5 485.7 mm to (-128.9, 54.8)
- moved R1 485.7 mm to (-163.9, 58.1)
- moved R11 485.7 mm to (-95.7, 52.8)
- moved R13 485.7 mm to (-126.7, 47.5)
- moved R14 485.7 mm to (-130.8, 47.5)
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Routing:
- net (no net): vias 4 -> 12
Other:
- board size 739 x 217.2 mm -> 467.9 x 234.3 mm
- board text added: "CROSS"
- board text added: "HLD: choose encoder"
- board text added: "HLD: top LEDs"
- board text added: "SIDE VIEW"
- board text added: "TOP VIEW"
- board text added: "screw on this side to fix in place and clamp the sidewall of the other side"
- board text added: "there is technically space for hose + an 18650 battery. but nothing left. might be able to find a creative way? but how to make batt contacts reliable"
- board text added: "this could also be built into a sidewall to be fixed to the side tube."
- board text added: "~90 mm to work with 12/8 hose 36/32 pipe ~15mm barb len - maxdiam ~9.5 sensor top-intake, 14x14 rough footprint"
