File: CAD/clarinoid3-bodytest/04/clarinoid-bodytest.kicad_pcb (KiCad board)
At the start: 2 copper layers, 467.9 x 234.3 mm, 181 parts, among them IC1 PCA9554APW,118, IC2 Injoinic IP5306 battery charge, IC3 PCA9554APW,118, J1 header i2c pressure, J10 LH header multi to main, J11 microSD SOFNG TF-15x15, J12 main header multi to LH, J13 clarinoid3 main usb interconn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, J14 header_i2c_lh to pressure, J15 clarinoid3 DAC and POT subboa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, J16 AudioOut, J17 clarinoid3 main usb interconn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, J18 header lh_keys, J19 clarinoid3 DAC and POT subboa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, J2 lh_header_i2c_main, J21 encoder header, J3 MIDI IN, J4 MIDI OUT, J5 XKB_U262-16XN-4BVC11 USB-C re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, J6 RH touch keys header, J7 I2C HEADER main to PITCH, J8 CapTouchSlider3, J9 OLED_HEADER, SW1 sw_batteryindicator, SW10 SW_x1, SW11 SW_x2, SW12 SW_x3, SW13 SW_y1, SW14 SW_y2, SW2 sw_RHx1, SW3 sw_RHx2, SW4 sw_RHx3, SW5 sw_RHx4, SW6 sw_program, SW7 SW_OK, SW9 SW_BACK, U1 Pressure1_0x28_I2C0, U10 MPR121, 0x5A, U11 MPR121, 0x5A, U12 octave_keys_6, U15 OK cutout, U16 BACK cutout, U17 OLED graphic, U18 encoder cutout, U2 APCI0108-P001A Teensy_4.0_Mic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, U3 Micromod outline, U4 PCM5102A, U5 TLV75533PDBV, U6 6N138, U7 TLV75733PDBV, U8 MPR121, 0x5A, U9 WS2812_HEADER LH to external

Commit message: c3 design work adding more 3dp tests
Parts:
- removed D7, D8: WS2812B, LED_SMD:LED_WS2812B_PLCC4_5.0x5.0mm_P3.2mm
- removed REF**: Teensy 4.1, teensy:Teensy41
- added C30: 0.1uF, Capacitor_SMD:C_0603_1608Metric, F.Cu at (63.1, -250.9)
- added J11: microSD SOFNG TF-15x15, clarinoid2:SOFNG TF-15x15 (LCSC C111196), F.Cu at (-198.4, 241.9)
- added J16: AudioOut, clarinoid2:SWITCHCRAFT_35RAPC4BV4_OvalHoles, B.Cu at (-156.1, 261.0)
- added J16: AudioOut, clarinoid2:SWITCHCRAFT_35RAPC4BV4_OvalHoles, B.Cu at (-150.3, 181.4)
- added J19: clarinoid3 DAC and POT subboard interconnect, clarinoid2:Bourns_POT_PTR902-2020K-A103 Panel interconnect, F.Cu at (-220.1, 249.0)
- added J3: MIDI IN, clarinoid2:SWITCHCRAFT_35RAPC4BV4_OvalHoles, B.Cu at (-169.1, 261.0)
- added J3: MIDI IN, clarinoid2:SWITCHCRAFT_35RAPC4BV4_OvalHoles, B.Cu at (-167.1, 183.0)
- added J4: MIDI OUT, clarinoid2:SWITCHCRAFT_35RAPC4BV4_OvalHoles, B.Cu at (-184.6, 183.0)
- added J4: MIDI OUT, clarinoid2:SWITCHCRAFT_35RAPC4BV4_OvalHoles, B.Cu at (-182.1, 261.0)
- added J5: XKB_U262-16XN-4BVC11 USB-C recept, clarinoid2:USB_C_Receptacle_XKB_U262-16XN-4BVC11, F.Cu at (-198.8, 261.7)
- U1: footprint SamacSys_Parts:ABPMAND001PG2A3 -> clarinoid2:Honeywell-ABPMAND001PG2A3
- moved U1 314.4 mm to (80.7, -263.1), turned to 90 degrees
- moved H8 297.3 mm to (64.4, -238.4)
- moved J1 272.9 mm to (50.4, -250.6)
- moved J9 55.4 mm to (-167.1, -195.7)
- moved J6 50.1 mm to (-285.1, -184.3)
- moved J7 46.4 mm to (-306.6, -188.7)
- moved U2 39.5 mm to (-161.2, -210.5)
- moved H1 39.5 mm to (-182.9, -214.5)
- moved U3 39.5 mm to (-165.4, -213.2)
- moved J12 36.5 mm to (-253.0, -189.5)
Connections:
- BT1 pad 1: (no net) -> /MainBoard/power/batt+
- BT1 pad 2: (no net) -> /MainBoard/main_gnd
- IC3 pad 9: Net-(IC3-Pad9) -> Net-(IC3-IO4)
- SW12 pad 1: (no net) -> /LHBoard/lh_gnd (x10)
- SW12 pad 2: (no net) -> Net-(IC3-IO4) (x10)
- SW12 pad 2: Net-(IC3-Pad9) -> Net-(IC3-IO4)
- U1 pad 1: /PressureBoard/pressure_gnd -> Net-(U1-GND)
Routing:
- net /PressureBoard/pressure_sck: track 19.4 -> 0.00 mm
- net /PressureBoard/pressure_sda: track 15.0 -> 0.00 mm
- net /PressureBoard/pressure_gnd: track 9.38 -> 0.00 mm
- net /PressureBoard/pressure_3v3: track 6.06 -> 0.00 mm
- removed copper zone on B.Cu, net /PressureBoard/pressure_gnd
- removed copper zone on F.Cu, net /PressureBoard/pressure_gnd
Other:
- board size 467.9 x 234.3 mm -> 614.7 x 342.6 mm
- board text added: "BATT 24x100"
- board text added: "BATTERY"
- board text added: "LH CONTROLS"
- board text added: "MAIN"
- board text added: "Main pcb"
- board text added: "OLED"
- board text added: "PB pcb"
- board text added: "PCB HLD"
- board text added: "PITCH 12x100"
- board text added: "PRESSURE"
- board text added: "RH CONTROLS"
- board text added: "RH CONTROLS 28x"
- board text added: "RH controls PCB"
- board text added: "TOPDOWN"
- board text added: "header"
- board text added: "hose"
- board text added: "m.2"
- board text added: "plumbing 100"
- board text removed: "SIDE VIEW"
- board text removed: "TOP VIEW"
- board text removed: "there is technically space for hose + an 18650 battery. but nothing left. might be able to find a creative way? but how to make batt contacts reliable"

Commit message: c3 design notes
Parts:
- added R21: PTR902-2020K-A103, SamacSys_Parts:PTR902-2020K-A103, B.Cu at (-80.0, 897.0)
- added R21: PTR902-2020K-A103, SamacSys_Parts:PTR902-2020K-A103, B.Cu at (-78.5, 841.3)
- added R21: PTR902-2020K-A103, SamacSys_Parts:PTR902-2020K-A103, B.Cu at (-267.0, 491.1)
- added REF**: LED_SK6805_PLCC4_2.4x2.7mm_P1.3mm, LED_SMD:LED_SK6805_PLCC4_2.4x2.7mm_P1.3mm, F.Cu at (-463.9, -56.7)
- added REF**: LED_SK6805_PLCC4_2.4x2.7mm_P1.3mm, LED_SMD:LED_SK6805_PLCC4_2.4x2.7mm_P1.3mm, F.Cu at (-473.0, -67.5)
- added REF**: LED_SK6805_PLCC4_2.4x2.7mm_P1.3mm, LED_SMD:LED_SK6805_PLCC4_2.4x2.7mm_P1.3mm, F.Cu at (-445.9, -90.1)
- added REF**: LED_SK6805_PLCC4_2.4x2.7mm_P1.3mm, LED_SMD:LED_SK6805_PLCC4_2.4x2.7mm_P1.3mm, F.Cu at (-459.8, -89.9)
- added REF**: LED_SK6805_PLCC4_2.4x2.7mm_P1.3mm, LED_SMD:LED_SK6805_PLCC4_2.4x2.7mm_P1.3mm, F.Cu at (-455.2, -89.8)
- added REF**: LED_SK6805_PLCC4_2.4x2.7mm_P1.3mm, LED_SMD:LED_SK6805_PLCC4_2.4x2.7mm_P1.3mm, F.Cu at (-472.9, -76.7)
- added REF**: LED_SK6805_PLCC4_2.4x2.7mm_P1.3mm, LED_SMD:LED_SK6805_PLCC4_2.4x2.7mm_P1.3mm, F.Cu at (-468.5, -56.7)
- added REF**: LED_SK6805_PLCC4_2.4x2.7mm_P1.3mm, LED_SMD:LED_SK6805_PLCC4_2.4x2.7mm_P1.3mm, F.Cu at (-473.0, -72.1)
- added REF**: LED_SK6805_PLCC4_2.4x2.7mm_P1.3mm, LED_SMD:LED_SK6805_PLCC4_2.4x2.7mm_P1.3mm, F.Cu at (-440.4, -80.6)
- added REF**: LED_SK6805_PLCC4_2.4x2.7mm_P1.3mm, LED_SMD:LED_SK6805_PLCC4_2.4x2.7mm_P1.3mm, F.Cu at (-450.7, -89.9)
- added REF**: LED_SK6805_PLCC4_2.4x2.7mm_P1.3mm, LED_SMD:LED_SK6805_PLCC4_2.4x2.7mm_P1.3mm, F.Cu at (-445.4, -56.9)
- added REF**: LED_SK6805_PLCC4_2.4x2.7mm_P1.3mm, LED_SMD:LED_SK6805_PLCC4_2.4x2.7mm_P1.3mm, F.Cu at (-440.3, -76.1)
- added REF**: LED_SK6805_PLCC4_2.4x2.7mm_P1.3mm, LED_SMD:LED_SK6805_PLCC4_2.4x2.7mm_P1.3mm, F.Cu at (-450.2, -56.7)
- added REF**: LED_SK6805_PLCC4_2.4x2.7mm_P1.3mm, LED_SMD:LED_SK6805_PLCC4_2.4x2.7mm_P1.3mm, F.Cu at (-473.0, -62.9)
- added REF**: LED_SK6805_PLCC4_2.4x2.7mm_P1.3mm, LED_SMD:LED_SK6805_PLCC4_2.4x2.7mm_P1.3mm, F.Cu at (-473.0, -81.2)
- added REF**: LED_SK6805_PLCC4_2.4x2.7mm_P1.3mm, LED_SMD:LED_SK6805_PLCC4_2.4x2.7mm_P1.3mm, F.Cu at (-454.7, -56.6)
- added REF**: LED_SK6805_PLCC4_2.4x2.7mm_P1.3mm, LED_SMD:LED_SK6805_PLCC4_2.4x2.7mm_P1.3mm, F.Cu at (-473.2, -86.0)
- added REF**: LED_SK6805_PLCC4_2.4x2.7mm_P1.3mm, LED_SMD:LED_SK6805_PLCC4_2.4x2.7mm_P1.3mm, F.Cu at (-440.6, -85.4)
- added REF**: LED_SK6805_PLCC4_2.4x2.7mm_P1.3mm, LED_SMD:LED_SK6805_PLCC4_2.4x2.7mm_P1.3mm, F.Cu at (-440.4, -62.3)
- added REF**: LED_SK6805_PLCC4_2.4x2.7mm_P1.3mm, LED_SMD:LED_SK6805_PLCC4_2.4x2.7mm_P1.3mm, F.Cu at (-440.4, -71.5)
- added REF**: LED_SK6805_PLCC4_2.4x2.7mm_P1.3mm, LED_SMD:LED_SK6805_PLCC4_2.4x2.7mm_P1.3mm, F.Cu at (-440.4, -66.9)
- added REF**: LED_SK6805_PLCC4_2.4x2.7mm_P1.3mm, LED_SMD:LED_SK6805_PLCC4_2.4x2.7mm_P1.3mm, F.Cu at (-469.0, -89.9)
- added REF**: LED_SK6805_PLCC4_2.4x2.7mm_P1.3mm, LED_SMD:LED_SK6805_PLCC4_2.4x2.7mm_P1.3mm, F.Cu at (-464.4, -89.9)
- added REF**: LED_SK6805_PLCC4_2.4x2.7mm_P1.3mm, LED_SMD:LED_SK6805_PLCC4_2.4x2.7mm_P1.3mm, F.Cu at (-459.3, -56.7)
Other:
- outline, holes or cut-outs redrawn
- board text added: "15mm shaft is similar profile as the audio jacks PTR902-1015K-A103"
- board text added: "< 1,6mm >"
- board text added: "Main & RH controls cannot be 1 PCB because hose must go Behind the pCB, but battery needs to be there. only way would be to put the battery outside."
- board text added: "POT"
- board text added: "PTR902 with castelaltion subboard, cutout in main pcb, leaves little space for hose."
- board text added: "TODO: consider not pcb-mounting the 18650. solder the leads and it can drop down into the PCB in a hole. take a different approach: make the difficult stuff / highly constrained stuff as easy as possible, then fill in"
- board text added: "and with the vertical headers, the RH controls looks nice. The issue now is there's no room for the hose. actually i don't see any way of making that work."
- board text added: "audio 3,5mm"
- board text added: "but if we maintain the same offset as the battery then there's space for the PTR-902. Q: how does hose pass through the main pcb? just a hole to allow passthrough is sufficient."
- board text added: "difficulty of this 2-tier PCB is that i need to figure out how to route battery, hose, etc."
- board text added: "in order to fit battery, main cannot be centered. which means LHcontrols + RHcontrols cannot just be opposite side offsets, IF main+battery are to be on same plane. 1,6mm offset is actually min as shown. that is pretty convenient because it's almost a PCB thickness, implying a castellated connection resolves diffreences between RH and LH controls. pin header is too high. so margin is narrow here."
- board text added: "microSD"
- board text added: "this orientation (flat main pcb) comes with conflicts as well: pitch bend PCB is sorta inaccessible., or leaves no room for hose"
- board text added: "vertical mounting pot is too high"
- board text added: "with 25mm shaft, the vert pot if i go through a board, exposes 12mm of shaft. C2 exposes about 12mm, but the knob only requires probably 8-9. so this {dblquote}should{dblquote} work. NOTE: this is a D-shaft, not knurled so i need a different knob type."
- board text removed: "CROSS"
