File: CAD/clarinoid3-bodytest/04/clarinoid-bodytest.kicad_pcb (KiCad board)
At the start: 2 copper layers, 614.7 x 342.6 mm, 215 parts, among them IC1 PCA9554APW,118, IC2 Injoinic IP5306 battery charge, IC3 PCA9554APW,118, J1 header i2c pressure, J10 LH header multi to main, J11 microSD SOFNG TF-15x15, J12 main header multi to LH, J13 clarinoid3 main usb interconn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, J14 header_i2c_lh to pressure, J15 clarinoid3 DAC and POT subboa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, J16 AudioOut, J17 clarinoid3 main usb interconn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, J18 header lh_keys, J19 clarinoid3 DAC and POT subboa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, J2 lh_header_i2c_main, J21 encoder header, J3 MIDI IN, J4 MIDI OUT, J5 XKB_U262-16XN-4BVC11 USB-C re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, J6 RH touch keys header, J7 I2C HEADER main to PITCH, J8 CapTouchSlider3, J9 OLED_HEADER, SW1 sw_batteryindicator, SW10 SW_x1, SW11 SW_x2, SW12 SW_x3, SW13 SW_y1, SW14 SW_y2, SW2 sw_RHx1, SW3 sw_RHx2, SW4 sw_RHx3, SW5 sw_RHx4, SW6 sw_program, SW7 SW_OK, SW9 SW_BACK, U1 Pressure1_0x28_I2C0, U10 MPR121, 0x5A, U11 MPR121, 0x5A, U12 octave_keys_6, U15 OK cutout, U16 BACK cutout, U17 OLED graphic, U18 encoder cutout, U2 APCI0108-P001A Teensy_4.0_Mic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, U3 Micromod outline, U4 PCM5102A, U5 TLV75533PDBV, U6 6N138, U7 TLV75733PDBV, U8 MPR121, 0x5A, U9 WS2812_HEADER LH to external

Commit message: ìter c3 body
Parts:
- added LED**: SK6805EC15, library_loader:SK6805EC15, F.Cu at (-359.3, -65.0)
- added LED**: SK6805EC15, library_loader:SK6805EC15, F.Cu at (-348.8, -89.5)
- added LED**: SK6805EC15, library_loader:SK6805EC15, F.Cu at (-348.8, -82.5)
- added LED**: SK6805EC15, library_loader:SK6805EC15, F.Cu at (-348.8, -79.0)
- added LED**: SK6805EC15, library_loader:SK6805EC15, F.Cu at (-348.8, -100.0)
- added LED**: SK6805EC15, library_loader:SK6805EC15, F.Cu at (-383.8, -82.5)
- added LED**: SK6805EC15, library_loader:SK6805EC15, F.Cu at (-348.8, -96.5)
- added LED**: SK6805EC15, library_loader:SK6805EC15, F.Cu at (-359.3, -100.0)
- added LED**: SK6805EC15, library_loader:SK6805EC15, F.Cu at (-373.3, -65.0)
- added LED**: SK6805EC15, library_loader:SK6805EC15, F.Cu at (-383.8, -86.0)
- added LED**: SK6805EC15, library_loader:SK6805EC15, F.Cu at (-348.8, -93.0)
- added LED**: SK6805EC15, library_loader:SK6805EC15, F.Cu at (-383.8, -72.0)
- added LED**: SK6805EC15, library_loader:SK6805EC15, F.Cu at (-373.3, -100.0)
- added LED**: SK6805EC15, library_loader:SK6805EC15, F.Cu at (-376.8, -100.0)
- added LED**: SK6805EC15, library_loader:SK6805EC15, F.Cu at (-380.3, -100.0)
- added LED**: SK6805EC15, library_loader:SK6805EC15, F.Cu at (-369.8, -100.0)
- added LED**: SK6805EC15, library_loader:SK6805EC15, F.Cu at (-383.8, -79.0)
- added LED**: SK6805EC15, library_loader:SK6805EC15, F.Cu at (-348.8, -72.0)
- added LED**: SK6805EC15, library_loader:SK6805EC15, F.Cu at (-383.8, -75.5)
- added LED**: SK6805EC15, library_loader:SK6805EC15, F.Cu at (-366.3, -65.0)
- added LED**: SK6805EC15, library_loader:SK6805EC15, F.Cu at (-355.8, -65.0)
- added LED**: SK6805EC15, library_loader:SK6805EC15, F.Cu at (-380.3, -65.0)
- added LED**: SK6805EC15, library_loader:SK6805EC15, F.Cu at (-362.8, -65.0)
- added LED**: SK6805EC15, library_loader:SK6805EC15, F.Cu at (-383.8, -100.0)
- added LED**: SK6805EC15, library_loader:SK6805EC15, F.Cu at (-352.3, -65.0)
- added LED**: SK6805EC15, library_loader:SK6805EC15, F.Cu at (-348.8, -86.0)
- added LED**: SK6805EC15, library_loader:SK6805EC15, F.Cu at (-376.8, -65.0)
- added LED**: SK6805EC15, library_loader:SK6805EC15, F.Cu at (-348.8, -68.5)
- added LED**: SK6805EC15, library_loader:SK6805EC15, F.Cu at (-362.8, -100.0)
- added LED**: SK6805EC15, library_loader:SK6805EC15, F.Cu at (-383.8, -68.5)
- added LED**: SK6805EC15, library_loader:SK6805EC15, F.Cu at (-366.3, -100.0)
- added LED**: SK6805EC15, library_loader:SK6805EC15, F.Cu at (-383.8, -89.5)
- added LED**: SK6805EC15, library_loader:SK6805EC15, F.Cu at (-352.3, -100.0)
- added LED**: SK6805EC15, library_loader:SK6805EC15, F.Cu at (-383.8, -65.0)
- added LED**: SK6805EC15, library_loader:SK6805EC15, F.Cu at (-348.8, -75.5)
- added LED**: SK6805EC15, library_loader:SK6805EC15, F.Cu at (-369.8, -65.0)
- added LED**: SK6805EC15, library_loader:SK6805EC15, F.Cu at (-348.8, -65.0)
- added LED**: SK6805EC15, library_loader:SK6805EC15, F.Cu at (-383.8, -93.0)
- added LED**: SK6805EC15, library_loader:SK6805EC15, F.Cu at (-383.8, -96.5)
- added LED**: SK6805EC15, library_loader:SK6805EC15, F.Cu at (-355.8, -100.0)
- added R21: PTR902-2020K-A103, SamacSys_Parts:PTR902-2020K-A103, B.Cu at (-8.08, 653.0)
- added U17: OLED graphic, clarinoid2:SSD1306_128x64_approximate, F.Cu at (-380.2, -96.5)
- moved R21 113.0 mm to (-190.7, 827.3)
- moved R21 113.0 mm to (-192.1, 883.0)
Other:
- outline, holes or cut-outs redrawn
- board text added: "18650"
- board text added: "if we sink the battery under the pcb a bit, we gain space to center the PCB. this is important because it means a single main board, and the same connectivity for LH and RH."
